File: resources/V9958_kicad/VT.kicad_sch (KiCad schematic)
At the start: 0 parts

Commit message: update 20240921
Parts:
- added TP? (x3): ~, symbol Connector:TestPoint
- added U1000, U1002, U1004, U1006, U913, U914, U915, U916, U917, U918, U919, U920, U921, U922, U937, U941, U942, U944, U946, U948, U950, U951, U953, U955, U958, U959, U962, U963, U966, U967, U970, U971, U974, U976, U977, U979, U982, U984, U985, U987, U989, U990, U994, U996, U998: NMOS, symbol Raki_ASIC_cells:NMOS
- added U1001, U1003, U1005, U806, U812, U836, U837, U844, U845, U846, U847, U848, U849, U850, U851, U852, U854, U900, U923, U928, U943, U945, U947, U957, U961, U965, U969, U973, U975, U981, U983, U993, U995, U997, U999: INV, symbol Raki_ASIC_cells:INV
- added U142: GT043, symbol Raki_ASIC_cells:NOR3
- added U143 (x9), U808, U810, U813: NOR2, symbol Raki_ASIC_cells:NOR2
- added U145: GT013, symbol Raki_ASIC_cells:VY_CONSTCNTR1
- added U145: GT011, symbol Raki_ASIC_cells:VY_CONSTCNTR1
- added U145: GT001, symbol Raki_ASIC_cells:VY_CONSTCNTR1
- added U145: GT009, symbol Raki_ASIC_cells:VY_CONSTCNTR1
- added U145: GT000, symbol Raki_ASIC_cells:VY_CONSTCNTR1
- added U145: GT002, symbol Raki_ASIC_cells:VY_CONSTCNTR1
- added U145: GT012, symbol Raki_ASIC_cells:VY_CONSTCNTR1
- added U145: GT003, symbol Raki_ASIC_cells:VY_CONSTCNTR1
- added U145: GT010, symbol Raki_ASIC_cells:VY_CONSTCNTR1
- added U661: GT008, symbol Raki_ASIC_cells:VY_DDL_small
- added U661: GT019, symbol Raki_ASIC_cells:VY_DDL_small
- added U661: GT020, symbol Raki_ASIC_cells:VY_DDL_small
- added U687: GT005, symbol Raki_ASIC_cells:NOR2
- added U689: GT004, symbol Raki_ASIC_cells:AOI21
- added U792: GT006, symbol Raki_ASIC_cells:NOR2
- added U793: GT007, symbol Raki_ASIC_cells:NOR2
- added U795: GT014, symbol Raki_ASIC_cells:NOR2
- added U796: GT015, symbol Raki_ASIC_cells:NOR2
- added U797: GT016, symbol Raki_ASIC_cells:AOI21
- added U798: GT017, symbol Raki_ASIC_cells:AOI21
- added U804: GT018, symbol Raki_ASIC_cells:AOI21
- added U807: GT021, symbol Raki_ASIC_cells:AOI31
- added U809: NOR3, symbol Raki_ASIC_cells:NOR3
- added U811, U949, U952, U954, U956, U960, U964, U968, U972, U978, U980, U986, U988, U991, U992: INVP, symbol Raki_ASIC_cells:INVP
- added U814: GT045, symbol Raki_ASIC_cells:VY_DDL_small
- added U817: GT046, symbol Raki_ASIC_cells:VY_DDL_small
- added U819, U822, U823, U830, U834, U835: DDL, symbol Raki_ASIC_cells:VY_DDL_small
- added U821: GT026, symbol Raki_ASIC_cells:NOR2
- added U824: GT027, symbol Raki_ASIC_cells:VY_DDL_small
- added U825: GT028, symbol Raki_ASIC_cells:VY_DDL_small
- added U826: GT029, symbol Raki_ASIC_cells:NAND2
- added U827: GT030, symbol Raki_ASIC_cells:VY_DDL_small
- added U828: GT031, symbol Raki_ASIC_cells:NAND2
- added U829: GT032, symbol Raki_ASIC_cells:VY_DDL_small
- added U831: GT035, symbol Raki_ASIC_cells:NOR4
- added U832: GT034, symbol Raki_ASIC_cells:OR3
- added U833: GT033, symbol Raki_ASIC_cells:NOR2
- added U838: GT037, symbol Raki_ASIC_cells:VY_DDL_small
- added U839: GT038, symbol Raki_ASIC_cells:VY_DDL_small
- added U840: GT039, symbol Raki_ASIC_cells:VY_DDL_small
- added U841: GT036, symbol Raki_ASIC_cells:VY_DDL_small
- added U842: GT041, symbol Raki_ASIC_cells:VY_DDL_small
- added U843: NAND2, symbol Raki_ASIC_cells:NAND2
- added U853, U855, U856, U857, U858, U859, U860, U861, U862, U863, U864, U865, U866, U867, U868, U869, U870, U871, U872, U873, U874, U875, U876, U877, U878, U879, U880, U881, U882, U883, U884, U885, U886, U887, U888, U889, U890, U891, U892, U893, U894, U895, U896, U897, U898, U901, U902, U903, U904, U905, U906, U907, U908, U909, U910, U911, U912: NORWIDE, symbol Raki_ASIC_cells:NORWIDE
- added U899: GT040, symbol Raki_ASIC_cells:NOR2
- added U924: GT044, symbol Raki_ASIC_cells:VY_DSR_small
- added U925: GT047, symbol Raki_ASIC_cells:VY_DDL_small
- added U926: GT022, symbol Raki_ASIC_cells:VY_DSR_small
- added U932: GT042, symbol Raki_ASIC_cells:NOR2
- added U933: GT023, symbol Raki_ASIC_cells:VY_DSR_small
- added U934: GT024, symbol Raki_ASIC_cells:VY_DSR_small
- added U935: GT048, symbol Raki_ASIC_cells:VY_DDL_small
- added U936: GT025, symbol Raki_ASIC_cells:VY_DSR_small
- added U940: GT049, symbol Raki_ASIC_cells:VY_DDL_small
Connections:
- new net: U876., U966.
- new net: U965., U966.
- new net: U865., U937.
- new net: U143., U143., U925. (Φ1)
- new net: U943., U944.
- new net: U868., U944.
- new net: U1004., U877.
- new net: U981., U982.
- new net: U959., U960.
- new net: U953., U954.
- new net: U873., U958.
- new net: U957., U958.
- new net: U808., U809., U810., U813., U824. (Φ1), U825. (Φ1)
- new net: U809., U933. (Φ2)
- new net: U809., U926. (Φ2)
- new net: U809., U924. (Φ2)
- new net: U1005., U1006.
- new net: U878., U970.
- new net: U973., U974.
- new net: U830. (Φ1), U831.
- new net: U807., U829. (Φ1), U830. (Φ1)
- new net: U947., U948.
- new net: U828., U838. (Φ1), U842. (Φ1), U924. (Φ2)
- new net: U821., U828., U926. (Φ2)
- new net: U828., U829. (Φ1)
- new net: U813., U934. (Φ2)
- new net: U808., U934. (Φ2)
- new net: U963., U964.
- new net: U871., U948.
- new net: U142., U823. (Φ1), U826., U834. (Φ1)
- new net: U142., U143.
- new net: U142., U143., U843.
- new net: U143., U143. (x4)
- new net: U143., U143., U817. (Φ1)
- new net: U1006., U880.
- new net: U955., U956.
- new net: U863., U921.
- new net: U870., U998.
- new net: U861., U919.
- new net: U971., U972.
- new net: U879., U982.
- new net: U867., U941.
- new net: U813., U933. (Φ2)
- new net: U143., U143., U935. (Φ1)
- new net: U995., U996.
- new net: U983., U984.
- new net: U969., U970.
- new net: TP?.1, U145. (~{DOUT}), U661. (Φ1)
- new net: U993., U994.
- new net: U979., U980.
- new net: U862., U920.
- new net: TP?.1, U661. (Φ1), U687., U689., U792., U793.
- new net: U145. (~{DOUT}), U793.
- new net: U882., U994.
- new net: U821., U823. (Φ1)
- new net: U825. (Φ1), U826., U827. (Φ1)
- new net: U145. (~{DOUT}), U145. (~{DOUT}), U145. (~{DOUT}), U145. (~{DOUT}), U145. (~{DOUT}), U661. (Φ1), U832.
- new net: U145. (~{DOUT}), U804.
- new net: U145. (~{DOUT}), U145. (~{DOUT}) (x7)
- new net: U807., U824. (Φ1), U826.
- new net: U812., U915.
- new net: U857., U915.
- new net: U842. (Φ1), U843.
- new net: U821., U822. (Φ1)
- new net: U949., U950.
- new net: U869., U946.
- new net: U945., U946.
- new net: U687., U689., U796., U797., U798., U804., U840. (Φ1)
- new net: U827. (Φ1), U831., U832., U840. (Φ1)
- new net: U874., U962.
- new net: U807., U838. (Φ1)
- new net: U1002., U875.
- new net: U145. (~{DOUT}), U797.
- new net: U145. (~{DOUT}), U145. (~{DOUT}), U145. (~{DOUT}), U145. (~{DOUT}), U661. (Φ1), U836.
- new net: U145. (~{DOUT}), U687.
- new net: U860., U918.
- new net: U843., U900.
- new net: U661. (Φ1), U795., U796., U797., U798., U804.
- new net: TP?.1, U689., U795., U797., U798., U804., U839. (Φ1)
- new net: U961., U962.
- new net: U143., U143., U940. (Φ1)
- new net: U831., U836.
- new net: U866., U942.
- new net: U807., U819. (Φ1)
- new net: U810., U819. (Φ1)
- new net: U864., U922.
- new net: U145. (~{DOUT}), U796.
- new net: U997., U998.
- new net: U808., U936. (Φ2)
- new net: U810., U936. (Φ2)
- new net: U831., U832., U841. (Φ1)
- new net: U977., U978.
- new net: U858., U916.
- new net: U989., U991.
- new net: U831., U832., U833., U839. (Φ1)
- new net: U975., U976.
- new net: U883., U996.
- new net: U985., U986.
- new net: U914., U923.
- new net: U856., U914.
- new net: U145. (~{DOUT}), U689.
- new net: U967., U968.
- new net: U1003., U1004.
- new net: U1001., U1002.
- new net: U990., U992.
- new net: U859., U917.
- new net: U145. (~{DOUT}), U795.
- new net: U806., U807.
- new net: U833., U835. (Φ1)
- new net: U835. (Φ1), U932.
- new net: U145. (~{DOUT}), U792.
- new net: U837., U913.
- new net: U853., U913.
- new net: U145. (~{DOUT}), U798.
- new net: U951., U952.
- new net: U987., U988.
- new net: U1000., U999.
- new net: U1000., U872.
- new net: U928., U942.
- new net: U833., U834. (Φ1)
- new net: U661. (Φ1), U806.
- new net: U881., U984.
- new net CLK.phiL: U1000., U1002., U1004., U1006., U661. (Φ1), U661. (Φ1), U819. (Φ1), U824. (Φ1), U829. (Φ1), U838. (Φ1), U839. (Φ1), U840. (Φ1), U913., U914., U915., U916., U917., U918., U919., U920., U921., U922., U924. (Φ2), U926. (Φ2), U933. (Φ2), U934. (Φ2), U936. (Φ2), U937., U941., U942., U944., U946., U948., U958., U962., U966., U970., U974., U976., U982., U984., U994., U996., U998.
- new net CLK.~{phiL}: U145. (~{DOUT}), U145. (~{DOUT}), U145. (~{DOUT}), U145. (~{DOUT}), U145. (~{DOUT}), U145. (~{DOUT}), U145. (~{DOUT}), U145. (~{DOUT}), U145. (~{DOUT}), U661. (Φ1), U814. (Φ1), U817. (Φ1), U822. (Φ1), U823. (Φ1), U825. (Φ1), U827. (Φ1), U830. (Φ1), U834. (Φ1), U835. (Φ1), U841. (Φ1), U842. (Φ1), U924. (Φ2), U925. (Φ1), U926. (Φ2), U933. (Φ2), U934. (Φ2), U935. (Φ1), U936. (Φ2), U940. (Φ1)
- new net GND: U145. (~{DOUT}), U145. (~{DOUT}), U145. (~{DOUT}), U145. (~{DOUT}), U145. (~{DOUT}), U145. (~{DOUT}), U145. (~{DOUT}), U145. (~{DOUT}), U145. (~{DOUT})
- new net NET.PLA.~{TXTMODE}: U145. (~{DOUT}), U145. (~{DOUT}), U145. (~{DOUT}), U145. (~{DOUT}), U145. (~{DOUT}), U145. (~{DOUT}), U145. (~{DOUT}), U145. (~{DOUT}), U145. (~{DOUT}), U844., U845., U846., U847., U848., U849., U850., U851., U852., U853., U854., U855., U856., U857., U858., U859., U860., U861., U862., U863., U864., U865., U866., U867., U868., U869., U870., U871., U872., U873., U874., U875., U876., U877., U878., U879., U880., U881., U882., U883., U884., U885., U886., U887., U888., U889., U899., U900., U974., U976.
- new net NET.PLA0.CNTR.~{D_{0}}_0.5Z: U973., U989.
- new net NET.PLA0.CNTR.~{D_{0}}_Z: U991.
- new net NET.PLA0.CNTR.~{D_{3}}_0.5Z: U975., U990.
- new net NET.PLA0.CNTR.~{D_{3}}_Z: U992.
- new net NET.PLA0.COL_{10}: U143., U143., U937.
- new net NET.PLA0.COL_{12}: U143., U941.
- new net NET.PLA0.COL_{3}: U143., U916.
- new net NET.PLA0.COL_{4}: U917., U932.
- new net NET.PLA0.COL_{5}: U143., U143., U918.
- new net NET.PLA0.COL_{6}: U919., U932.
- new net NET.PLA0.COL_{7}: U143., U811., U920.
- new net NET.PLA0.COL_{8}: U143., U143., U921.
- new net NET.PLA0.COL_{9}: U142., U922.
- new net NET.PLA0.M16CYC10: U980.
- new net NET.PLA0.M16CYC11: U978.
- new net NET.PLA0.M16CYC8: U986.
- new net NET.PLA0.M16CYC9: U988.
- new net NET.PLA0.M8CYC0: U949.
- new net NET.PLA0.M8CYC1: U952.
- new net NET.PLA0.M8CYC2: U954.
- new net NET.PLA0.M8CYC3: U956.
- new net NET.PLA0.M8CYC4: U960.
- new net NET.PLA0.M8CYC5: U964.
- new net NET.PLA0.M8CYC6: U968.
- new net NET.PLA0.M8CYC7: U972.
- new net NET.PLA0.~{COL_{0}}: U822. (Φ1), U837.
- new net NET.PLA0.~{COL_{11}}: U928., U950.
- new net NET.PLA0.~{COL_{13}}: U943., U951.
- new net NET.PLA0.~{COL_{14}}: U945., U953.
- new net NET.PLA0.~{COL_{15}}: U997.
- new net NET.PLA0.~{COL_{16}}: U947., U955.
- new net NET.PLA0.~{COL_{17}}: U999.
- new net NET.PLA0.~{COL_{18}}: U957., U959.
- new net NET.PLA0.~{COL_{19}}: U961., U963.
- new net NET.PLA0.~{COL_{1}}: U814. (Φ1), U923.
- new net NET.PLA0.~{COL_{20}}: U1001.
- new net NET.PLA0.~{COL_{21}}: U965., U967.
- new net NET.PLA0.~{COL_{22}}: U1003.
- new net NET.PLA0.~{COL_{23}}: U969., U971.
- new net NET.PLA0.~{COL_{24}}: U981., U985.
- new net NET.PLA0.~{COL_{25}}: U1005.
- new net NET.PLA0.~{COL_{26}}: U983., U987.
- new net NET.PLA0.~{COL_{27}}: U979., U993.
- new net NET.PLA0.~{COL_{28}}: U977., U995.
- new net NET.PLA0.~{COL_{2}}: U812., U841. (Φ1)
- new net NET.PLA0.~{COL_{7}}: U811.
- new net VDD: U145. (~{DOUT}), U792., U793.
- no-connect marks 0 -> 118
Other:
- note added: "0"
- note added: "1"
- note added: "10"
- note added: "11"
- note added: "12"
- note added: "13"
- note added: "14"
- note added: "15"
- note added: "16"
- note added: "17"
- note added: "18"
- note added: "19"
- note added: "2"
- note added: "20"
- note added: "21"
- note added: "22"
- note added: "23"
- note added: "24"
- note added: "25"
- note added: "26"
- note added: "27"
- note added: "28"
- note added: "29"
- note added: "3"
- note added: "4"
- note added: "5"
- note added: "6"
- note added: "7"
- note added: "8"
- note added: "9"
- note added: "EXT"
- note added: "M16CYC10"
- note added: "M16CYC11"
- note added: "M16CYC8"
- note added: "M16CYC9"
- note added: "M8CYC0"
- note added: "M8CYC1"
- note added: "M8CYC2"
- note added: "M8CYC3"
- note added: "M8CYC4"
- note added: "M8CYC5"
- note added: "M8CYC6"
- note added: "M8CYC7"
- note added: "PLA0"
- note added: "TXTMODE && 1XXX"
- note added: "carry chain is inverted on the actual chip counter cell's LOAD circuit works with the external NOR2/AOI21 gates(see NOTE6)"
- note added: "dynamic latches"
