File: resources/V9958_kicad/CI.kicad_sch (KiCad schematic)
At the start: 187 parts, among them U100 GA042, U101 GA043, U102 DLPEN, U103 DLPEN, U104 GA044, U105 GA045, U106 GA047, U106 GA115, U107 GA046, U108 INV, U109 GA048, U110 GA049, U111 INV, U112 GA051, U113 GA050, U114 GA052, U115 GA053, U116 GA054, U117 GA055, U118 GA056, U119 DLPRPEN, U119 GA057, U120 DLPRPEN, U120 GA058, U121 DLPRPEN, U121 GA059, U122 DLPRPEN, U122 INV, U123 DLPRPEN, U123 INV, U133 DLPRPEN, U134 DLPRPEN, U138 GA122, U138 INV, U139 GA070, U14 GA001, U140 DSR, U140 GA073, U141 GA074, U142 GA071, U143 GA072, U143 GA124, U15 DSR, U162 NAND2OD, U163 NAND2OD, U166 DLPEN, U166 NAND2OD, U167 INV, U167 NAND2OD, U168 DLPEN, U168 NAND2OD, U169 GA085, U169 NAND2OD, U170 DLPEN, U171 DLPEN, U174 DLPEN, U175 DLPEN, U176 DLPEN, U177 DLPEN, U182 GA084, U183 INV, U184 GA086, U185 GA087, U186 GA088, U187 GA097, U190 GA095, U190 GA100, U218 NMOS, U219 NMOS, U220 NMOS, U221 NMOS, U222 COMPBUF, U223 NMOS, U224 NMOS, U225 COMPBUF, U226 NMOS, U227 NMOS, U228 NMOS, U229 NMOS, U230 NMOS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

Commit message: update 20240913
Parts:
- added U350: NAND2OD, symbol Raki_ASIC_cells:NAND2OD
- added U351: INVOD, symbol Raki_ASIC_cells:INVOD
- added U373: GA125, symbol Raki_ASIC_cells:NOR2
Connections:
- net NET.REG_d45_b6_MXC_OE: now also U350.
- net at U90.: now also U140. (Φ2); no longer U143.
- net at U190.: now also U190., U254.; no longer U99.
- net at U92.: now also U94., U96.; no longer U93. (Φ1)
- net at U91.: no longer U92.
- net at U92.: now also U99.; no longer U86. (Φ2)
- net at U71.: no longer U72.
- net at U97.: now also U99.; no longer U86. (Φ2)
- net at U232.: now also U226., U228., U230.; no longer U269.
- net at U245., U249.: now also U237., U241.; no longer U278.
- net at U80.: now also U101. (Φ2), U83.
- net at U81.: now also U138., U82., U86. (Φ2), U91., U94.; no longer U80.
- net at U83.: now also U85. (Φ2); no longer U84. (Φ2)
- net at U82.: now also U97.; no longer U88.
- net at U97.: now also U89. (Φ2); no longer U82.
- net at U138.: now also U90., U97.; no longer U99.
- net at U99.: now also U86. (Φ2), U89. (Φ2), U97., U97.
- net at U142.: now also U143.
- net at U94.: now also U96.
- net at U139.: now also U138.; no longer U140. (Φ2)
- new net: U143., U90. (x2)
- new net: U139., U141. (Φ2), U142.
- new net: U187., U220., U224., U230., U231., U242., U243., U244., U245.
- new net: U236., U240., U244., U248.
- new net: U244., U248., U276.
- new net: U109., U110.
- new net: U109., U110., U111., U119.
- new net: U109., U112., U113.
- new net: U220., U222., U265.
- new net: U218., U219., U220., U222.
- new net: U190., U99.
- new net: U89. (Φ2), U91., U92.
- new net: U92., U93. (Φ1)
- new net: U91., U92.
- new net: U86. (Φ2), U92. (x2)
- new net: U86. (Φ2), U86. (Φ2)
- new net: U71., U72., U76.
- new net: U71., U72.
- new net: U190., U264., U267., U269., U271., U273., U275., U277., U279.
- new net: U86. (Φ2), U97.
- new net: U54. (Φ1), U55.
- new net: U183., U184., U185., U186.
- new net: U167., U184., U186.
- new net: U110., U112., U113.
- new net: U169., U177. (~{Q})
- new net: U232., U269.
- new net: U60., U62., U63.
- new net: U61., U62., U63.
- new net: U121., U123.
- new net: U54. (Φ1), U56. (Φ1)
- new net: U95. (Φ2), U95. (Φ2)
- new net: U242., U246., U272.
- new net: U120., U122.
- new net: U245., U249., U278.
- new net: U52., U53. (Φ2)
- new net: U163., U171. (~{Q})
- new net: U224., U225., U266.
- new net: U221., U223., U224., U225.
- new net: U169., U182., U183.
- new net: U80., U81., U84. (Φ2)
- new net: U80., U81.
- new net: U190., U218., U221., U226., U227., U234., U235., U236., U237.
- new net: U234., U238., U242., U246.
- new net: U83., U84. (Φ2)
- new net: U86. (Φ2), U92., U97.
- new net: U104., U106., U107.
- new net: U105., U106., U107.
- new net: U82., U89. (Φ2), U90.
- new net: U59., U60., U61.
- new net: U14., U60., U61.
- new net: U102. (~{Q}), U115., U116., U119.
- new net: U103. (~{Q}), U114., U116., U118.
- new net: U235., U239., U243., U247.
- new net: U14., U59.
- new net: U243., U247., U274.
- new net: U187., U219., U223., U228., U229., U238., U239., U240., U241., U251.
- new net: U249., U279.
- new net: U56. (Φ1), U57. (Φ2)
- new net: U70. (Φ2), U71.
- new net: U169., U182.
- new net: U95. (Φ2), U99.
- new net: U95. (Φ2), U98. (~{RST})
- new net: U82., U88.
- new net: U138., U99.
- new net: U104., U105., U108., U118.
- new net: U104., U105.
- new net: U102. (~{Q}), U114., U117., U118.
- new net: U103. (~{Q}), U115., U117., U119.
- new net: U100., U98. (~{RST})
- new net: U227., U229., U231., U233.
- new net: U57. (Φ2), U58.
- new net: U230., U232., U268.
- new net: U77., U78., U79. (Φ1)
- new net: U166., U174. (~{Q})
- new net: U73., U75.
- new net: U162., U170. (~{Q})
- new net: U68., U69.
- new net: U231., U233., U270.
- new net: U168., U176. (~{Q})
- new net: U83., U86. (Φ2)
- new net: U167., U175. (~{Q})
- new net: U83., U87.
- new net: U66., U67.
- new net: U106., U58.
- new net: U140. (Φ2), U142., U143.
- new net: U97., U98. (~{RST})
- new net: TP001.1, U83., U85. (Φ2), U86. (Φ2), U99.
- new net: U351., U373.
- new net: U15. (Φ2), U52.
- new net: U139., U140. (Φ2)
- new net: U106., U348.
- new net BUS.REG_d45_b6_MXC: U350., U351.
- now unconnected: U71., U71., U78., U91., U91.
Changed lines of the file:
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@@
     (stroke (width 0) (type default))
   )
+  (wire (pts (xy 703.58 425.45) (xy 730.25 425.45))
+    (stroke (width 0) (type default))
+  )
   (wire (pts (xy 504.19 71.12) (xy 506.73 71.12))
     (stroke (width 0) (type default))
@@
     (stroke (width 0) (type default))
   )
+  (wire (pts (xy 694.69 426.72) (xy 668.02 426.72))
+    (stroke (width 0) (type default))
+  )
   (wire (pts (xy 401.32 128.27) (xy 403.86 128.27))
     (stroke (width 0) (type default))
@@
     (stroke (width 0) (type default))
   )
+  (wire (pts (xy 703.58 435.61) (xy 730.25 435.61))
+    (stroke (width 0) (type default))
+  )
   (wire (pts (xy 680.72 303.53) (xy 681.99 303.53))
     (stroke (width 0) (type default))
@@
     (effects (font (size 1.27 1.27)) (justify left bottom))
   )
+  (label "BUS.REG_d45_b6_MXC" (at 730.25 435.61 180) (fields_autoplaced)
+    (effects (font (size 1.27 1.27)) (justify right bottom))
+  )
   (label "PAD.CD4.IN" (at 384.81 135.89 0) (fields_autoplaced)
     (effects (font (size 1.27 1.27)) (justify left bottom))
@@
     (effects (font (size 1.27 1.27)) (justify left bottom))
   )
+  (label "BUS.REG_d45_b6_MXC" (at 730.25 425.45 180) (fields_autoplaced)
+    (effects (font (size 1.27 1.27)) (justify right bottom))
+  )
   (label "BUS.FIRST_DATA.D_{5}" (at 450.85 115.57 180) (fields_autoplaced)
     (effects (font (size 1.27 1.27)) (justify right bottom))
@@
     (effects (font (size 1.27 1.27)) (justify right bottom))
   )
+  (label "NET.REG_d45_b6_MXC_OE" (at 668.02 426.72 0) (fields_autoplaced)
+    (effects (font (size 1.27 1.27)) (justify left bottom))
+  )
   (label "BUS.VRAM01X_OUTBUF.D_{5}" (at 161.29 281.94 180) (fields_autoplaced)
     (effects (font (size 1.27 1.27)) (justify right bottom))
@@
     )
   )
+  (symbol (lib_id "Raki_ASIC_cells:NAND2OD") (at 698.5 425.45 0) (unit 1)
+    (in_bom yes) (on_board yes) (dnp no) (fields_autoplaced)
+    (property "Reference" "U350" (at 698.5 419.1 0)
+      (effects (font (size 1.27 1.27)) hide)
+    )
+    (property "Value" "NAND2OD" (at 699.135 420.37 0)
+      (effects (font (size 1.27 1.27)))
+    )
+    (property "Footprint" "" (at 698.5 425.45 0)
+      (effects (font (size 1.27 1.27)) hide)
+    )
+    (property "Datasheet" "" (at 698.5 425.45 0)
+      (effects (font (size 1.27 1.27)) hide)
+    )
+    (pin "")
+    (pin "")
+    (pin "")
+    (instances
+      (project "V9958"
+        (path "/b5e1370a-fef4-4131-9314-bdfc21cb5e0f/fe6f0a80-9631-4d2e-8fef-202ec26c9197"
+          (reference "U350") (unit 1)
+        )
+      )
+    )
+  )
   (symbol (lib_id "Raki_ASIC_cells:VY_DDL_small") (at 494.03 344.17 0) (unit 1)
     (in_bom yes) (on_board yes) (dnp no)
@@
     )
   )
+  (symbol (lib_id "Raki_ASIC_cells:NOR2") (at 689.61 435.61 0) (unit 1)
+    (in_bom yes) (on_board yes) (dnp no) (fields_autoplaced)
+    (property "Reference" "U373" (at 689.61 427.99 0)
+      (effects (font (size 1.27 1.27)) hide)
+    )
+    (property "Value" "GA125" (at 690.245 430.53 0)
+      (effects (font (size 1.27 1.27)))
+    )
+    (property "Footprint" "" (at 689.61 427.99 0)
+      (effects (font (size 1.27 1.27)) hide)
+    )
+    (property "Datasheet" "" (at 689.61 427.99 0)
+      (effects (font (size 1.27 1.27)) hide)
+    )
+    (pin "")
+    (pin "")
+    (pin "")
+    (instances
+      (project "V9958"
+        (path "/b5e1370a-fef4-4131-9314-bdfc21cb5e0f/fe6f0a80-9631-4d2e-8fef-202ec26c9197"
+          (reference "U373") (unit 1)
+        )
+      )
+    )
+  )
   (symbol (lib_id "Raki_ASIC_cells:NMOS") (at 90.17 351.79 90) (unit 1)
     (in_bom yes) (on_board yes) (dnp no)
@@
         )
       )
+    )
+  )
+  (symbol (lib_id "Raki_ASIC_cells:INVOD") (at 698.5 435.61 0) (unit 1)
+    (in_bom yes) (on_board yes) (dnp no) (fields_autoplaced)
+    (property "Reference" "U351" (at 698.5 429.26 0)
+      (effects (font (size 1.27 1.27)) hide)
+    )
+    (property "Value" "INVOD" (at 699.135 430.53 0)
+      (effects (font (size 1.27 1.27)))
+    )
+    (property "Footprint" "" (at 697.992 435.61 0)
+      (effects (font (size 1.27 1.27)) hide)
+    )
+    (property "Datasheet" "" (at 697.992 435.61 0)
+      (effects (font (size 1.27 1.27)) hide)
+    )
+    (pin "")
+    (pin "")
+    (instances
+      (project "V9958"
+        (path "/b5e1370a-fef4-4131-9314-bdfc21cb5e0f/fe6f0a80-9631-4d2e-8fef-202ec26c9197"
+          (reference "U351") (unit 1)
+        )
+      )

Commit message: update 20240921
Connections:
- net at U90.: now also U140. (Φ2); no longer U143.
- net at U190.: now also U190., U254.; no longer U99.
- net at U92.: now also U94., U96.; no longer U93. (Φ1)
- net at U91.: no longer U92.
- net at U92.: now also U99.; no longer U86. (Φ2)
- net at U71.: no longer U72.
- net at U97.: now also U99.; no longer U86. (Φ2)
- net at U232.: now also U226., U228., U230.; no longer U269.
- net at U245., U249.: now also U237., U241.; no longer U278.
- net at U80.: now also U101. (Φ2), U83.
- net at U81.: now also U138., U82., U86. (Φ2), U91., U94.; no longer U80.
- net at U83.: now also U85. (Φ2); no longer U84. (Φ2)
- net at U82.: now also U97.; no longer U88.
- net at U97.: now also U89. (Φ2); no longer U82.
- net at U138.: now also U90., U97.; no longer U99.
- net at U99.: now also U86. (Φ2), U89. (Φ2), U97., U97.
- net at U142.: now also U143.
- net at U373.: now also U351.
- net BUS.REG_VRAMX_SEL: now reaches U351.
- net BUS.REG_VRAMX_SEL: now also U350.; no longer U373.
- net at U94.: now also U96.
- net at U139.: now also U138.; no longer U140. (Φ2)
- removed net BUS.REG_d45_b6_MXC: U350., U351.
- new net: U143., U90. (x2)
- new net: U139., U141. (Φ2), U142.
- new net: U187., U220., U224., U230., U231., U242., U243., U244., U245.
- new net: U236., U240., U244., U248.
- new net: U244., U248., U276.
- new net: U109., U110.
- new net: U109., U110., U111., U119.
- new net: U109., U112., U113.
- new net: U220., U222., U265.
- new net: U218., U219., U220., U222.
- new net: U190., U99.
- new net: U89. (Φ2), U91., U92.
- new net: U92., U93. (Φ1)
- new net: U91., U92.
- new net: U86. (Φ2), U92. (x2)
- new net: U86. (Φ2), U86. (Φ2)
- new net: U71., U72., U76.
- new net: U71., U72.
- new net: U190., U264., U267., U269., U271., U273., U275., U277., U279.
- new net: U86. (Φ2), U97.
- new net: U54. (Φ1), U55.
- new net: U183., U184., U185., U186.
- new net: U167., U184., U186.
- new net: U110., U112., U113.
- new net: U169., U177. (~{Q})
- new net: U232., U269.
- new net: U60., U62., U63.
- new net: U61., U62., U63.
- new net: U121., U123.
- new net: U54. (Φ1), U56. (Φ1)
- new net: U95. (Φ2), U95. (Φ2)
- new net: U242., U246., U272.
- new net: U120., U122.
- new net: U245., U249., U278.
- new net: U52., U53. (Φ2)
- new net: U163., U171. (~{Q})
- new net: U224., U225., U266.
- new net: U221., U223., U224., U225.
- new net: U169., U182., U183.
- new net: U80., U81., U84. (Φ2)
- new net: U80., U81.
- new net: U190., U218., U221., U226., U227., U234., U235., U236., U237.
- new net: U234., U238., U242., U246.
- new net: U83., U84. (Φ2)
- new net: U86. (Φ2), U92., U97.
- new net: U104., U106., U107.
- new net: U105., U106., U107.
- new net: U82., U89. (Φ2), U90.
- new net: U59., U60., U61.
- new net: U14., U60., U61.
- new net: U102. (~{Q}), U115., U116., U119.
- new net: U103. (~{Q}), U114., U116., U118.
- new net: U235., U239., U243., U247.
- new net: U14., U59.
- new net: U243., U247., U274.
- new net: U187., U219., U223., U228., U229., U238., U239., U240., U241., U251.
- new net: U249., U279.
- new net: U56. (Φ1), U57. (Φ2)
- new net: U70. (Φ2), U71.
- new net: U169., U182.
- new net: U95. (Φ2), U99.
- new net: U95. (Φ2), U98. (~{RST})
- new net: U82., U88.
- new net: U138., U99.
- new net: U104., U105., U108., U118.
- new net: U104., U105.
- new net: U102. (~{Q}), U114., U117., U118.
- new net: U103. (~{Q}), U115., U117., U119.
- new net: U100., U98. (~{RST})
- new net: U227., U229., U231., U233.
- new net: U57. (Φ2), U58.
- new net: U230., U232., U268.
- new net: U77., U78., U79. (Φ1)
- new net: U166., U174. (~{Q})
- new net: U73., U75.
- new net: U162., U170. (~{Q})
- new net: U68., U69.
- new net: U231., U233., U270.
- new net: U168., U176. (~{Q})
- new net: U83., U86. (Φ2)
- new net: U167., U175. (~{Q})
- new net: U83., U87.
- new net: U66., U67.
- new net: U106., U58.
- new net: U140. (Φ2), U142., U143.
- new net: U97., U98. (~{RST})
- new net: TP001.1, U83., U85. (Φ2), U86. (Φ2), U99.
- new net: U15. (Φ2), U52.
- new net: U139., U140. (Φ2)
- new net: U106., U348.
- now unconnected: U71., U71., U78., U91., U91.
Changed lines of the file:
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@@
     (effects (font (size 1.27 1.27)) (justify left bottom))
   )
-  (label "BUS.REG_d45_b6_MXC" (at 730.25 435.61 180) (fields_autoplaced)
+  (label "BUS.REG_VRAMX_SEL" (at 730.25 435.61 180) (fields_autoplaced)
     (effects (font (size 1.27 1.27)) (justify right bottom))
   )
@@
     (effects (font (size 1.27 1.27)) (justify left bottom))
   )
-  (label "BUS.REG_d45_b6_MXC" (at 730.25 425.45 180) (fields_autoplaced)
+  (label "BUS.REG_VRAMX_SEL" (at 730.25 425.45 180) (fields_autoplaced)
     (effects (font (size 1.27 1.27)) (justify right bottom))
   )

Commit message: update 20241020
Connections:
- net at U90.: now also U140. (Φ2); no longer U143.
- net at U190.: now also U190., U254.; no longer U99.
- net at U92.: now also U94., U96.; no longer U93. (Φ1)
- net at U91.: no longer U92.
- net at U92.: now also U99.; no longer U86. (Φ2)
- net at U71.: no longer U72.
- net at U97.: now also U99.; no longer U86. (Φ2)
- net at U232.: now also U226., U228., U230.; no longer U269.
- net at U245., U249.: now also U237., U241.; no longer U278.
- net at U80.: now also U101. (Φ2), U83.
- net at U81.: now also U138., U82., U86. (Φ2), U91., U94.; no longer U80.
- net at U83.: now also U85. (Φ2); no longer U84. (Φ2)
- net at U82.: now also U97.; no longer U88.
- net at U97.: now also U89. (Φ2); no longer U82.
- net at U138.: now also U90., U97.; no longer U99.
- net at U99.: now also U86. (Φ2), U89. (Φ2), U97., U97.
- net at U142.: now also U143.
- net at U373.: now also U351.
- net at U94.: now also U96.
- net at U139.: now also U138.; no longer U140. (Φ2)
- new net: U143., U90. (x2)
- new net: U139., U141. (Φ2), U142.
- new net: U187., U220., U224., U230., U231., U242., U243., U244., U245.
- new net: U236., U240., U244., U248.
- new net: U244., U248., U276.
- new net: U109., U110.
- new net: U109., U110., U111., U119.
- new net: U109., U112., U113.
- new net: U220., U222., U265.
- new net: U218., U219., U220., U222.
- new net: U190., U99.
- new net: U89. (Φ2), U91., U92.
- new net: U92., U93. (Φ1)
- new net: U91., U92.
- new net: U86. (Φ2), U92. (x2)
- new net: U86. (Φ2), U86. (Φ2)
- new net: U71., U72., U76.
- new net: U71., U72.
- new net: U190., U264., U267., U269., U271., U273., U275., U277., U279.
- new net: U86. (Φ2), U97.
- new net: U54. (Φ1), U55.
- new net: U183., U184., U185., U186.
- new net: U167., U184., U186.
- new net: U110., U112., U113.
- new net: U169., U177. (~{Q})
- new net: U232., U269.
- new net: U60., U62., U63.
- new net: U61., U62., U63.
- new net: U121., U123.
- new net: U54. (Φ1), U56. (Φ1)
- new net: U95. (Φ2), U95. (Φ2)
- new net: U242., U246., U272.
- new net: U120., U122.
- new net: U245., U249., U278.
- new net: U52., U53. (Φ2)
- new net: U163., U171. (~{Q})
- new net: U224., U225., U266.
- new net: U221., U223., U224., U225.
- new net: U169., U182., U183.
- new net: U80., U81., U84. (Φ2)
- new net: U80., U81.
- new net: U190., U218., U221., U226., U227., U234., U235., U236., U237.
- new net: U234., U238., U242., U246.
- new net: U83., U84. (Φ2)
- new net: U86. (Φ2), U92., U97.
- new net: U104., U106., U107.
- new net: U105., U106., U107.
- new net: U82., U89. (Φ2), U90.
- new net: U59., U60., U61.
- new net: U14., U60., U61.
- new net: U102. (~{Q}), U115., U116., U119.
- new net: U103. (~{Q}), U114., U116., U118.
- new net: U235., U239., U243., U247.
- new net: U14., U59.
- new net: U243., U247., U274.
- new net: U187., U219., U223., U228., U229., U238., U239., U240., U241., U251.
- new net: U249., U279.
- new net: U56. (Φ1), U57. (Φ2)
- new net: U70. (Φ2), U71.
- new net: U169., U182.
- new net: U95. (Φ2), U99.
- new net: U95. (Φ2), U98. (~{RST})
- new net: U82., U88.
- new net: U138., U99.
- new net: U104., U105., U108., U118.
- new net: U104., U105.
- new net: U102. (~{Q}), U114., U117., U118.
- new net: U103. (~{Q}), U115., U117., U119.
- new net: U100., U98. (~{RST})
- new net: U227., U229., U231., U233.
- new net: U57. (Φ2), U58.
- new net: U230., U232., U268.
- new net: U77., U78., U79. (Φ1)
- new net: U166., U174. (~{Q})
- new net: U73., U75.
- new net: U162., U170. (~{Q})
- new net: U68., U69.
- new net: U231., U233., U270.
- new net: U168., U176. (~{Q})
- new net: U83., U86. (Φ2)
- new net: U167., U175. (~{Q})
- new net: U83., U87.
- new net: U66., U67.
- new net: U106., U58.
- new net: U140. (Φ2), U142., U143.
- new net: U97., U98. (~{RST})
- new net: TP001.1, U83., U85. (Φ2), U86. (Φ2), U99.
- new net: U15. (Φ2), U52.
- new net: U139., U140. (Φ2)
- new net: U106., U348.
- now unconnected: U71., U71., U78., U91., U91.

Commit message: update 20250809
HVCNTR
Parts:
- renumbered U140 to U100, U142 to U101, U103 to U102, U109 to U103, U110 to U105, U105 to U106, U111 to U107, U114 to U109, U115 to U110, U116 to U111, U117 to U112, U118 to U113, U119 to U114, U121 to U115, U123 to U116, U95 to U117, U329 to U118, U143 to U124, U90 to U125, U143 to U126, U90 to U127, U140 to U129, U120 to U135, U166 to U136, U15 to U14, U168 to U144, U170 to U145, U171 to U146, U174 to U147, U175 to U148, U176 to U149, U52 to U15, U177 to U150, U122 to U151, U162 to U152, U163 to U153, U166 to U162, U167 to U163, U168 to U166, U169 to U167, U169 to U168, U182 to U169, U167 to U178, U183 to U179, U185 to U181, U184 to U182, U186 to U184, U75 to U185, U73 to U186, U139 to U216, U254 to U218, U99 to U219, U251 to U220, U190 to U221, U190 to U222, U187 to U223, U218 to U224, U221 to U225, U234 to U228, U235 to U229, U236 to U230, U237 to U231, U219 to U232, U223 to U233, U228 to U234, U229 to U235, U238 to U236, U239 to U237, U240 to U238, U241 to U239, U220 to U240, U224 to U241, U230 to U242, U231 to U243, U242 to U244, U243 to U245, U244 to U246, U245 to U247, U222 to U248, U225 to U249, U232 to U250, U233 to U251, U246 to U252, U247 to U253, U248 to U254, U249 to U264, U264 to U266, U266 to U267, U267 to U268, U268 to U269, U269 to U270, U270 to U271, U271 to U272, U272 to U273, U273 to U274, U274 to U275, U275 to U276, U276 to U277, U277 to U278, U278 to U279, U279 to U280, U141 to U307, U74 to U329, U99 to U33, U100 to U34, U106 to U347, U58 to U349, U86 to U355, U99 to U356, U97 to U357, U86 to U358, U92 to U359, U86 to U360, U86 to U361, U86 to U362, U85 to U363, U99 to U364, U95 to U365, U87 to U366, U95 to U367, U83 to U368, U80 to U369, U81 to U370, U84 to U371, U101 to U372, U53 to U52, U63 to U53, U62 to U54, U95 to U55, U67 to U56, U69 to U57, U54 to U58, U66 to U59, U68 to U60, U60 to U61, U61 to U62, U98 to U63, U56 to U64, U64 to U65, U65 to U66, U57 to U67, U94 to U68, U96 to U69, U97 to U70, U14 to U71, U93 to U72, U70 to U73, U92 to U74, U59 to U75, U58 to U76, U55 to U77, U91 to U78, U71 to U79, U112 to U80, U72 to U81, U89 to U82, U113 to U83, U106 to U84, U107 to U85, U88 to U86, U76 to U87, U102 to U88, U77 to U89, U82 to U91, U78 to U92, U138 to U93, U79 to U94, U89 to U95, U97 to U96, U138 to U97, U97 to U98
Connections:
- net at U125.: now also U100. (Φ2); no longer U126.
- net at U222.: now also U218., U221.; no longer U219.
- net at U74.: now also U68., U69.; no longer U72. (Φ1)
- net at U78.: no longer U74.
- net NET.GT107: now reaches U359.
- net NET.GT107: now also U356.; no longer U360. (Φ2)
- net at U79.: no longer U81.
- net at U357.: now also U356.; no longer U358. (Φ2)
- net at U250.: now also U226., U234., U242.; no longer U270.
- net at U247., U264.: now also U231., U239.; no longer U279.
- net at U369.: now also U368., U372. (Φ2)
- net at U370.: now also U362. (Φ2), U68., U78., U91., U93.; no longer U369.
- net at U368.: now also U363. (Φ2); no longer U371. (Φ2)
- net at U91.: now also U96.; no longer U86.
- net NET.GT108: now reaches U96.
- net NET.GT108: now also U355. (Φ2), U95. (Φ2), U98., U99.; no longer U91.
- net at U97.: now also U90., U98.; no longer U99.
- net at U101.: now also U124.
- net at U373.: now also U351.
- net at U68.: now also U69.
- net at U216.: now also U93.; no longer U129. (Φ2)
- new net: U125., U126.
- new net: U101., U216., U307. (Φ2)
- new net: U223., U240., U241., U242., U243., U244., U245., U246., U247.
- new net: U230., U238., U246., U254.
- new net: U246., U254., U277.
- new net: U103., U105.
- new net: U103., U105., U107., U114.
- new net: U103., U80., U83.
- new net: U240., U248., U265.
- new net: U224., U232., U240., U248.
- new net: U219., U222.
- new net: U74., U78., U82. (Φ2)
- new net: U72. (Φ1), U74.
- new net: U74., U78.
- new net: U359., U360. (Φ2)
- new net: U360. (Φ2), U361. (Φ2)
- new net: U79., U81., U87.
- new net: U79., U81.
- new net: U221., U266., U268., U270., U272., U274., U276., U278., U280.
- new net: U358. (Φ2), U359.
- new net: U357., U358. (Φ2)
- new net: U58. (Φ1), U77.
- new net: U179., U181., U182., U184.
- new net: U178., U182., U184.
- new net: U105., U80., U83.
- new net: U150. (~{Q}), U167.
- new net: U250., U270.
- new net: U53., U54., U61.
- new net: U53., U54., U62.
- new net: U115., U116.
- new net: U58. (Φ1), U64. (Φ1)
- new net: U365. (Φ2), U367. (Φ2)
- new net: U244., U252., U273.
- new net: U135., U151.
- new net: U247., U264., U279.
- new net: U15., U52. (Φ2)
- new net: U146. (~{Q}), U153.
- new net: U241., U249., U267.
- new net: U225., U233., U241., U249.
- new net: U168., U169., U179.
- new net: U369., U370., U371. (Φ2)
- new net: U369., U370.
- new net: U222., U224., U225., U226., U227., U228., U229., U230., U231.
- new net: U228., U236., U244., U252.
- new net: U368., U371. (Φ2)
- new net: U355. (Φ2), U357., U359.
- new net: U126., U127.
- new net: U104., U84., U85.
- new net: U106., U84., U85.
- new net: U82. (Φ2), U90., U91.
- new net: U61., U62., U75.
- new net: U61., U62., U71.
- new net: U110., U111., U114., U88. (~{Q})
- new net: U102. (~{Q}), U109., U111., U113.
- new net: U229., U237., U245., U253.
- new net: U71., U75.
- new net: U245., U253., U275.
- new net: U220., U223., U232., U233., U234., U235., U236., U237., U238., U239.
- new net: U264., U280.
- new net: U64. (Φ1), U67. (Φ2)
- new net: U73. (Φ2), U79.
- new net: U168., U169.
- new net: U33., U55. (Φ2)
- new net: U55. (Φ2), U63. (~{RST})
- new net: U86., U91.
- new net: U97., U99.
- new net: U104., U106., U108., U113.
- new net: U104., U106.
- new net: U109., U112., U113., U88. (~{Q})
- new net: U102. (~{Q}), U110., U112., U114.
- new net: U34., U63. (~{RST})
- new net: U227., U235., U243., U251.
- new net: U67. (Φ2), U76.
- new net: U242., U250., U269.
- new net: U89., U92., U94. (Φ1)
- new net: U147. (~{Q}), U162.
- new net: U185., U186.
- new net: U145. (~{Q}), U152.
- new net: U57., U60.
- new net: U243., U251., U271.
- new net: U149. (~{Q}), U166.
- new net: U361. (Φ2), U368.
- new net: U95. (Φ2), U96.
- new net: U148. (~{Q}), U163.
- new net: U366., U368.
- new net: U56., U59.
- new net: U347., U349.
- new net: U101., U124., U129. (Φ2)
- new net: U63. (~{RST}), U70.
- new net: TP001.1, U362. (Φ2), U363. (Φ2), U364., U368.
- new net: U14. (Φ2), U15.
- new net: U129. (Φ2), U216.
- new net: U347., U348.
- new net: U100. (Φ2), U98.
- now unconnected: U78., U78., U79., U79., U92.
