File: resources/V9958_kicad/CI.kicad_sch (KiCad schematic)
At the start: 190 parts, among them U100 DSR, U101 GA071, U102 DLPEN, U103 GA048, U104 GA044, U105 GA049, U106 GA045, U107 INV, U108 INV, U109 GA052, U110 GA053, U111 GA054, U112 GA055, U113 GA056, U114 GA057, U115 GA059, U116 INV, U117 GB001, U118 DLPRPEN, U119 DLPRPEN, U120 DLPRPEN, U121 DLPRPEN, U122 DLPRPEN, U123 DLPRPEN, U124 GA072, U125 INVP, U126 GA124, U127 INVP, U129 GA073, U133 DLPRPEN, U134 DLPRPEN, U135 GA058, U136 DLPEN, U14 DSR, U144 DLPEN, U145 DLPEN, U146 DLPEN, U147 DLPEN, U148 DLPEN, U149 DLPEN, U15 NOR2, U150 DLPEN, U151 INV, U152 NAND2OD, U153 NAND2OD, U162 NAND2OD, U163 NAND2OD, U166 NAND2OD, U167 NAND2OD, U168 GA085, U169 GA084, U178 INV, U179 INV, U181 GA087, U182 GA086, U184 GA088, U185 INV, U186 GA022, U216 GA070, U218 GA092, U219 GA099, U220 GA096, U221 GA100, U222 GA095, U223 GA097, U224 NMOS, U225 NMOS, U226 NMOS, U227 NMOS, U228 NMOS, U229 NMOS, U230 NMOS, U231 NMOS, U232 NMOS, U233 NMOS, U234 NMOS, U235 NMOS, U236 NMOS, U237 NMOS, U238 NMOS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

Commit message: update 20251106
Parts:
- removed U228, U233, U237, U242, U246: NMOS, symbol Raki_ASIC_cells:NMOS
- removed U248, U249, U250, U251, U252, U253, U254, U264: COMPBUF, symbol Raki_ASIC_cells:COMPBUF
- added U1703, U228, U233, U237, U242, U246, U250, U254: BUFC, symbol Raki_ASIC_cells:BUFC
- added U248, U249, U251, U252, U253: NMOS, symbol Raki_ASIC_cells:NMOS
Connections:
- net BUS.VRAM01X_INBUF.D_{0}: now also U251.; no longer U231.
- net BUS.VRAM01X_INBUF.D_{1}: now also U247.; no longer U230.
- net BUS.VRAM01X_INBUF.D_{2}: now also U243.; no longer U229.
- net BUS.VRAM01X_INBUF.D_{3}: now also U238.
- net BUS.VRAM01X_INBUF.D_{4}: now also U234.; no longer U227.
- net BUS.VRAM01X_INBUF.D_{5}: now also U229.; no longer U226.
- net PAD.CD0.IN: now also U252.; no longer U239.
- net PAD.CD1.IN: now also U248.; no longer U238.
- net PAD.CD2.IN: now also U244.
- net PAD.CD3.IN: now also U239.; no longer U236.
- net PAD.CD5.IN: now also U230.; no longer U234.
- net PAD.CD6.IN: now also U226.
- net at U125.: now also U100. (Φ2); no longer U126.
- net at U240.: now also U224., U232., U1703.; no longer U265.
- net at U222.: now also U218., U221.; no longer U219.
- net at U74.: now also U68., U69.; no longer U72. (Φ1)
- net GBL.phiL_RST: now reaches U78.
- net GBL.phiL_RST: now also U101., U103., U104., U117. (Φ2), U168., U369., U53., U68., U79., U83., U85.; no longer U74.
- net at U357.: now also U356.; no longer U358. (Φ2)
- net at U241.: now also U238., U239., U242.; no longer U267.
- net at U370.: now also U362. (Φ2), U68., U78., U91., U93.; no longer U369.
- net at U236.: now also U271., U237.; no longer U244.
- net at U368.: now also U363. (Φ2); no longer U371. (Φ2)
- net at U245.: now also U243., U244., U246.; no longer U229.
- net at U91.: now also U96.; no longer U86.
- net at U97.: now also U90., U98.; no longer U99.
- net at U373.: now also U351.
- net at U216.: now also U93.; no longer U129. (Φ2)
- new net: U125., U126.
- new net: U101., U216., U307. (Φ2)
- new net: U103., U105.
- new net: U103., U105., U107., U114.
- new net: U103., U80., U83.
- new net: U219., U222.
- new net: U74., U78., U82. (Φ2)
- new net: U72. (Φ1), U74.
- new net: U74., U78.
- new net: U359., U360. (Φ2)
- new net: U360. (Φ2), U361. (Φ2)
- new net: U79., U81., U87.
- new net: U79., U81.
- new net: U221., U266., U268., U270., U272., U274., U276., U278., U280.
- new net: U250., U278.
- new net: U358. (Φ2), U359.
- new net: U357., U358. (Φ2)
- new net: U58. (Φ1), U77.
- new net: U179., U181., U182., U184.
- new net: U178., U182., U184.
- new net: U105., U80., U83.
- new net: U150. (~{Q}), U167.
- new net: U233., U270.
- new net: U53., U54., U61.
- new net: U53., U54., U62.
- new net: U115., U116.
- new net: U58. (Φ1), U64. (Φ1)
- new net: U365. (Φ2), U367. (Φ2)
- new net: U241., U242., U273.
- new net: U247., U248., U249., U250.
- new net: U222., U224., U225., U229., U234., U238., U243., U247., U251.
- new net: U249., U250., U277.
- new net: U135., U151.
- new net: U229., U230., U231., U233.
- new net: U231., U233., U269.
- new net: U253., U254., U279.
- new net: U15., U52. (Φ2)
- new net: U146. (~{Q}), U153.
- new net: U220., U223., U226., U230., U232., U235., U239., U244., U248., U252.
- new net: U251., U252., U253., U254.
- new net: U223., U227., U231., U236., U240., U241., U245., U249., U253.
- new net: U234., U235., U236., U237.
- new net: U168., U169., U179.
- new net: U369., U370., U371. (Φ2)
- new net: U369., U370.
- new net: U368., U369., U372. (Φ2)
- new net: U368., U371. (Φ2)
- new net: U355. (Φ2), U357., U359.
- new net: U126., U127.
- new net: U104., U84., U85.
- new net: U106., U84., U85.
- new net: U1703., U240., U265.
- new net: U82. (Φ2), U90., U91.
- new net: U225., U226., U227., U228.
- new net: U61., U62., U75.
- new net: U61., U62., U71.
- new net: U110., U111., U114., U88. (~{Q})
- new net: U102. (~{Q}), U109., U111., U113.
- new net: U227., U228., U267.
- new net: U71., U75.
- new net: U64. (Φ1), U67. (Φ2)
- new net: U228., U268.
- new net: U73. (Φ2), U79.
- new net: U168., U169.
- new net: U33., U55. (Φ2)
- new net: U55. (Φ2), U63. (~{RST})
- new net: U1703., U266.
- new net: U86., U91.
- new net: U97., U99.
- new net: U104., U106., U108., U113.
- new net: U104., U106.
- new net: U254., U280.
- new net: U109., U112., U113., U88. (~{Q})
- new net: U102. (~{Q}), U110., U112., U114.
- new net: U34., U63. (~{RST})
- new net: U67. (Φ2), U76.
- new net: U89., U92., U94. (Φ1)
- new net: U147. (~{Q}), U162.
- new net: U185., U186.
- new net: U145. (~{Q}), U152.
- new net: U57., U60.
- new net: U242., U274.
- new net: U245., U246., U275.
- new net: U149. (~{Q}), U166.
- new net: U361. (Φ2), U368.
- new net: U237., U272.
- new net: U95. (Φ2), U96.
- new net: U148. (~{Q}), U163.
- new net: U246., U276.
- new net: U366., U368.
- new net: U56., U59.
- new net: U347., U349.
- new net: U101., U124., U129. (Φ2)
- new net: U101., U124.
- new net: U63. (~{RST}), U70.
- new net: TP001.1, U362. (Φ2), U363. (Φ2), U364., U368.
- new net: U14. (Φ2), U15.
- new net: U68., U69.
- new net: U129. (Φ2), U216.
- new net: U347., U348.
- new net: U100. (Φ2), U98.
- now unconnected: U92.
Other:
- note added: "2.5Z"
- note removed: "RST?"
