File: resources/V9958_kicad/MI.kicad_sch (KiCad schematic)
At the start: 453 parts, among them U1 IDRV, U10 ODRV, U11 BUFD, U12 ODRV, U128 GM008, U13 BUFD, U14 ODRV, U15 BUFD, U16 ODRV, U17 BUFD, U18 ODRV, U19 BUFD, U2 IDRV, U20 ODRV, U21 BUFD, U217 GM011, U22 ODRV, U257 GM002, U258 GM003, U259 IDRV, U260 IDRV, U261 IDRV, U262 GM005, U263 GM006, U3 IDRV, U308 GM009, U309 GM010, U346 GM007, U352 DDL, U353 DDL, U354 GM012, U380 DDL, U381 DDL, U382 DDL, U383 DDL, U384 DDL, U385 DDL, U386 DDL, U387 DDL, U388 DDL, U389 DDL, U390 DDL, U391 DDL, U392 DDL, U393 DDL, U394 DDL, U395 DDL, U396 DDL, U397 DDL, U398 DDL, U399 DDL, U4 IDRV, U400 DDL, U401 DDL, U402 DDL, U403 DDL, U404 DDL, U405 DDL, U406 DDL, U407 DDL, U408 DDL, U409 DDL, U410 DDL, U411 DDL, U412 DDL, U413 DDL, U414 DDL, U415 DDL, U416 DDL, U417 DDL, U418 DDL, U419 DDL, U420 DDL, U421 DDL, U422 DDL, U423 DDL, U424 DDL, U425 DDL, U426 DDL, U427 DDL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

Commit message: update 20250809
HVCNTR
Connections:
- net at U626.: now also U625.; no longer U627.
- net at U739.: now also U737.; no longer U9.
- net at U391. (Φ1): no longer U393.
- net at U?.: now also U633., U634.; no longer U636.
- net at U?.: now also U308. (Φ1), U353. (Φ1), U381. (Φ1), U384. (Φ1), U387. (Φ1), U391. (Φ1), U392. (Φ1), U397. (Φ1), U398. (Φ1), U403. (Φ1), U407. (Φ1), U411. (Φ1), U415. (Φ1), U419. (Φ1), U423. (Φ1), U427. (Φ1); no longer U431. (Φ1)
- net at U789.: now also U738.; no longer U788.
- net at U411. (Φ1): now also U410. (Φ1); no longer U412.
- net at U610.: now also U607.; no longer U611.
- net at U609.: now also U607., U608.; no longer U610.
- net at U352. (Φ1): now also U353. (Φ1)
- net at U353. (Φ1): now also U354.; no longer U352. (Φ1)
- net at U787.: now also U21.; no longer U786.
- net at U21.: now also U22.; no longer U787.
- net at U584.: now also U582., U583.; no longer U585.
- net at U763.: now also U15.; no longer U762.
- net at U629.: now also U662. (Φ1); no longer U630. (Φ2)
- net at U308. (Φ1): now also U128. (Φ1)
- net at U644.: now also U643. (Φ1); no longer U642.
- net at U11.: now also U747.; no longer U12.
- net at U747.: now also U746.; no longer U11.
- net at U619.: now also U617., U618.; no longer U620.
- net at U410. (Φ1): no longer U409. (Φ1)
- net at U655.: now also U659. (Φ1), U660. (Φ1); no longer U657. (Φ1)
- net at U670.: now also U668. (S); no longer U674. (Φ1)
- net at U476.: now also U474., U475.; no longer U477.
- net at U620.: now also U618.; no longer U621.
- net at U397. (Φ1): now also U395. (Φ1)
- net at U426. (Φ1): now also U427. (Φ1)
- net at U427. (Φ1): now also U428.; no longer U426. (Φ1)
- net at U414. (Φ1): now also U415. (Φ1); no longer U413. (Φ1)
- net at U625.: now also U624.; no longer U626.
- net at U651.: now also U653. (Φ2); no longer U650. (Φ2)
- net at U771.: now also U17.; no longer U770.
- net at U387. (Φ1): no longer U386. (Φ1)
- net at U422. (Φ1): now also U423. (Φ1)
- net at U423. (Φ1): no longer U422. (Φ1)
- net at U579.: now also U576., U577.; no longer U581. (Φ1)
- net at U642.: now also U647. (Φ1); no longer U641. (Φ1)
- net at U525.: now also U522., U523.; no longer U527. (Φ1)
- net at U418. (Φ1): now also U419. (Φ1)
- net at U419. (Φ1): no longer U418. (Φ1)
- net NET.GT112: now reaches U86. (Φ2)
- net at U?.: now also U437. (Φ1); no longer U436.
- net at U456.: now also U454., U455.; no longer U446. (Φ1)
- net at U681.: now also U680.; no longer U682.
- net at U17.: now also U18.; no longer U771.
- net at U13.: now also U755.; no longer U14.
- net at U624.: now also U622.; no longer U625.
- net at U530.: now also U528., U529.; no longer U531.
- net at U392. (Φ1): now also U390. (Φ1); no longer U394.
- net at U381. (Φ1): now also U382.; no longer U380. (Φ1)
- net at U738.: now also U730.; no longer U789.
- net at U578.: now also U574., U575.; no longer U580. (Φ1)
- net at U697.: now also U696. (Φ1); no longer U702. (Φ2)
- net at U699.: now also U700.; no longer U698. (Φ1)
- net at U685.: now also U684.; no longer U688. (Φ1)
- net at U384. (Φ1): now also U385.; no longer U383. (Φ1)
- net at U671.: now also U673. (Φ1); no longer U668. (S)
- net at U415. (Φ1): no longer U416.
- net at U669.: now also U674. (Φ1); no longer U668. (S)
- net at U402. (Φ1): no longer U401. (Φ1)
- net at U403. (Φ1): now also U402. (Φ1)
- net at U779.: now also U778.; no longer U19.
- net at U407. (Φ1): now also U406. (Φ1)
- net at U406. (Φ1): now also U405. (Φ1); no longer U407. (Φ1)
- net at U?.: now also U439.; no longer U440. (Φ1)
- net NET.GT107: now reaches U675.
- net NET.GT107: no longer U86. (Φ2)
- new net: U626., U627.
- new net: U689. (Φ1), U86. (Φ2)
- new net: U647. (Φ1), U648., U649. (Φ2)
- new net: U648., U649. (Φ2), U650. (Φ2)
- new net: U684., U686., U687.
- new net: U651., U652., U654. (Φ1)
- new net: U654. (Φ1), U655., U656. (Φ1)
- new net: U448., U454., U466., U468., U484., U486., U502., U504., U520., U522., U538., U540., U556., U558., U574., U576., U591., U592.
- new net: U520., U521., U524.
- new net: U518., U520., U557.
- new net: U739., U9.
- new net: U556., U557., U560.
- new net: U262., U263., U?.
- new net: U309., U382., U385., U388., U393., U394., U399., U400., U?.
- new net: U391. (Φ1), U393.
- new net: U676., U86. (Φ2)
- new net: U636., U?.
- new net: U431. (Φ1), U?.
- new net: U430., U431. (Φ1), U?.
- new net: U788., U789.
- new net: U354., U404., U408., U412., U416., U420., U424., U428., U?.
- new net: U411. (Φ1), U412.
- new net: U449., U455., U467., U469., U485., U487., U503., U505., U521., U523., U539., U541., U557., U559., U575., U577., U590., U591., U593.
- new net: U467., U573., U576.
- new net: U466., U467., U470.
- new net: U751. (Φ1), U86. (Φ2)
- new net: U610., U611.
- new net: U609., U610.
- new net: U465., U468., U487.
- new net: U468., U469., U471.
- new net: U614., U615.
- new net: U615., U616. (Φ1)
- new net: U442., U444., U445.
- new net: U445., U446. (Φ1)
- new net: U217. (Φ1), U352. (Φ1)
- new net: U352. (Φ1), U402. (Φ1), U406. (Φ1), U410. (Φ1), U414. (Φ1), U418. (Φ1), U422. (Φ1), U426. (Φ1), U?.
- new net: U486., U487., U489.
- new net: U396. (Φ1), U398. (Φ1)
- new net: U546., U547., U548.
- new net: U398. (Φ1), U400.
- new net: U564., U598. (Φ1)
- new net: U563. (Φ1), U598. (Φ1)
- new net: U743. (Φ1), U745. (Φ1)
- new net: U745. (Φ1), U746.
- new net: U761. (Φ1), U762.
- new net: U759. (Φ1), U761. (Φ1)
- new net: U389. (Φ1), U391. (Φ1)
- new net: U448., U451., U469.
- new net: U786., U787.
- new net: U584., U585.
- new net: U491. (Φ1), U602. (Φ1)
- new net: U447. (Φ1), U604. (Φ1)
- new net: U444., U604. (Φ1)
- new net: U762., U763.
- new net: U760. (Φ1), U762.
- new net: U742. (Φ1), U86. (Φ2)
- new net: U734. (Φ1), U86. (Φ2)
- new net: U629., U630. (Φ2)
- new net: U630. (Φ2), U631. (Φ2), U?.
- new net: U308. (Φ1), U309.
- new net: U642., U644.
- new net: U665. (Φ1), U667. (Φ1), U668. (S), U671.
- new net: U663. (Φ1), U665. (Φ1)
- new net: U665. (Φ1), U673. (Φ1)
- new net: U11., U12.
- new net: U619., U620.
- new net: U638. (Φ1), U86. (Φ2)
- new net: U637. (Φ1), U638. (Φ1)
- new net: U540., U541., U543.
- new net: U537., U540., U559.
- new net: U536., U538., U575.
- new net: U538., U539., U542.
- new net: U661. (Φ1), U662. (Φ1)
- new net: U661. (Φ1), U664. (Φ1)
- new net: U581. (Φ1), U597. (Φ1)
- new net: U582., U597. (Φ1)
- new net: U564., U565., U566.
- new net: U498., U499., U501.
- new net: U453., U458., U461., U463., U479., U481., U497., U499., U515., U517., U533., U535., U551., U553., U569., U571., U586., U588.
- new net: U692., U694. (Φ2), U695. (Φ1)
- new net: U695. (Φ1), U696. (Φ1), U698. (Φ1)
- new net: U483., U486., U505.
- new net: U504., U505., U507.
- new net: U750. (Φ1), U86. (Φ2)
- new net: U750. (Φ1), U752. (Φ1)
- new net: U409. (Φ1), U410. (Φ1)
- new net: U629., U657. (Φ1)
- new net: U655., U657. (Φ1)
- new net: U733. (Φ1), U735. (Φ1)
- new net: U735. (Φ1), U737.
- new net: U697., U699., U86. (Φ2)
- new net: U86. (Φ2), U86. (Φ2) (x2)
- new net: U767. (Φ1), U86. (Φ2)
- new net: U482., U484., U521.
- new net: U452., U457., U460., U462., U478., U480., U496., U498., U514., U516., U532., U534., U550., U552., U568., U570., U586., U587.
- new net: U478., U479., U482.
- new net: U516., U517., U519.
- new net: U462., U463., U465.
- new net: U492., U602. (Φ1)
- new net: U448., U449., U450.
- new net: U451., U452., U453.
- new net: U651., U653. (Φ2), U674. (Φ1)
- new net: U670., U674. (Φ1)
- new net: U476., U477.
- new net: U514., U515., U518.
- new net: U592., U593., U594.
- new net: U782. (Φ1), U86. (Φ2)
- new net: U783. (Φ1), U86. (Φ2)
- new net: U620., U621.
- new net: U759. (Φ1), U86. (Φ2)
- new net: U502., U503., U506.
- new net: U496., U497., U500.
- new net: U473. (Φ1), U603. (Φ1)
- new net: U743. (Φ1), U86. (Φ2)
- new net: U397. (Φ1), U399.
- new net: U774. (Φ1), U776. (Φ1)
- new net: U776. (Φ1), U778.
- new net: U480., U481., U483.
- new net: U425. (Φ1), U426. (Φ1)
- new net: U413. (Φ1), U414. (Φ1)
- new net: U15., U16.
- new net: U784. (Φ1), U786.
- new net: U785. (Φ1), U786.
- new net: U767. (Φ1), U769. (Φ1)
- new net: U769. (Φ1), U770.
- new net: U766. (Φ1), U86. (Φ2)
- new net: U766. (Φ1), U768. (Φ1)
- new net: U692., U693.
- new net: U650. (Φ2), U651.
- new net: U552., U553., U555.
- new net: U455., U555., U558., U577.
- new net: U484., U485., U488.
- new net: U770., U771.
- new net: U768. (Φ1), U770.
- new net: U386. (Φ1), U387. (Φ1)
- new net: U421. (Φ1), U422. (Φ1)
- new net: U744. (Φ1), U746.
- new net: U742. (Φ1), U744. (Φ1)
- new net: U579., U581. (Φ1)
- new net: U658. (Φ2), U660. (Φ1)
- new net: U734. (Φ1), U736. (Φ1)
- new net: U736. (Φ1), U737.
- new net: U544. (Φ1), U547.
- new net: U641. (Φ1), U642.
- new net: U525., U527. (Φ1)
- new net: U527. (Φ1), U600. (Φ1)
- new net: U417. (Φ1), U418. (Φ1)
- new net: U758. (Φ1), U760. (Φ1)
- new net: U758. (Φ1), U86. (Φ2)
- new net: U645., U646. (Φ2)
- new net: U751. (Φ1), U753. (Φ1)
- new net: U753. (Φ1), U754.
- new net: U436., U?.
- new net: U612., U613.
- new net: U446. (Φ1), U456.
- new net: U681., U682.
- new net: U532., U533., U536.
- new net: U692., U694. (Φ2), U699.
- new net: U433., U434. (Φ1), U?.
- new net: U580. (Φ1), U583.
- new net: U423. (Φ1), U424.
- new net: U656. (Φ1), U659. (Φ1)
- new net: U733. (Φ1), U86. (Φ2)
- new net: U550., U551., U554.
- new net: U775. (Φ1), U777. (Φ1)
- new net: U777. (Φ1), U778.
- new net: U457., U458., U459.
- new net: U705. (Φ1), U706. (Φ1)
- new net: U258., U261.
- new net: U13., U14.
- new net: U595. (Φ1), U596. (Φ1)
- new net: U643. (Φ1), U645.
- new net: U688. (Φ1), U689. (Φ1)
- new net: U530., U531.
- new net: U640., U641. (Φ1)
- new net: U727. (Φ1), U86. (Φ2)
- new net: U775. (Φ1), U86. (Φ2)
- new net: U631. (Φ2), U?.
- new net: U631. (Φ2), U632. (Φ1)
- new net: U392. (Φ1), U394.
- new net: U545. (Φ1), U599. (Φ1)
- new net: U546., U599. (Φ1)
- new net: U622., U623. (Φ1)
- new net: U492., U493., U494.
- new net: U490. (Φ1), U493.
- new net: U570., U571., U573.
- new net: U678., U679., U680.
- new net: U380. (Φ1), U381. (Φ1)
- new net: U578., U580. (Φ1)
- new net: U510., U511., U512.
- new net: U508. (Φ1), U511.
- new net: U726. (Φ1), U728. (Φ1)
- new net: U728. (Φ1), U730.
- new net: U726. (Φ1), U86. (Φ2)
- new net: U754., U755.
- new net: U697., U702. (Φ2)
- new net: U698. (Φ1), U699.
- new net: U685., U688. (Φ1)
- new net: U474., U603. (Φ1)
- new net: U568., U569., U572.
- new net: U383. (Φ1), U384. (Φ1)
- new net: U528., U600. (Φ1)
- new net: U258., U346.
- new net: U257., U258., U?.
- new net: U258., U259., U263.
- new net: U258., U260.
- new net: U587., U588., U589.
- new net: U774. (Φ1), U86. (Φ2)
- new net: U668. (S), U671.
- new net: U671., U674. (Φ1)
- new net: U415. (Φ1), U416.
- new net: U460., U461., U464.
- new net: U668. (S), U669.
- new net: U562. (Φ1), U565.
- new net: U783. (Φ1), U785. (Φ1)
- new net: U401. (Φ1), U402. (Φ1)
- new net: U782. (Φ1), U784. (Φ1)
- new net: U403. (Φ1), U404.
- new net: U612., U683. (Φ2)
- new net: U19., U779.
- new net: U407. (Φ1), U408.
- new net: U727. (Φ1), U729. (Φ1)
- new net: U729. (Φ1), U730.
- new net: U440. (Φ1), U?.
- new net: U663. (Φ1), U664. (Φ1)
- new net: U419. (Φ1), U420.
- new net: U472. (Φ1), U475.
- new net: U526. (Φ1), U529.
- new net: U534., U535., U537.
- new net: U605., U606. (Φ1)
- new net: U674. (Φ1), U674. (Φ1)
- new net: U509. (Φ1), U601. (Φ1)
- new net: U510., U601. (Φ1)
- new net: U632. (Φ1), U633.
- new net: U752. (Φ1), U754.
- new net: U634., U?.
- new net: U387. (Φ1), U388.
- new net: U675., U86. (Φ2)
- new net: U667. (Φ1), U675.
- now unconnected: U387. (Φ1), U387. (Φ1), U391. (Φ1), U391. (Φ1), U402. (Φ1), U402. (Φ1), U410. (Φ1), U410. (Φ1), U415. (Φ1), U415. (Φ1), U419. (Φ1), U419. (Φ1), U423. (Φ1), U423. (Φ1)

Commit message: update 20251028
Connections:
- net at U626.: now also U625.; no longer U627.
- net at U739.: now also U737.; no longer U9.
- net at U391. (Φ1): no longer U393.
- net at U?.: now also U633., U634.; no longer U636.
- net at U?.: now also U308. (Φ1), U353. (Φ1), U381. (Φ1), U384. (Φ1), U387. (Φ1), U391. (Φ1), U392. (Φ1), U397. (Φ1), U398. (Φ1), U403. (Φ1), U407. (Φ1), U411. (Φ1), U415. (Φ1), U419. (Φ1), U423. (Φ1), U427. (Φ1); no longer U431. (Φ1)
- net at U789.: now also U738.; no longer U788.
- net at U411. (Φ1): now also U410. (Φ1); no longer U412.
- net at U610.: now also U607.; no longer U611.
- net at U609.: now also U607., U608.; no longer U610.
- net at U352. (Φ1): now also U353. (Φ1)
- net at U353. (Φ1): now also U354.; no longer U352. (Φ1)
- net at U787.: now also U21.; no longer U786.
- net at U21.: now also U22.; no longer U787.
- net at U584.: now also U582., U583.; no longer U585.
- net at U763.: now also U15.; no longer U762.
- net at U629.: now also U662. (Φ1); no longer U630. (Φ2)
- net at U308. (Φ1): now also U128. (Φ1)
- net at U644.: now also U643. (Φ1); no longer U642.
- net at U11.: now also U747.; no longer U12.
- net at U747.: now also U746.; no longer U11.
- net at U619.: now also U617., U618.; no longer U620.
- net at U410. (Φ1): no longer U409. (Φ1)
- net at U655.: now also U659. (Φ1), U660. (Φ1); no longer U657. (Φ1)
- net at U670.: now also U668. (S); no longer U674. (Φ1)
- net at U476.: now also U474., U475.; no longer U477.
- net at U620.: now also U618.; no longer U621.
- net at U397. (Φ1): now also U395. (Φ1)
- net at U426. (Φ1): now also U427. (Φ1)
- net at U427. (Φ1): now also U428.; no longer U426. (Φ1)
- net at U414. (Φ1): now also U415. (Φ1); no longer U413. (Φ1)
- net at U625.: now also U624.; no longer U626.
- net at U651.: now also U653. (Φ2); no longer U650. (Φ2)
- net at U771.: now also U17.; no longer U770.
- net at U387. (Φ1): no longer U386. (Φ1)
- net at U422. (Φ1): now also U423. (Φ1)
- net at U423. (Φ1): no longer U422. (Φ1)
- net at U579.: now also U576., U577.; no longer U581. (Φ1)
- net at U642.: now also U647. (Φ1); no longer U641. (Φ1)
- net at U525.: now also U522., U523.; no longer U527. (Φ1)
- net at U418. (Φ1): now also U419. (Φ1)
- net at U419. (Φ1): no longer U418. (Φ1)
- net at U?.: now also U437. (Φ1); no longer U436.
- net at U456.: now also U454., U455.; no longer U446. (Φ1)
- net at U681.: now also U680.; no longer U682.
- net at U17.: now also U18.; no longer U771.
- net at U13.: now also U755.; no longer U14.
- net at U624.: now also U622.; no longer U625.
- net at U530.: now also U528., U529.; no longer U531.
- net at U392. (Φ1): now also U390. (Φ1); no longer U394.
- net at U381. (Φ1): now also U382.; no longer U380. (Φ1)
- net at U738.: now also U730.; no longer U789.
- net at U578.: now also U574., U575.; no longer U580. (Φ1)
- net at U697.: now also U696. (Φ1); no longer U702. (Φ2)
- net at U699.: now also U700.; no longer U698. (Φ1)
- net at U685.: now also U684.; no longer U688. (Φ1)
- net at U384. (Φ1): now also U385.; no longer U383. (Φ1)
- net at U671.: now also U673. (Φ1); no longer U668. (S)
- net at U415. (Φ1): no longer U416.
- net at U669.: now also U674. (Φ1); no longer U668. (S)
- net at U402. (Φ1): no longer U401. (Φ1)
- net at U403. (Φ1): now also U402. (Φ1)
- net at U779.: now also U778.; no longer U19.
- net at U407. (Φ1): now also U406. (Φ1)
- net at U406. (Φ1): now also U405. (Φ1); no longer U407. (Φ1)
- net at U?.: now also U439.; no longer U440. (Φ1)
- new net: U626., U627.
- new net: U689. (Φ1), U86. (Φ2)
- new net: U647. (Φ1), U648., U649. (Φ2)
- new net: U648., U649. (Φ2), U650. (Φ2)
- new net: U684., U686., U687.
- new net: U651., U652., U654. (Φ1)
- new net: U654. (Φ1), U655., U656. (Φ1)
- new net: U448., U454., U466., U468., U484., U486., U502., U504., U520., U522., U538., U540., U556., U558., U574., U576., U591., U592.
- new net: U520., U521., U524.
- new net: U518., U520., U557.
- new net: U739., U9.
- new net: U556., U557., U560.
- new net: U262., U263., U?.
- new net: U309., U382., U385., U388., U393., U394., U399., U400., U?.
- new net: U391. (Φ1), U393.
- new net: U676., U86. (Φ2)
- new net: U636., U?.
- new net: U431. (Φ1), U?.
- new net: U430., U431. (Φ1), U?.
- new net: U788., U789.
- new net: U354., U404., U408., U412., U416., U420., U424., U428., U?.
- new net: U411. (Φ1), U412.
- new net: U449., U455., U467., U469., U485., U487., U503., U505., U521., U523., U539., U541., U557., U559., U575., U577., U590., U591., U593.
- new net: U467., U573., U576.
- new net: U466., U467., U470.
- new net: U751. (Φ1), U86. (Φ2)
- new net: U610., U611.
- new net: U609., U610.
- new net: U465., U468., U487.
- new net: U468., U469., U471.
- new net: U614., U615.
- new net: U615., U616. (Φ1)
- new net: U442., U444., U445.
- new net: U445., U446. (Φ1)
- new net: U217. (Φ1), U352. (Φ1)
- new net: U352. (Φ1), U402. (Φ1), U406. (Φ1), U410. (Φ1), U414. (Φ1), U418. (Φ1), U422. (Φ1), U426. (Φ1), U?.
- new net: U486., U487., U489.
- new net: U396. (Φ1), U398. (Φ1)
- new net: U546., U547., U548.
- new net: U398. (Φ1), U400.
- new net: U564., U598. (Φ1)
- new net: U563. (Φ1), U598. (Φ1)
- new net: U743. (Φ1), U745. (Φ1)
- new net: U745. (Φ1), U746.
- new net: U761. (Φ1), U762.
- new net: U759. (Φ1), U761. (Φ1)
- new net: U389. (Φ1), U391. (Φ1)
- new net: U448., U451., U469.
- new net: U786., U787.
- new net: U584., U585.
- new net: U491. (Φ1), U602. (Φ1)
- new net: U447. (Φ1), U604. (Φ1)
- new net: U444., U604. (Φ1)
- new net: U762., U763.
- new net: U760. (Φ1), U762.
- new net: U742. (Φ1), U86. (Φ2)
- new net: U734. (Φ1), U86. (Φ2)
- new net: U629., U630. (Φ2)
- new net: U630. (Φ2), U631. (Φ2), U?.
- new net: U308. (Φ1), U309.
- new net: U642., U644.
- new net: U665. (Φ1), U667. (Φ1), U668. (S), U671.
- new net: U663. (Φ1), U665. (Φ1)
- new net: U665. (Φ1), U673. (Φ1)
- new net: U11., U12.
- new net: U619., U620.
- new net: U638. (Φ1), U86. (Φ2)
- new net: U637. (Φ1), U638. (Φ1)
- new net: U540., U541., U543.
- new net: U537., U540., U559.
- new net: U536., U538., U575.
- new net: U538., U539., U542.
- new net: U661. (Φ1), U662. (Φ1)
- new net: U661. (Φ1), U664. (Φ1)
- new net: U581. (Φ1), U597. (Φ1)
- new net: U582., U597. (Φ1)
- new net: U564., U565., U566.
- new net: U498., U499., U501.
- new net: U453., U458., U461., U463., U479., U481., U497., U499., U515., U517., U533., U535., U551., U553., U569., U571., U586., U588.
- new net: U692., U694. (Φ2), U695. (Φ1)
- new net: U695. (Φ1), U696. (Φ1), U698. (Φ1)
- new net: U483., U486., U505.
- new net: U504., U505., U507.
- new net: U750. (Φ1), U86. (Φ2)
- new net: U750. (Φ1), U752. (Φ1)
- new net: U409. (Φ1), U410. (Φ1)
- new net: U629., U657. (Φ1)
- new net: U655., U657. (Φ1)
- new net: U733. (Φ1), U735. (Φ1)
- new net: U735. (Φ1), U737.
- new net: U697., U699., U86. (Φ2)
- new net: U86. (Φ2), U86. (Φ2) (x2)
- new net: U767. (Φ1), U86. (Φ2)
- new net: U482., U484., U521.
- new net: U452., U457., U460., U462., U478., U480., U496., U498., U514., U516., U532., U534., U550., U552., U568., U570., U586., U587.
- new net: U478., U479., U482.
- new net: U516., U517., U519.
- new net: U462., U463., U465.
- new net: U492., U602. (Φ1)
- new net: U448., U449., U450.
- new net: U451., U452., U453.
- new net: U651., U653. (Φ2), U674. (Φ1)
- new net: U670., U674. (Φ1)
- new net: U476., U477.
- new net: U514., U515., U518.
- new net: U592., U593., U594.
- new net: U782. (Φ1), U86. (Φ2)
- new net: U783. (Φ1), U86. (Φ2)
- new net: U620., U621.
- new net: U759. (Φ1), U86. (Φ2)
- new net: U502., U503., U506.
- new net: U496., U497., U500.
- new net: U473. (Φ1), U603. (Φ1)
- new net: U743. (Φ1), U86. (Φ2)
- new net: U397. (Φ1), U399.
- new net: U774. (Φ1), U776. (Φ1)
- new net: U776. (Φ1), U778.
- new net: U480., U481., U483.
- new net: U425. (Φ1), U426. (Φ1)
- new net: U413. (Φ1), U414. (Φ1)
- new net: U15., U16.
- new net: U784. (Φ1), U786.
- new net: U785. (Φ1), U786.
- new net: U767. (Φ1), U769. (Φ1)
- new net: U769. (Φ1), U770.
- new net: U766. (Φ1), U86. (Φ2)
- new net: U766. (Φ1), U768. (Φ1)
- new net: U692., U693.
- new net: U650. (Φ2), U651.
- new net: U552., U553., U555.
- new net: U455., U555., U558., U577.
- new net: U484., U485., U488.
- new net: U770., U771.
- new net: U768. (Φ1), U770.
- new net: U386. (Φ1), U387. (Φ1)
- new net: U421. (Φ1), U422. (Φ1)
- new net: U744. (Φ1), U746.
- new net: U742. (Φ1), U744. (Φ1)
- new net: U579., U581. (Φ1)
- new net: U658. (Φ2), U660. (Φ1)
- new net: U734. (Φ1), U736. (Φ1)
- new net: U736. (Φ1), U737.
- new net: U544. (Φ1), U547.
- new net: U641. (Φ1), U642.
- new net: U525., U527. (Φ1)
- new net: U527. (Φ1), U600. (Φ1)
- new net: U417. (Φ1), U418. (Φ1)
- new net: U758. (Φ1), U760. (Φ1)
- new net: U758. (Φ1), U86. (Φ2)
- new net: U645., U646. (Φ2)
- new net: U751. (Φ1), U753. (Φ1)
- new net: U753. (Φ1), U754.
- new net: U436., U?.
- new net: U612., U613.
- new net: U446. (Φ1), U456.
- new net: U681., U682.
- new net: U532., U533., U536.
- new net: U692., U694. (Φ2), U699.
- new net: U433., U434. (Φ1), U?.
- new net: U580. (Φ1), U583.
- new net: U423. (Φ1), U424.
- new net: U656. (Φ1), U659. (Φ1)
- new net: U733. (Φ1), U86. (Φ2)
- new net: U550., U551., U554.
- new net: U775. (Φ1), U777. (Φ1)
- new net: U777. (Φ1), U778.
- new net: U457., U458., U459.
- new net: U705. (Φ1), U706. (Φ1)
- new net: U258., U261.
- new net: U13., U14.
- new net: U595. (Φ1), U596. (Φ1)
- new net: U643. (Φ1), U645.
- new net: U688. (Φ1), U689. (Φ1)
- new net: U530., U531.
- new net: U640., U641. (Φ1)
- new net: U727. (Φ1), U86. (Φ2)
- new net: U775. (Φ1), U86. (Φ2)
- new net: U631. (Φ2), U?.
- new net: U631. (Φ2), U632. (Φ1)
- new net: U392. (Φ1), U394.
- new net: U545. (Φ1), U599. (Φ1)
- new net: U546., U599. (Φ1)
- new net: U622., U623. (Φ1)
- new net: U492., U493., U494.
- new net: U490. (Φ1), U493.
- new net: U570., U571., U573.
- new net: U678., U679., U680.
- new net: U380. (Φ1), U381. (Φ1)
- new net: U578., U580. (Φ1)
- new net: U510., U511., U512.
- new net: U508. (Φ1), U511.
- new net: U726. (Φ1), U728. (Φ1)
- new net: U728. (Φ1), U730.
- new net: U726. (Φ1), U86. (Φ2)
- new net: U754., U755.
- new net: U697., U702. (Φ2)
- new net: U698. (Φ1), U699.
- new net: U685., U688. (Φ1)
- new net: U474., U603. (Φ1)
- new net: U568., U569., U572.
- new net: U383. (Φ1), U384. (Φ1)
- new net: U528., U600. (Φ1)
- new net: U258., U346.
- new net: U257., U258., U?.
- new net: U258., U259., U263.
- new net: U258., U260.
- new net: U587., U588., U589.
- new net: U774. (Φ1), U86. (Φ2)
- new net: U668. (S), U671.
- new net: U671., U674. (Φ1)
- new net: U415. (Φ1), U416.
- new net: U460., U461., U464.
- new net: U668. (S), U669.
- new net: U562. (Φ1), U565.
- new net: U783. (Φ1), U785. (Φ1)
- new net: U401. (Φ1), U402. (Φ1)
- new net: U782. (Φ1), U784. (Φ1)
- new net: U403. (Φ1), U404.
- new net: U612., U683. (Φ2)
- new net: U19., U779.
- new net: U407. (Φ1), U408.
- new net: U727. (Φ1), U729. (Φ1)
- new net: U729. (Φ1), U730.
- new net: U440. (Φ1), U?.
- new net: U663. (Φ1), U664. (Φ1)
- new net: U419. (Φ1), U420.
- new net: U472. (Φ1), U475.
- new net: U526. (Φ1), U529.
- new net: U534., U535., U537.
- new net: U605., U606. (Φ1)
- new net: U674. (Φ1), U674. (Φ1)
- new net: U509. (Φ1), U601. (Φ1)
- new net: U510., U601. (Φ1)
- new net: U632. (Φ1), U633.
- new net: U752. (Φ1), U754.
- new net: U634., U?.
- new net: U387. (Φ1), U388.
- new net: U675., U86. (Φ2)
- new net: U667. (Φ1), U675.
- new net BUS.CASBUS.D_{0}: U86. (Φ2)
- new net BUS.CASBUS.D_{1}: U86. (Φ2)
- new net BUS.CASBUS.D_{2}: U86. (Φ2)
- new net BUS.CASBUS.D_{3}: U86. (Φ2)
- new net BUS.CASBUS.D_{4}: U86. (Φ2)
- new net BUS.CASBUS.D_{5}: U86. (Φ2)
- new net BUS.CASBUS.D_{6}: U86. (Φ2)
- new net BUS.CASBUS.D_{7}: U86. (Φ2)
- now unconnected: U387. (Φ1), U387. (Φ1), U391. (Φ1), U391. (Φ1), U402. (Φ1), U402. (Φ1), U410. (Φ1), U410. (Φ1), U415. (Φ1), U415. (Φ1), U419. (Φ1), U419. (Φ1), U423. (Φ1), U423. (Φ1)
Changed lines of the file:
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@@
 	(wire
 		(pts
+			(xy 279.4 256.54) (xy 303.53 256.54)
+		)
+		(stroke
+			(width 0)
+			(type default)
+		)
+	)
+	(wire
+		(pts
 			(xy 374.65 314.96) (xy 374.65 313.69)
 		)
@@
 	(wire
 		(pts
+			(xy 279.4 180.34) (xy 303.53 180.34)
+		)
+		(stroke
+			(width 0)
+			(type default)
+		)
+	)
+	(wire
+		(pts
 			(xy 520.7 707.39) (xy 534.67 707.39)
 		)
@@
 	(wire
 		(pts
+			(xy 279.4 195.58) (xy 303.53 195.58)
+		)
+		(stroke
+			(width 0)
+			(type default)
+		)
+	)
+	(wire
+		(pts
 			(xy 803.91 146.05) (xy 803.91 130.81)
 		)
@@
 	(wire
 		(pts
+			(xy 279.4 241.3) (xy 303.53 241.3)
+		)
+		(stroke
+			(width 0)
+			(type default)
+		)
+	)
+	(wire
+		(pts
 			(xy 805.18 267.97) (xy 803.91 267.97)
 		)
@@
 	(wire
 		(pts
+			(xy 279.4 210.82) (xy 303.53 210.82)
+		)
+		(stroke
+			(width 0)
+			(type default)
+		)
+	)
+	(wire
+		(pts
 			(xy 388.62 234.95) (xy 424.18 234.95)
 		)
@@
 	(wire
 		(pts
+			(xy 279.4 226.06) (xy 303.53 226.06)
+		)
+		(stroke
+			(width 0)
+			(type default)
+		)
+	)
+	(wire
+		(pts
 			(xy 845.82 533.4) (xy 848.36 533.4)
 		)
@@
 	(wire
 		(pts
+			(xy 279.4 271.78) (xy 303.53 271.78)
+		)
+		(stroke
+			(width 0)
+			(type default)
+		)
+	)
+	(wire
+		(pts
 			(xy 660.4 422.91) (xy 664.21 422.91)
 		)
@@
 	(wire
 		(pts
+			(xy 279.4 165.1) (xy 303.53 165.1)
+		)
+		(stroke
+			(width 0)
+			(type default)
+		)
+	)
+	(wire
+		(pts
 			(xy 543.56 558.8) (xy 551.18 558.8)
 		)
@@
 		)
 	)
+	(label "BUS.CASBUS.D_{0}"
+		(at 279.4 165.1 0)
+		(fields_autoplaced yes)
+		(effects
+			(font
+				(size 1.27 1.27)
+			)
+			(justify left bottom)
+		)
+	)
 	(label "CLK.phiL"
 		(at 429.26 147.32 0)
@@
 		)
 	)
+	(label "BUS.CASBUS.D_{1}"
+		(at 279.4 180.34 0)
+		(fields_autoplaced yes)
+		(effects
+			(font
+				(size 1.27 1.27)
+			)
+			(justify left bottom)
+		)
+	)
 	(label "NET.VA.A_{13}"
 		(at 344.17 312.42 0)
@@
 		)
 	)
+	(label "BUS.CASBUS.D_{4}"
+		(at 279.4 226.06 0)
+		(fields_autoplaced yes)
+		(effects
+			(font
+				(size 1.27 1.27)
+			)
+			(justify left bottom)
+		)
+	)
 	(label "NET.VA.A_{5}"
 		(at 328.93 236.22 180)
@@
 		)
 	)
+	(label "BUS.CASBUS.D_{5}"
+		(at 279.4 241.3 0)
+		(fields_autoplaced yes)
+		(effects
+			(font
+				(size 1.27 1.27)
+			)
+			(justify left bottom)
+		)
+	)
 	(label "NET.REG_d8_b3_VR"
 		(at 288.29 453.39 0)
@@
 		)
 	)
+	(label "BUS.CASBUS.D_{3}"
+		(at 279.4 210.82 0)
+		(fields_autoplaced yes)
+		(effects
+			(font
+				(size 1.27 1.27)
+			)
+			(justify left bottom)
+		)
+	)
 	(label "NET.DRAM.COLADDR_EN"
 		(at 906.78 725.17 180)
@@
 		)
 	)
+	(label "BUS.CASBUS.D_{2}"
+		(at 279.4 195.58 0)
+		(fields_autoplaced yes)
+		(effects
+			(font
+				(size 1.27 1.27)
+			)
+			(justify left bottom)
+		)
+	)
 	(label "CLK.~{phiA}"
 		(at 830.58 520.7 0)
@@
 		)
 	)
+	(label "BUS.CASBUS.D_{7}"
+		(at 279.4 271.78 0)
+		(fields_autoplaced yes)
+		(effects
+			(font
+				(size 1.27 1.27)
+			)
+			(justify left bottom)
+		)
+	)
 	(label "NET.RD.D_{3}"
 		(at 631.19 361.95 0)
@@
 		)
 	)
+	(label "BUS.CASBUS.D_{6}"
+		(at 279.4 256.54 0)
+		(fields_autoplaced yes)
+		(effects
+			(font
+				(size 1.27 1.27)
+			)
+			(justify left bottom)
+		)
+	)

Commit message: update 20251106
Parts:
- removed U586: GM029, symbol Raki_ASIC_cells:COMPBUFP
- removed U700: GM090, symbol Raki_ASIC_cells:COMPBUFP
- added U1726: GM090, symbol Raki_ASIC_cells:BUFC
- added U700: GM029, symbol Raki_ASIC_cells:BUFCP1
Connections:
- net BUS.VRAM01X_INLATCH.D_{0} is gone; now on net BUS.VRAM01X_INBUF.D_{0}: U309.
- net BUS.VRAM01X_INLATCH.D_{1} is gone; now on net BUS.VRAM01X_INBUF.D_{1}: U382.
- net BUS.VRAM01X_INLATCH.D_{2} is gone; now on net BUS.VRAM01X_INBUF.D_{2}: U385.
- net BUS.VRAM01X_INLATCH.D_{3} is gone; now on net BUS.VRAM01X_INBUF.D_{3}: U388.
- net BUS.VRAM01X_INLATCH.D_{6} is gone; now on net BUS.VRAM01X_INBUF.D_{6}: U399.
- net BUS.VRAM01X_INLATCH.D_{7} is gone; now on net BUS.VRAM01X_INBUF.D_{7}: U400.
- net BUS.VRAM01X_INLATCH.OE is gone; now on net CLK.~{phiL}: U437. (Φ1)
- net NET.DRAM.OUTLATCH_SEL0: now also U1726.
- net NET.DRAM.OUTLATCH_SEL1: now also U1726.
- net at U626.: now also U625.; no longer U627.
- net at U739.: now also U737.; no longer U9.
- net at U391. (Φ1): no longer U393.
- net NET.GT109: now reaches U676.
- net at U?.: now also U633., U634.; no longer U636.
- net at U?.: now also U308. (Φ1), U353. (Φ1), U381. (Φ1), U384. (Φ1), U387. (Φ1), U391. (Φ1), U392. (Φ1), U397. (Φ1), U398. (Φ1), U403. (Φ1), U407. (Φ1), U411. (Φ1)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; no longer U431. (Φ1)
- net at U789.: now also U738.; no longer U788.
- net at U411. (Φ1): now also U410. (Φ1); no longer U412.
- net at U610.: now also U607.; no longer U611.
- net at U609.: now also U607., U608.; no longer U610.
- net at U352. (Φ1): now also U353. (Φ1)
- net at U353. (Φ1): now also U354.; no longer U352. (Φ1)
- net BUS.VRAM01X_INBUF.D_{7}: now reaches U400.
- net BUS.VRAM01X_INBUF.D_{7}: no longer U398. (Φ1)
- net at U787.: now also U21.; no longer U786.
- net at U21.: now also U22.; no longer U787.
- net at U584.: now also U582., U583.; no longer U585.
- net at U763.: now also U15.; no longer U762.
- net at U629.: now also U662. (Φ1); no longer U630. (Φ2)
- net at U308. (Φ1): now also U128. (Φ1)
- net BUS.VRAM01X_INBUF.D_{0}: now reaches U309.
- net BUS.VRAM01X_INBUF.D_{0}: no longer U308. (Φ1)
- net at U644.: now also U643. (Φ1); no longer U642.
- net at U11.: now also U747.; no longer U12.
- net at U747.: now also U746.; no longer U11.
- net at U619.: now also U617., U618.; no longer U620.
- net at U410. (Φ1): no longer U409. (Φ1)
- net at U655.: now also U659. (Φ1), U660. (Φ1); no longer U657. (Φ1)
- net at U670.: now also U668. (S); no longer U674. (Φ1)
- net at U476.: now also U474., U475.; no longer U477.
- net at U620.: now also U618.; no longer U621.
- net at U397. (Φ1): now also U395. (Φ1)
- net BUS.VRAM01X_INBUF.D_{6}: now reaches U399.
- net BUS.VRAM01X_INBUF.D_{6}: no longer U397. (Φ1)
- net at U426. (Φ1): now also U427. (Φ1)
- net at U427. (Φ1): now also U428.; no longer U426. (Φ1)
- net at U414. (Φ1): now also U415. (Φ1); no longer U413. (Φ1)
- net at U625.: now also U624.; no longer U626.
- net at U651.: now also U653. (Φ2); no longer U650. (Φ2)
- net at U771.: now also U17.; no longer U770.
- net at U387. (Φ1): no longer U386. (Φ1)
- net at U422. (Φ1): now also U423. (Φ1)
- net at U423. (Φ1): no longer U422. (Φ1)
- net at U579.: now also U576., U577.; no longer U581. (Φ1)
- net NET.~{GT106}_Z: now reaches U658. (Φ2)
- net at U642.: now also U647. (Φ1); no longer U641. (Φ1)
- net at U525.: now also U522., U523.; no longer U527. (Φ1)
- net at U418. (Φ1): now also U419. (Φ1)
- net at U419. (Φ1): no longer U418. (Φ1)
- net at U?.: now also U437. (Φ1); no longer U436.
- net at U456.: now also U454., U455.; no longer U446. (Φ1)
- net at U681.: now also U680.; no longer U682.
- net BUS.VRAM1_INBUF.D_{6}: now reaches U424.
- net BUS.VRAM1_INBUF.D_{6}: now also U86. (Φ2); no longer U423. (Φ1)
- net at U17.: now also U18.; no longer U771.
- net at U13.: now also U755.; no longer U14.
- net at U624.: now also U622.; no longer U625.
- net at U530.: now also U528., U529.; no longer U531.
- net at U392. (Φ1): now also U390. (Φ1); no longer U394.
- net BUS.VRAM1_INBUF.OE: now reaches U441.
- net BUS.VRAM1_INBUF.OE: now also U440. (Φ1)
- net at U381. (Φ1): now also U382.; no longer U380. (Φ1)
- net at U738.: now also U730.; no longer U789.
- net at U578.: now also U574., U575.; no longer U580. (Φ1)
- net at U697.: now also U696. (Φ1); no longer U702. (Φ2)
- net at U699.: now also U1726.; no longer U698. (Φ1)
- net at U685.: now also U684.; no longer U688. (Φ1)
- net at U384. (Φ1): now also U385.; no longer U383. (Φ1)
- net BUS.VRAM1_INBUF.D_{0}: now reaches U354.
- net BUS.VRAM1_INBUF.D_{0}: now also U86. (Φ2); no longer U353. (Φ1)
- net BUS.VRAM01X_INBUF.D_{1}: now reaches U382.
- net BUS.VRAM01X_INBUF.D_{1}: no longer U381. (Φ1)
- net at U671.: now also U673. (Φ1); no longer U668. (S)
- net at U415. (Φ1): no longer U416.
- net at U669.: now also U674. (Φ1); no longer U668. (S)
- net at U402. (Φ1): no longer U401. (Φ1)
- net at U403. (Φ1): now also U402. (Φ1)
- net BUS.VRAM1_INBUF.D_{1}: now reaches U404.
- net BUS.VRAM1_INBUF.D_{1}: now also U86. (Φ2); no longer U403. (Φ1)
- net at U779.: now also U778.; no longer U19.
- net at U407. (Φ1): now also U406. (Φ1)
- net BUS.VRAM1_INBUF.D_{2}: now reaches U408.
- net BUS.VRAM1_INBUF.D_{2}: now also U86. (Φ2); no longer U407. (Φ1)
- net at U406. (Φ1): now also U405. (Φ1); no longer U407. (Φ1)
- net at U?.: now also U439.; no longer U440. (Φ1)
- net BUS.VRAM1_INBUF.D_{5}: now reaches U420.
- net BUS.VRAM1_INBUF.D_{5}: now also U86. (Φ2); no longer U419. (Φ1)
- net BUS.VRAM1_INBUF.D_{7}: now reaches U428.
- net BUS.VRAM1_INBUF.D_{7}: now also U86. (Φ2); no longer U427. (Φ1)
- net BUS.VRAM01X_INBUF.D_{3}: now reaches U388.
- net BUS.VRAM01X_INBUF.D_{3}: no longer U387. (Φ1)
- net BUS.VRAM01X_INBUF.D_{2}: now reaches U385.
- net BUS.VRAM01X_INBUF.D_{2}: no longer U384. (Φ1)
- net BUS.VRAM01X_INLATCH.D_{4} renamed BUS.VRAM01X_INBUF.D_{4}
- net BUS.VRAM01X_INLATCH.D_{5} renamed BUS.VRAM01X_INBUF.D_{5}
- removed net BUS.VRAM1_INLATCH.D_{0}: U354., U86. (Φ2)
- removed net BUS.VRAM1_INLATCH.D_{1}: U404., U86. (Φ2)
- removed net BUS.VRAM1_INLATCH.D_{2}: U408., U86. (Φ2)
- net BUS.VRAM1_INLATCH.D_{3} renamed BUS.VRAM1_INBUF.D_{3}
- net BUS.VRAM1_INLATCH.D_{4} renamed BUS.VRAM1_INBUF.D_{4}
- removed net BUS.VRAM1_INLATCH.D_{5}: U420., U86. (Φ2)
- removed net BUS.VRAM1_INLATCH.D_{6}: U424., U86. (Φ2)
- removed net BUS.VRAM1_INLATCH.D_{7}: U428., U86. (Φ2)
- removed net BUS.VRAM1_INLATCH.OE: U440. (Φ1), U441.
- new net: U626., U627.
- new net: U689. (Φ1), U86. (Φ2)
- new net: U647. (Φ1), U648., U649. (Φ2)
- new net: U648., U649. (Φ2), U650. (Φ2)
- new net: U684., U686., U687.
- new net: U651., U652., U654. (Φ1)
- new net: U654. (Φ1), U655., U656. (Φ1)
- new net: U448., U454., U466., U468., U484., U486., U502., U504., U520., U522., U538., U540.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
- new net: U520., U521., U524.
- new net: U518., U520., U557.
- new net: U739., U9.
- new net: U556., U557., U560.
- new net: U262., U263., U?.
- new net: U309., U382., U385., U388., U393., U394., U399., U400., U?.
- new net: U391. (Φ1), U393.
- new net: U676., U86. (Φ2)
- new net: U636., U?.
- new net: U431. (Φ1), U?.
- new net: U430., U431. (Φ1), U?.
- new net: U788., U789.
- new net: U354., U404., U408., U412., U416., U420., U424., U428., U?.
- new net: U411. (Φ1), U412.
- new net: U449., U455., U467., U469., U485., U487., U503., U505., U521., U523., U539., U541.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
- new net: U467., U573., U576.
- new net: U466., U467., U470.
- new net: U751. (Φ1), U86. (Φ2)
- new net: U610., U611.
- new net: U609., U610.
- new net: U465., U468., U487.
- new net: U468., U469., U471.
- new net: U614., U615.
- new net: U615., U616. (Φ1)
- new net: U442., U444., U445.
- new net: U445., U446. (Φ1)
- new net: U217. (Φ1), U352. (Φ1)
- new net: U352. (Φ1), U402. (Φ1), U406. (Φ1), U410. (Φ1), U414. (Φ1), U418. (Φ1), U422. (Φ1), U426. (Φ1), U?.
- new net: U486., U487., U489.
- new net: U396. (Φ1), U398. (Φ1)
- new net: U546., U547., U548.
- new net: U398. (Φ1), U400.
- new net: U564., U598. (Φ1)
- new net: U563. (Φ1), U598. (Φ1)
- new net: U743. (Φ1), U745. (Φ1)
- new net: U745. (Φ1), U746.
- new net: U761. (Φ1), U762.
- new net: U759. (Φ1), U761. (Φ1)
- new net: U389. (Φ1), U391. (Φ1)
- new net: U448., U451., U469.
- new net: U786., U787.
- new net: U584., U585.
- new net: U491. (Φ1), U602. (Φ1)
- new net: U447. (Φ1), U604. (Φ1)
- new net: U444., U604. (Φ1)
- new net: U762., U763.
- new net: U760. (Φ1), U762.
- new net: U742. (Φ1), U86. (Φ2)
- new net: U734. (Φ1), U86. (Φ2)
- new net: U629., U630. (Φ2)
- new net: U630. (Φ2), U631. (Φ2), U?.
- new net: U308. (Φ1), U309.
- new net: U642., U644.
- new net: U665. (Φ1), U667. (Φ1), U668. (S), U671.
- new net: U663. (Φ1), U665. (Φ1)
- new net: U665. (Φ1), U673. (Φ1)
- new net: U11., U12.
- new net: U619., U620.
- new net: U638. (Φ1), U86. (Φ2)
- new net: U637. (Φ1), U638. (Φ1)
- new net: U540., U541., U543.
- new net: U537., U540., U559.
- new net: U536., U538., U575.
- new net: U538., U539., U542.
- new net: U661. (Φ1), U662. (Φ1)
- new net: U661. (Φ1), U664. (Φ1)
- new net: U581. (Φ1), U597. (Φ1)
- new net: U582., U597. (Φ1)
- new net: U564., U565., U566.
- new net: U498., U499., U501.
- new net: U453., U458., U461., U463., U479., U481., U497., U499., U515., U517., U533., U535.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
- new net: U692., U694. (Φ2), U695. (Φ1)
- new net: U695. (Φ1), U696. (Φ1), U698. (Φ1)
- new net: U483., U486., U505.
- new net: U504., U505., U507.
- new net: U750. (Φ1), U86. (Φ2)
- new net: U750. (Φ1), U752. (Φ1)
- new net: U409. (Φ1), U410. (Φ1)
- new net: U629., U657. (Φ1)
- new net: U655., U657. (Φ1)
- new net: U733. (Φ1), U735. (Φ1)
- new net: U735. (Φ1), U737.
- new net: U697., U699., U86. (Φ2)
- new net: U86. (Φ2), U86. (Φ2) (x2)
- new net: U767. (Φ1), U86. (Φ2)
- new net: U482., U484., U521.
- new net: U452., U457., U460., U462., U478., U480., U496., U498., U514., U516., U532., U534.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
- new net: U478., U479., U482.
- new net: U516., U517., U519.
- new net: U462., U463., U465.
- new net: U492., U602. (Φ1)
- new net: U448., U449., U450.
- new net: U451., U452., U453.
- new net: U651., U653. (Φ2), U674. (Φ1)
- new net: U670., U674. (Φ1)
- new net: U476., U477.
- new net: U514., U515., U518.
- new net: U592., U593., U594.
- new net: U782. (Φ1), U86. (Φ2)
- new net: U783. (Φ1), U86. (Φ2)
- new net: U620., U621.
- new net: U759. (Φ1), U86. (Φ2)
- new net: U502., U503., U506.
- new net: U496., U497., U500.
- new net: U473. (Φ1), U603. (Φ1)
- new net: U743. (Φ1), U86. (Φ2)
- new net: U397. (Φ1), U399.
- new net: U774. (Φ1), U776. (Φ1)
- new net: U776. (Φ1), U778.
- new net: U480., U481., U483.
- new net: U425. (Φ1), U426. (Φ1)
- new net: U413. (Φ1), U414. (Φ1)
- new net: U15., U16.
- new net: U784. (Φ1), U786.
- new net: U785. (Φ1), U786.
- new net: U767. (Φ1), U769. (Φ1)
- new net: U769. (Φ1), U770.
- new net: U766. (Φ1), U86. (Φ2)
- new net: U766. (Φ1), U768. (Φ1)
- new net: U692., U693.
- new net: U650. (Φ2), U651.
- new net: U552., U553., U555.
- new net: U455., U555., U558., U577.
- new net: U484., U485., U488.
- new net: U770., U771.
- new net: U768. (Φ1), U770.
- new net: U386. (Φ1), U387. (Φ1)
- new net: U421. (Φ1), U422. (Φ1)
- new net: U744. (Φ1), U746.
- new net: U742. (Φ1), U744. (Φ1)
- new net: U579., U581. (Φ1)
- new net: U658. (Φ2), U660. (Φ1)
- new net: U734. (Φ1), U736. (Φ1)
- new net: U736. (Φ1), U737.
- new net: U544. (Φ1), U547.
- new net: U641. (Φ1), U642.
- new net: U525., U527. (Φ1)
- new net: U527. (Φ1), U600. (Φ1)
- new net: U417. (Φ1), U418. (Φ1)
- new net: U758. (Φ1), U760. (Φ1)
- new net: U758. (Φ1), U86. (Φ2)
- new net: U645., U646. (Φ2)
- new net: U751. (Φ1), U753. (Φ1)
- new net: U753. (Φ1), U754.
- new net: U436., U?.
- new net: U612., U613.
- new net: U446. (Φ1), U456.
- new net: U681., U682.
- new net: U532., U533., U536.
- new net: U692., U694. (Φ2), U699.
- new net: U433., U434. (Φ1), U?.
- new net: U580. (Φ1), U583.
- new net: U423. (Φ1), U424.
- new net: U656. (Φ1), U659. (Φ1)
- new net: U733. (Φ1), U86. (Φ2)
- new net: U550., U551., U554.
- new net: U775. (Φ1), U777. (Φ1)
- new net: U777. (Φ1), U778.
- new net: U457., U458., U459.
- new net: U705. (Φ1), U706. (Φ1)
- new net: U700., U705. (Φ1)
- new net: U258., U261.
- new net: U13., U14.
- new net: U595. (Φ1), U596. (Φ1)
- new net: U643. (Φ1), U645.
- new net: U688. (Φ1), U689. (Φ1)
- new net: U530., U531.
- new net: U640., U641. (Φ1)
- new net: U727. (Φ1), U86. (Φ2)
- new net: U775. (Φ1), U86. (Φ2)
- new net: U631. (Φ2), U?.
- new net: U631. (Φ2), U632. (Φ1)
- new net: U392. (Φ1), U394.
- new net: U545. (Φ1), U599. (Φ1)
- new net: U546., U599. (Φ1)
- new net: U622., U623. (Φ1)
- new net: U492., U493., U494.
- new net: U490. (Φ1), U493.
- new net: U570., U571., U573.
- new net: U678., U679., U680.
- new net: U380. (Φ1), U381. (Φ1)
- new net: U578., U580. (Φ1)
- new net: U510., U511., U512.
- new net: U508. (Φ1), U511.
- new net: U726. (Φ1), U728. (Φ1)
- new net: U728. (Φ1), U730.
- new net: U726. (Φ1), U86. (Φ2)
- new net: U754., U755.
- new net: U697., U702. (Φ2)
- new net: U698. (Φ1), U699.
- new net: U685., U688. (Φ1)
- new net: U474., U603. (Φ1)
- new net: U568., U569., U572.
- new net: U383. (Φ1), U384. (Φ1)
- new net: U528., U600. (Φ1)
- new net: U258., U346.
- new net: U257., U258., U?.
- new net: U258., U259., U263.
- new net: U258., U260.
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