File: resources/V9958_kicad/PLA0.kicad_sch (KiCad schematic)
At the start: 343 parts, among them U1000 NMOS, U1001 INV, U1002 NMOS, U1003 INV, U1004 NMOS, U1005 INV, U1006 NMOS, U1007 GT050, U1008 GT051, U1009 GT052, U1010 GT053, U1011 GT054, U1012 AND2, U1013 AND2, U1014 OR2, U1015 OR6, U1016 TBD, U1017 INVP, U1018 INVP, U1019 OR4, U1020 INV, U1021 TBD, U1022 INV, U1023 INV, U1024 INV, U1025 INV, U1026 INV, U1027 INV, U1028 INV, U1029 INV, U1030 INV, U1031 NMOS, U1032 NMOS, U1033 NMOS, U1034 NMOS, U1035 INV, U1036 INV, U1037 INV, U1038 INV, U1041 GT055, U1044 GT056, U1047 GT057, U1050 GT058, U1051 NMOS, U1052 NMOS, U1053 GT060, U1054 NMOS, U1055 NMOS, U1056 NMOS, U1057 NMOS, U1058 NMOS, U1059 NMOS, U1068 GT065, U1069 GT066, U1070 GT067, U1071 GT068, U1072 NMOS, U1073 NMOS, U1074 NMOS, U1075 GT070, U1076 GT069, U1077 INV, U1078 GT071, U1079 GT072, U1080 GT079, U1081 INV, U1082 NMOS, U1084 GT074, U1085 GT075, U1086 GT076, U1087 GT077, U1088 GT078, U1089 GT081, U1090 NMOS, U1091 NMOS, U1092 NMOS, U1093 NMOS, U1094 NMOS, U1095 GT079, U1096 GT080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

Commit message: update 20250809
HVCNTR
Parts:
- added TP008, TP009: ~, symbol Connector:TestPoint
- added U1125, U1126, U1139, U1140, U1141, U1180, U1254, U1255, U1258, U1260, U1262, U1296, U1298, U1299, U1301, U1302, U1303, U1304, U1305: INV, symbol Raki_ASIC_cells:INV
- added U1127, U1128, U1129, U1130, U1131, U1132, U1133, U1134, U1135, U1136, U1137, U1138, U1142, U1143, U1144, U1145, U1146, U1147, U1148, U1149, U1150, U1151, U1152, U1153, U1154, U1155, U1156, U1157, U1158, U1159, U1160, U1161, U1162, U1163, U1164, U1165, U1166, U1167, U1168, U1169, U1170, U1171, U1189, U1213, U1215, U1217, U1219, U1221, U1223, U1225, U1227, U1229, U1231, U1233, U1235, U1237, U1239, U1241, U1263, U1266, U1268, U1270, U1272, U1274, U1276, U1278, U1280, U1282, U1284, U1286, U1288, U1290: NORWIDE, symbol Raki_ASIC_cells:NORWIDE
- added U1172: GT094, symbol Raki_ASIC_cells:NOR4
- added U1173: GT095, symbol Raki_ASIC_cells:NOR5
- added U1174: GT096, symbol Raki_ASIC_cells:NOR2
- added U1175: GT097, symbol Raki_ASIC_cells:NAND2
- added U1176: GT101, symbol Raki_ASIC_cells:NORWIDE
- added U1177: GT098, symbol Raki_ASIC_cells:NOR3
- added U1178: GT100, symbol Raki_ASIC_cells:NORWIDE
- added U1179: GT099, symbol Raki_ASIC_cells:NORWIDE
- added U1181: GT103, symbol Raki_ASIC_cells:INV
- added U1182, U1186, U1187, U1188, U1210, U1212, U1214, U1216, U1218, U1220, U1222, U1224, U1226, U1228, U1230, U1232, U1234, U1236, U1238, U1240, U1259, U1265, U1267, U1269, U1271, U1273, U1275, U1277, U1279, U1281, U1283, U1285, U1287, U1289, U1327, U1329, U1330, U1331, U1332, U1333, U1334, U1335, U1337, U1338: NMOS, symbol Raki_ASIC_cells:NMOS
- added U1183: GT104, symbol Raki_ASIC_cells:INV
- added U1184: GT105, symbol Raki_ASIC_cells:NMOS
- added U1185: GT106, symbol Raki_ASIC_cells:INV
- added U1190: GT080, symbol Raki_ASIC_cells:INV
- added U1196, U1197, U1199, U1202, U1203, U1204, U1208, U1293, U1308, U1311, U1312, U1314, U1319, U1320, U1321, U1324, U1325: DDL, symbol Raki_ASIC_cells:VY_DDL_small
- added U1198: GT107, symbol Raki_ASIC_cells:INVP
- added U1200: GT105, symbol Raki_ASIC_cells:NOR3
- added U1201: GT108, symbol Raki_ASIC_cells:NOR2P
- added U1205: GT109, symbol Raki_ASIC_cells:INVP
- added U1206: GT110, symbol Raki_ASIC_cells:NOR2
- added U1207: GT111, symbol Raki_ASIC_cells:NOR2
- added U1209: GT112, symbol Raki_ASIC_cells:INVP
- added U1211: GT113, symbol Raki_ASIC_cells:INVP
- added U1242, U1249: NOR3, symbol Raki_ASIC_cells:NOR3
- added U1243: GT114, symbol Raki_ASIC_cells:NOR2
- added U1244: GT115, symbol Raki_ASIC_cells:NOR2
- added U1245, U1247, U1251, U1252, U1292, U1295: NOR2, symbol Raki_ASIC_cells:NOR2
- added U1246: GT116, symbol Raki_ASIC_cells:NOR2
- added U1248: GT117, symbol Raki_ASIC_cells:NOR3
- added U1250: GT118, symbol Raki_ASIC_cells:NOR2
- added U1253: GT119, symbol Raki_ASIC_cells:NOR2
- added U1256: GT121, symbol Raki_ASIC_cells:NOR2
- added U1257: GT120, symbol Raki_ASIC_cells:OR3
- added U1261: GT123, symbol Raki_ASIC_cells:NOR3
- added U1264: GT122, symbol Raki_ASIC_cells:OR4
- added U1291: GT124, symbol Raki_ASIC_cells:NOR2
- added U1294: GT125, symbol Raki_ASIC_cells:NOR2
- added U1297, U1300: BUF, symbol Raki_ASIC_cells:BUF
- added U1306: GT126, symbol Raki_ASIC_cells:NOR2
- added U1307: GT127, symbol Raki_ASIC_cells:INVP
- added U1309: GT128, symbol Raki_ASIC_cells:NOR3
- added U1310: GT129, symbol Raki_ASIC_cells:NOR2
- added U1313: GT130, symbol Raki_ASIC_cells:NOR2
- added U1315: GT131, symbol Raki_ASIC_cells:NOR3
- added U1316: GT132, symbol Raki_ASIC_cells:VY_DDL_small
- added U1317: GT134, symbol Raki_ASIC_cells:NAND2
- added U1318: GT133, symbol Raki_ASIC_cells:NOR2
- added U1322: GT135, symbol Raki_ASIC_cells:NAND2P2
- added U1323: GT136, symbol Raki_ASIC_cells:NOR2
- added U1326: GT137, symbol Raki_ASIC_cells:NOR2
- added U1328: GT139, symbol Raki_ASIC_cells:INV
- added U1336: GT138, symbol Raki_ASIC_cells:INVP
- added U1339: GT144, symbol Raki_ASIC_cells:NAND2
- added U1340: GT140, symbol Raki_ASIC_cells:INV
- added U1341: GT141, symbol Raki_ASIC_cells:INV
- added U1342: GT142, symbol Raki_ASIC_cells:INV
- added U1343: GT143, symbol Raki_ASIC_cells:INV
- U1095: value GT079 -> GT102
- U1097: value GT082 -> DL
- U1098: value INV -> GT082
- renumbered U143 to U1039, U143 to U1040, U143 to U1042, U143 to U1043, U143 to U1045, U143 to U1046, U143 to U1048, U143 to U1049, U143 to U1060, U143 to U1061, U143 to U1062, U143 to U1063, U143 to U1064, U143 to U1065, U143 to U1066, U143 to U1067, U143 to U1083, U143 to U1111, U143 to U1112, U145 to U686, U145 to U690, U145 to U790, U145 to U791, U145 to U799, U145 to U800, U145 to U801, U145 to U802, U145 to U803, U143 to U815, U143 to U816, U143 to U818, U143 to U820, U143 to U927, U142 to U929, U143 to U930, U143 to U931, U143 to U938, U143 to U939
Connections:
- net NET.PLA0.M16CYC11_Z is gone; now on net NET.PLA0.M16CYC10_Z: U978.
- net NET.PLA0.M16CYC8_Z is gone; now on net NET.PLA0.M16CYC10_Z: U986.
- net NET.PLA0.M16CYC9_Z is gone; now on net NET.PLA0.M16CYC10_Z: U988.
- net NET.PLA0.M8CYC0_Z is gone; now on net NET.PLA0.M16CYC10_Z: U949.
- net NET.PLA0.M8CYC1_Z is gone; now on net NET.PLA0.M16CYC10_Z: U1015., U1019., U952.
- net NET.PLA0.M8CYC2_Z is gone; now on net NET.PLA0.M16CYC10_Z: U1015., U1019., U954.
- net NET.PLA0.M8CYC3_Z is gone; now on net NET.PLA0.M16CYC10_Z: U1014., U1015., U956.
- net NET.PLA0.M8CYC4_Z is gone; now on net NET.PLA0.M16CYC10_Z: U1015., U960.
- net NET.PLA0.M8CYC5_Z is gone; now on net NET.PLA0.M16CYC10_Z: U1015., U1019., U964.
- net NET.PLA0.M8CYC6_Z is gone; now on net NET.PLA0.M16CYC10_Z: U1015., U1019., U968.
- net NET.PLA0.M8CYC7_Z is gone; now on net NET.PLA0.M16CYC10_Z: U1014., U972.
- net CLK.phiL: now also U1182., U1184., U1186., U1187., U1188., U1210., U1212., U1214., U1216., U1218., U1220., U1222.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
- net CLK.~{phiL}: now also U1196. (Φ1), U1197. (Φ1), U1199. (Φ1), U1202. (Φ1), U1203. (Φ1), U1204. (Φ1), U1208. (Φ1), U1293. (Φ1), U1308. (Φ1), U1311. (Φ1), U1312. (Φ1), U1314. (Φ1)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
- net GND: now also U1321. (Φ1)
- net NET.GT082: now also U1140., U1255., U1309., U1326.
- net NET.GT083: now also U1261., U1264.
- net NET.PLA.CNTR.D_{3}_Z: now also U1125.
- net NET.PLA0.M16CYC10_Z: now also U1127., U1128., U1129., U1130., U1131., U1132., U1133., U1134., U1135., U1136., U1137., U1138.
- net NET.REG_d1.D_{6}: now also U1254., U1260., U1262.
- net NET.REG_d8.D_{4}: now also U1257.
- net NET.GT058: now reaches U1123.
- net NET.GT058: now also U1086., U1087., U1088., U1122., U1124., U1135., U1140., U1141., U1145., U1169., U1170., U1171.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; no longer U1114.
- net NET.GT041: now reaches U876.
- net NET.GT041: now also U1017., U1020., U1022., U1023., U1024., U1025., U1026., U1027., U1028., U1029., U1030., U1084.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; no longer U966.
- net at U809.: now also U924. (Φ2); no longer U933. (Φ2)
- net at U831.: now also U832., U833., U839. (Φ1); no longer U830. (Φ1)
- net at U813.: now also U933. (Φ2); no longer U934. (Φ2)
- net at U808.: now also U936. (Φ2); no longer U934. (Φ2)
- net at U1016.: no longer U1013.
- net at U1100.: now also U1102.; no longer U1101.
- net NET.GT081: now reaches U1096.
- net NET.GT081: now also U1089. (Φ1), U1095., U1190.
- net at U821.: now also U822. (Φ1); no longer U823. (Φ1)
- removed net NET.PLA.CNTR.D_{0}: U1020., U1022., U1023., U1024., U1025., U1026., U1027., U1028., U1029., U1030., U1119., U686. (~{DOUT})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
- removed net NET.PLA.CNTR.D_{0}_Z: U1017., U991.
- new net: U1283., U1284.
- new net: U1283., U1302.
- new net: U1304., U1337., U1339.
- new net: U1212., U1213.
- new net: U1095., U1142., U1143., U1144., U1145., U1146., U1147., U1148., U1149., U1150., U1151., U1152.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
- new net: U1114., U1115., U1121.
- new net: U1114., U1119., U1120., U1261., U1264.
- new net: U1114., U1123.
- new net: U1114., U1116.
- new net: U1271., U1272.
- new net: U1271., U1296.
- new net: U1111., U1112.
- new net: U1111., U1112., U1113. (Φ1)
- new net: U876., U966.
- new net: U965., U966.
- new net: U865., U937.
- new net: U1121., U1258., U1309., U1323.
- new net: U1309., U1312. (Φ1)
- new net: U1216., U1217.
- new net: U818., U820., U925. (Φ1)
- new net: U1208. (Φ1), U1209.
- new net: U1207., U1208. (Φ1)
- new net: U1033., U886.
- new net: U1093., U905.
- new net: U943., U944.
- new net: U868., U944.
- new net: U1260., U1264.
- new net: U1004., U877.
- new net: U1042., U1043.
- new net: U1042., U1043., U1044. (Φ1)
- new net: U981., U982.
- new net: U1056., U892.
- new net: U1179., U1181.
- new net: U959., U960.
- new net: U1052., U889.
- new net: U953., U954.
- new net: U1079. (Φ2), U1086., U1087.
- new net: U1083., U1087.
- new net: U1070., U1087., U1088.
- new net: U1104., U1105.
- new net: U873., U958.
- new net: U957., U958.
- new net: U1294., U1295., U1324. (Φ1)
- new net: U808., U809., U810., U813., U824. (Φ1), U825. (Φ1)
- new net: U809., U933. (Φ2)
- new net: U809., U926. (Φ2)
- new net: U1242., U1243., U1306., U1307.
- new net: U1005., U1006.
- new net: U1054., U890.
- new net: U878., U970.
- new net: U1224., U1225.
- new net: U1298., U1335.
- new net: U1273., U1298.
- new net: U1265., U1266.
- new net: U1246., U1247.
- new net: U1246., U1247., U1310.
- new net: U1167., U1168., U1169., U1170., U1171., U1176.
- new net: U973., U974.
- new net: U1092., U904.
- new net: U1039., U1040.
- new net: U1039., U1040., U1041. (Φ1)
- new net: U1289., U1290.
- new net: U1060., U1061., U1069.
- new net: U1060., U1061.
- new net: U830. (Φ1), U831.
- new net: U807., U829. (Φ1), U830. (Φ1)
- new net: U1074., U896.
- new net: U1045., U1046.
- new net: U1045., U1046., U1047. (Φ1)
- new net: U947., U948.
- new net: U1048., U1049., U1050. (Φ1)
- new net: U1301., U1331.
- new net: U1281., U1301.
- new net: U1178., U1183.
- new net: U1255., U1257.
- new net: U821., U828., U926. (Φ2)
- new net: U828., U829. (Φ1)
- new net: U813., U934. (Φ2)
- new net: U808., U934. (Φ2)
- new net: U963., U964.
- new net: U1244., U1245.
- new net: U1296., U1334.
- new net: U1315., U1316. (Φ1)
- new net: U1316. (Φ1), U1322.
- new net: U871., U948.
- new net: U1236., U1237.
- new net: U823. (Φ1), U826., U834. (Φ1), U929.
- new net: U929., U931.
- new net: U843., U929., U931.
- new net: U1115., U1122.
- new net: U1115., U1117.
- new net: U1291., U1292.
- new net: U1291., U1292., U1293. (Φ1)
- new net: U1220., U1221.
- new net: U1013., U1016.
- new net: U1013., U1015.
- new net: U1062., U1063., U1069.
- new net: U1068., U1069., U1070., U1071.
- new net: U1218., U1219.
- new net: U1240., U1241.
- new net: U1197. (Φ1), U1201.
- new net: U1196. (Φ1), U1201.
- new net: U815., U816.
- new net: U815., U816., U817. (Φ1)
- new net: U1057., U893.
- new net: U1006., U880.
- new net: U1281., U1282.
- new net: U1101., U912.
- new net: U1100., U1101.
- new net: U955., U956.
- new net: U1285., U1286.
- new net: U863., U921.
- new net: U1248., U1249., U1313., U1315.
- new net: U1248., U1249.
- new net: U1300., U1330.
- new net: U870., U998.
- new net: U861., U919.
- new net: U971., U972.
- new net: U879., U982.
- new net: U1012., U1014.
- new net: U1012., U1016.
- new net: U867., U941.
- new net: U1214., U1215.
- new net: U1226., U1227.
- new net: U1289., U1305.
- new net: U927., U930., U935. (Φ1)
- new net: U1182., U1185.
- new net: U1118., U1119.
- new net: U1287., U1288.
- new net: U1256., U1258.
- new net: U1200., U1206., U1207.
- new net: U1279., U1280.
- new net: U995., U996.
- new net: U983., U984.
- new net: U1325. (Φ1), U1326.
- new net: U1303., U1333.
- new net: U1285., U1303.
- new net: U969., U970.
- new net: TP?.1, U661. (Φ1), U799. (~{DOUT})
- new net: U993., U994.
- new net: U1252., U1253., U1320. (Φ1)
- new net: U1097. (~{Q}), U1098.
- new net: U1299., U1329.
- new net: U1277., U1299.
- new net: U979., U980.
- new net: U1059., U895.
- new net: U862., U920.
- new net: TP?.1, U661. (Φ1), U687., U689., U792., U793.
- new net: U791. (~{DOUT}), U793.
- new net: U1165., U1184.
- new net: U1269., U1270.
- new net: U882., U994.
- new net: U1078., U1079. (Φ2), U1085.
- new net: U818., U820.
- new net: U821., U823. (Φ1)
- new net: U825. (Φ1), U826., U827. (Φ1)
- new net: U661. (Φ1), U799. (~{DOUT}), U800. (~{DOUT}), U801. (~{DOUT}), U802. (~{DOUT}), U803. (~{DOUT})
- new net: U803. (~{DOUT}), U804.
- new net: U802. (~{DOUT}), U803. (~{DOUT})
- new net: U1031., U884.
- new net: U1071., U1088.
- new net: U807., U824. (Φ1), U826.
- new net: U1073., U1077.
- new net: U812., U915.
- new net: U857., U915.
- new net: U1095., U1180.
- new net: U1019., U1021.
- new net: U1254., U1257.
- new net: U1076., U1078., U1080. (Φ2)
- new net: U842. (Φ1), U843.
- new net: U949., U950.
- new net: U869., U946.
- new net: U945., U946.
- new net: U1242., U1243.
- new net: U1181., U1186.
- new net: U687., U689., U796., U797., U798., U804., U840. (Φ1)
- new net: U827. (Φ1), U831., U832., U840. (Φ1)
- new net: U1234., U1235.
- new net: U1302., U1332.
- new net: U1082., U901.
- new net: U874., U962.
- new net: U1110., U908.
- new net: U1230., U1231.
- new net: U1166., U1182.
- new net: U807., U838. (Φ1)
- new net: U1002., U875.
- new net: U797., U801. (~{DOUT})
- new net: U801. (~{DOUT}), U802. (~{DOUT})
- new net: U800. (~{DOUT}), U801. (~{DOUT})
- new net: U661. (Φ1), U686. (~{DOUT}), U690. (~{DOUT}), U790. (~{DOUT}), U791. (~{DOUT})
- new net: U686. (~{DOUT}), U690. (~{DOUT})
- new net: U690. (~{DOUT}), U790. (~{DOUT})
- new net: U860., U918.
- new net: U1071., U1080. (Φ2)
- new net: U1275., U1276.
- new net: U661. (Φ1), U795., U796., U797., U798., U804.
- new net: U1222., U1223.
- new net: U1287., U1304.
- new net: U1188., U1189.
- new net: U1238., U1239.
- new net: U1099., U1103. (Φ1)
- new net: U961., U962.
- new net: U1109., U907.
- new net: U1279., U1300.
- new net: U938., U939., U940. (Φ1)
- new net: U661. (Φ1), U836.
- new net: U1062., U1063.
- new net: U866., U942.
- new net: U807., U819. (Φ1)
- new net: U810., U819. (Φ1)
- new net: U864., U922.
- new net: U1066., U1067.
- new net: U1275., U1297.
- new net: U1297., U1327.
- new net: U997., U998.
- new net: U1091., U903.
- new net: U1206., U1210.
- new net: U831., U832., U841. (Φ1)
- new net: U1305., U1338., U1339.
- new net: U977., U978.
- new net: U1318., U1319. (Φ1)
- new net: U1313., U1314. (Φ1)
- new net: U1090., U902.
- new net: U1081., U1082.
- new net: U858., U916.
- new net: U989., U991.
- new net: U927., U930.
- new net: U1294., U1295.
- new net: U1310., U1311. (Φ1)
- new net: U1261., U1262.
- new net: U1228., U1229.
- new net: U1267., U1268.
- new net: U1202. (Φ1), U1211.
- new net: U1259., U1263.
- new net: U661. (Φ1), U832.
- new net: U1183., U1187.
- new net: U975., U976.
- new net: U1252., U1253.
- new net: U883., U996.
- new net: U985., U986.
- new net: U1058., U894.
- new net: U914., U923.
- new net: U856., U914.
- new net: U1072., U897.
- new net: U1232., U1233.
- new net: U1034., U887.
- new net: U1064., U1065., U1070.
- new net: U1064., U1065.
- new net: U967., U968.
- new net: U1003., U1004.
- new net: U938., U939.
- new net: U1001., U1002.
- new net: U1204. (Φ1), U1205.
- new net: U1032., U885.
- new net: U990., U992.
- new net: U1317., U1321. (Φ1)
- new net: U1055., U891.
- new net: U1198., U1203. (Φ1)
- new net: U859., U917.
- new net: U799. (~{DOUT}), U800. (~{DOUT})
- new net: U1200., U1202. (Φ1)
- new net: U1273., U1274.
- new net: U1250., U1251., U1318.
- new net: U1051., U888.
- new net: U1277., U1278.
- new net: U833., U835. (Φ1)
- new net: U835. (Φ1), U932.
- new net: U790. (~{DOUT}), U792.
- new net: U790. (~{DOUT}), U791. (~{DOUT})
- new net: U837., U913.
- new net: U853., U913.
- new net: U951., U952.
- new net: U987., U988.
- new net: U1073., U898.
- new net: U1317., U1322.
- new net: U1306., U1308. (Φ1)
- new net: U1000., U999.
- new net: U1000., U872.
- new net: U1094., U906.
- new net: U928., U942.
- new net: U1250., U1251.
- new net: U881., U984.
- new net NET.GMODE_00001_T1: U899.
- new net NET.GMODE_01000_G3: U1173.
- new net NET.GMODE_01001_T2: U899.
- new net NET.GMODE_01100_G4: U1172., U1173.
- new net NET.GMODE_10000_G5: U1172., U1173.
- new net NET.GMODE_10100_G6: U1172., U1173., U1174.
- new net NET.GMODE_11100_G7: U1172., U1173., U1174.
- new net NET.GT075: U1085., U1168., U1175.
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Other:
- note added: "NET.GT041"
- note added: "NET.GT055"
- note added: "NET.GT056"
- note added: "NET.GT057"
- note added: "NET.GT058"
- note added: "NET.GT060"
- note added: "NET.GT082"
- note added: "NET.GT091"
- note added: "NET.GT092"
- note added: "NET.GT093"
- note added: "NET.PLA.~{TMODE}"
- note added: "NET.PLA1.CNTR.D_{0}_Z"
- note added: "NET.PLA1.CNTR.D_{3}_Z"
- note added: "NET.PLA1.CNTR.~{D_{0}}_Z"
- note added: "NET.PLA1.CNTR.~{D_{3}}_Z"
- note added: "NET.PLA1.CYCDEC_A"
- note added: "NET.PLA1.CYCDEC_B"
- note added: "NET.PLA1.CYCDEC_C"
- note added: "NET.PLA1.CYCDEC_D"
- note added: "NET.PLA1.CYCDEC_E"
- note added: "NET.PLA1.CYCDEC_F"
- note added: "NET.PLA1.CYCDEC_G"
- note added: "NET.PLA1.CYCDEC_H"
- note added: "NET.PLA1.CYCDEC_I"
- note added: "NET.PLA1.CYCDEC_J"
- note added: "NET.PLA1.CYCDEC_K"
- note added: "NET.PLA1.CYCDEC_L"
- note added: "NET.~{GT041}"
- note added: "NET.~{GT082}"
- note added: "NET.~{GT093}"
- note added: "OR-AND ARRAY"
- note added: "PLA1"
- note added: "phiLp"
- note added: "source signals are latched by phiL"

Commit message: update 20251028
Parts:
- added U1660: GT145, symbol Raki_ASIC_cells:VY_DSR_small
Connections:
- net CLK.phiL: now also U1660. (Φ2)
- net CLK.~{phiL}: now also U1660. (Φ2)
- net NET.GT041: now also U1044. (Φ1)
- net NET.GT055: now also U1041. (Φ1)
- net NET.GT057: now also U1047. (Φ1)
- net NET.GT058: now also U1050. (Φ1)
- net NET.GT060: now also U1053. (Φ1)
- net NET.PLA2.COL_{29}: now also U1660. (Φ2)
- net at U1284.: no longer U1283.
- net at U1302.: now also U1332.; no longer U1283.
- net at U1213.: now also U1212.
- net at U1163.: now also U1095., U1142., U1143., U1144., U1145., U1146., U1147., U1148., U1149., U1150., U1151., U1152., U1153., U1154., U1155., U1156., U1157., U1158., U1159., U1160., U1161., U1162., U1164., U1178., U1179., U1180.
- net at U1272.: no longer U1271.
- net at U1296.: now also U1334.; no longer U1271.
- net at U1217.: no longer U1216.
- net at U809.: now also U924. (Φ2); no longer U933. (Φ2)
- net at U1307.: now also U1242., U1243., U1306.
- net at U1225.: no longer U1224.
- net at U1298.: now also U1273.; no longer U1335.
- net at U1266.: no longer U1265.
- net at U1290.: now also U1289.
- net at U831.: now also U832., U833., U839. (Φ1); no longer U830. (Φ1)
- net at U1301.: now also U1281.; no longer U1331.
- net at U813.: now also U933. (Φ2); no longer U934. (Φ2)
- net at U808.: now also U936. (Φ2); no longer U934. (Φ2)
- net at U1237.: now also U1236.
- net at U1221.: no longer U1220.
- net at U1016.: no longer U1013.
- net at U1219.: no longer U1218.
- net at U1241.: no longer U1240.
- net at U1282.: now also U1281.
- net at U1100.: now also U1102.; no longer U1101.
- net at U1286.: now also U1285.
- net at U1300.: now also U1279.; no longer U1330.
- net at U1215.: no longer U1214.
- net at U1227.: no longer U1226.
- net at U1305.: now also U1338., U1339.; no longer U1289.
- net at U1288.: now also U1287.
- net NET.GC103: now reaches U1258.
- net NET.GC103: now also U1121., U1309., U1323.; no longer U1256.
- net at U1280.: now also U1279.
- net NET.GC106: now reaches U1121., U1264.
- net at U1303.: now also U1285.; no longer U1333.
- net at U1097. (~{Q}): now also U1099.; no longer U1098.
- net at U1299.: now also U1277.; no longer U1329.
- net at U1165.: no longer U1184.
- net at U1270.: now also U1269.
- net at U821.: now also U822. (Φ1); no longer U823. (Φ1)
- net NET.ST.HADD.~{EQ23}: now reaches U825. (Φ1)
- net NET.ST.HADD.~{EQ23}: now also U826., U827. (Φ1)
- net at U804.: now also TP?.1, U689., U795., U797., U798., U839. (Φ1); no longer U803. (~{DOUT})
- net at U1071.: now also U1066., U1067.; no longer U1088.
- net NET.ST.VPLA.COL_{27}: now reaches U1099.
- net NET.ST.VPLA.COL_{27}: no longer U1097. (~{Q})
- net at U843.: now also U900.; no longer U842. (Φ1)
- net at U1235.: no longer U1234.
- net at U1231.: no longer U1230.
- net at U1166.: no longer U1182.
- net at U807.: now also U806.; no longer U838. (Φ1)
- net at U1276.: now also U1275.
- net at U1223.: no longer U1222.
- net at U1189.: now also U1188.
- net at U1239.: now also U1238.
- net at U836.: now also U831.; no longer U661. (Φ1)
- net at U810.: now also U936. (Φ2); no longer U819. (Φ1)
- net at U1297.: now also U1327.; no longer U1275.
- net at U1229.: no longer U1228.
- net at U1268.: no longer U1267.
- net at U1263.: now also U1259.
- net at U1233.: now also U1232.
- net at U1205.: now also U1204. (Φ1)
- net at U1274.: now also U1273.
- net at U806.: now also U661. (Φ1); no longer U807.
- net at U1278.: now also U1277.
- net at U833.: now also U834. (Φ1); no longer U835. (Φ1)
- new net: U1283., U1284.
- new net: U1283., U1302.
- new net: U1304., U1337., U1339.
- new net: U1114., U1115., U1121.
- new net: U1114., U1119., U1120., U1261., U1264.
- new net: U1114., U1123.
- new net: U1114., U1116.
- new net: U1271., U1272.
- new net: U1271., U1296.
- new net: U1111., U1112.
- new net: U1111., U1112., U1113. (Φ1)
- new net: U876., U966.
- new net: U965., U966.
- new net: U1310., U1311. (Φ1)
- new net: U865., U937.
- new net: U1309., U1312. (Φ1)
- new net: U1216., U1217.
- new net: U818., U820., U925. (Φ1)
- new net: U1208. (Φ1), U1209.
- new net: U1207., U1208. (Φ1)
- new net: U1033., U886.
- new net: U1093., U905.
- new net: U943., U944.
- new net: U868., U944.
- new net: U1260., U1264.
- new net: U1004., U877.
- new net: U1042., U1043.
- new net: U1042., U1043., U1044. (Φ1)
- new net: U981., U982.
- new net: U1056., U892.
- new net: U959., U960.
- new net: U1052., U889.
- new net: U953., U954.
- new net: U1079. (Φ2), U1086., U1087.
- new net: U1083., U1087.
- new net: U1070., U1087., U1088.
- new net: U1104., U1105.
- new net: U873., U958.
- new net: U957., U958.
- new net: U1294., U1295., U1324. (Φ1)
- new net: U808., U809., U810., U813., U824. (Φ1), U825. (Φ1)
- new net: U809., U933. (Φ2)
- new net: U809., U926. (Φ2)
- new net: U1005., U1006.
- new net: U1054., U890.
- new net: U878., U970.
- new net: U1224., U1225.
- new net: U1298., U1335.
- new net: U1265., U1266.
- new net: U1246., U1247.
- new net: U1246., U1247., U1310.
- new net: U1167., U1168., U1169., U1170., U1171., U1176.
- new net: U973., U974.
- new net: U1092., U904.
- new net: U1039., U1040.
- new net: U1039., U1040., U1041. (Φ1)
- new net: U1060., U1061., U1069.
- new net: U1060., U1061.
- new net: U830. (Φ1), U831.
- new net: U807., U829. (Φ1), U830. (Φ1)
- new net: U1074., U896.
- new net: U1045., U1046.
- new net: U1045., U1046., U1047. (Φ1)
- new net: U947., U948.
- new net: U1048., U1049., U1050. (Φ1)
- new net: U1301., U1331.
- new net: U1255., U1257.
- new net: U821., U828., U926. (Φ2)
- new net: U828., U829. (Φ1)
- new net: U813., U934. (Φ2)
- new net: U808., U934. (Φ2)
- new net: U963., U964.
- new net: U1244., U1245.
- new net: U1315., U1316. (Φ1)
- new net: U1316. (Φ1), U1322.
- new net: U871., U948.
- new net: U823. (Φ1), U826., U834. (Φ1), U929.
- new net: U929., U931.
- new net: U843., U929., U931.
- new net: U1115., U1122.
- new net: U1115., U1117.
- new net: U1291., U1292.
- new net: U1291., U1292., U1293. (Φ1)
- new net: U1220., U1221.
- new net: U1013., U1016.
- new net: U1013., U1015.
- new net: U1062., U1063., U1069.
- new net: U1068., U1069., U1070., U1071.
- new net: U1218., U1219.
- new net: U1240., U1241.
- new net: U1197. (Φ1), U1201.
- new net: U1196. (Φ1), U1201.
- new net: U815., U816.
- new net: U815., U816., U817. (Φ1)
- new net: U1057., U893.
- new net: U1006., U880.
- new net: U1101., U912.
- new net: U1100., U1101.
- new net: U955., U956.
- new net: U863., U921.
- new net: U1248., U1249., U1313., U1315.
- new net: U1248., U1249.
- new net: U1300., U1330.
- new net: U870., U998.
- new net: U861., U919.
- new net: U971., U972.
- new net: U879., U982.
- new net: U1012., U1014.
- new net: U1012., U1016.
- new net: U867., U941.
- new net: U1214., U1215.
- new net: U1226., U1227.
- new net: U1289., U1305.
- new net: U927., U930., U935. (Φ1)
- new net: U1182., U1185.
- new net: U1118., U1119.
- new net: U1256., U1258.
- new net: U1200., U1206., U1207.
- new net: U995., U996.
- new net: U983., U984.
- new net: U1325. (Φ1), U1326.
- new net: U1303., U1333.
- new net: U969., U970.
- new net: TP?.1, U661. (Φ1), U799. (~{DOUT})
- new net: U993., U994.
- new net: U1097. (~{Q}), U1098.
- new net: U1299., U1329.
- new net: U979., U980.
- new net: U1059., U895.
- new net: U862., U920.
- new net: TP?.1, U661. (Φ1), U687., U689., U792., U793.
- new net: U791. (~{DOUT}), U793.
- new net: U1165., U1184.
- new net: U882., U994.
- new net: U1078., U1079. (Φ2), U1085.
- new net: U818., U820.
- new net: U821., U823. (Φ1)
- new net: U661. (Φ1), U799. (~{DOUT}), U800. (~{DOUT}), U801. (~{DOUT}), U802. (~{DOUT}), U803. (~{DOUT})
- new net: U803. (~{DOUT}), U804.
- new net: U802. (~{DOUT}), U803. (~{DOUT})
- new net: U1031., U884.
- new net: U1071., U1088.
- new net: U807., U824. (Φ1), U826.
- new net: U1073., U1077.
- new net: U812., U915.
- new net: U857., U915.
- new net: U1019., U1021.
- new net: U1254., U1257.
- new net: U1076., U1078., U1080. (Φ2)
- new net: U842. (Φ1), U843.
- new net: U949., U950.
- new net: U869., U946.
- new net: U945., U946.
- new net: U1242., U1243.
- new net: U687., U689., U796., U797., U798., U804., U840. (Φ1)
- new net: U827. (Φ1), U831., U832., U840. (Φ1)
- new net: U1234., U1235.
- new net: U1082., U901.
- new net: U874., U962.
- new net: U1110., U908.
- new net: U1230., U1231.
- new net: U1166., U1182.
- new net: U807., U838. (Φ1)
- new net: U1002., U875.
- new net: U797., U801. (~{DOUT})
- new net: U801. (~{DOUT}), U802. (~{DOUT})
- new net: U800. (~{DOUT}), U801. (~{DOUT})
- new net: U661. (Φ1), U686. (~{DOUT}), U690. (~{DOUT}), U790. (~{DOUT}), U791. (~{DOUT})
- new net: U686. (~{DOUT}), U690. (~{DOUT})
- new net: U690. (~{DOUT}), U790. (~{DOUT})
- new net: U860., U918.
- new net: U1071., U1080. (Φ2)
- new net: U661. (Φ1), U795., U796., U797., U798., U804.
- new net: U1222., U1223.
- new net: U1099., U1103. (Φ1)
- new net: U961., U962.
- new net: U1317., U1321. (Φ1)
- new net: U1109., U907.
- new net: U938., U939., U940. (Φ1)
- new net: U661. (Φ1), U836.
- new net: U1062., U1063.
- new net: U866., U942.
- new net: U807., U819. (Φ1)
- new net: U810., U819. (Φ1)
- new net: U1313., U1314. (Φ1)
- new net: U864., U922.
- new net: U1066., U1067.
- new net: U1275., U1297.
- new net: U1318., U1319. (Φ1)
- new net: U997., U998.
- new net: U1091., U903.
- new net: U1206., U1210.
- new net: U831., U832., U841. (Φ1)
- new net: U977., U978.
- new net: U1090., U902.
- new net: U1081., U1082.
- new net: U858., U916.
- new net: U989., U991.
- new net: U927., U930.
- new net: U1294., U1295.
- new net: U1261., U1262.
- new net: U1228., U1229.
- new net: U1267., U1268.
- new net: U1202. (Φ1), U1211.
- new net: U661. (Φ1), U832.
- new net: U975., U976.
- new net: U1252., U1253.
- new net: U1252., U1253., U1320. (Φ1)
- new net: U883., U996.
- new net: U985., U986.
- new net: U1058., U894.
- new net: U914., U923.
- new net: U856., U914.
- new net: U1072., U897.
- new net: U1034., U887.
- new net: U1064., U1065., U1070.
- new net: U1064., U1065.
- new net: U967., U968.
- new net: U1003., U1004.
- new net: U938., U939.
- new net: U1001., U1002.
- new net: U1032., U885.
- new net: U990., U992.
- new net: U1055., U891.
- new net: U1198., U1203. (Φ1)
- new net: U859., U917.
- new net: U799. (~{DOUT}), U800. (~{DOUT})
- new net: U1200., U1202. (Φ1)
- new net: U1250., U1251., U1318.
- new net: U1051., U888.
- new net: U833., U835. (Φ1)
- new net: U835. (Φ1), U932.
- new net: U790. (~{DOUT}), U792.
- new net: U790. (~{DOUT}), U791. (~{DOUT})
- new net: U837., U913.
- new net: U853., U913.
- new net: U951., U952.
- new net: U987., U988.
- new net: U1073., U898.
- new net: U1317., U1322.
- new net: U1306., U1308. (Φ1)
- new net: U1000., U999.
- new net: U1000., U872.
- new net: U1094., U906.
- new net: U928., U942.
- new net: U1250., U1251.
- new net: U881., U984.
- new net NET.GT145: U1660. (Φ2)
- now unconnected: U1016., U1113. (Φ1), U1146., U1147., U1148., U1149., U1150., U1151., U1152., U1153., U1154., U1155., U1156., U1157., U1158., U1159., U1160., U1161., U1162., U1164.
- no-connect marks 328 -> 329
Other:
- note removed: "EXT"
- note removed: "EXT PLA"
- moved on the sheet: TP?

Commit message: update 20251106
Parts:
- removed U1097: DL, symbol Raki_ASIC_cells:DLNE
- added U1702: DLNE, symbol Raki_ASIC_cells:DLNE
Connections:
- net NET.GT055 is gone; now on net NET.GT041: U1041. (Φ1)
- net NET.GT057 is gone; now on net NET.GT041: U1047. (Φ1)
- net NET.GT060 is gone; now on net NET.PLA0.~{COL_{29}}: U1053. (Φ1)
- net NET.PLA.~{GMODE34567} is gone; now on net NET.GT041: U1173.
- net NET.GC103: no longer U1309.
- net NET.GT041: now also U1012., U1018., U1021., U1050. (Φ1), U1053. (Φ1), U1085., U1086., U1087., U1088., U1098., U1104., U1122., U1123., U1124., U1125., U1127., U1128., U1131., U1132., U1133., U1134., U1135., U1136., U1137., U1138., U1140., U1141., U1145., U1146., U1147., U1148., U1149., U1150., U1151., U1152., U1153., U1154., U1155., U1156., U1157., U1158., U1159., U1160., U1161., U1162., U1163., U1164., U1165., U1166., U1168., U1169., U1170., U1171., U1172., U1174., U1177., U1190., U1200., U1206., U1255., U1256., U1309., U1326., U992.
- net at U1284.: no longer U1283.
- net at U1302.: now also U1332.; no longer U1283.
- net at U1213.: now also U1212.
- net at U1272.: no longer U1271.
- net at U1296.: now also U1334.; no longer U1271.
- net at U1217.: no longer U1216.
- net at U809.: now also U924. (Φ2); no longer U933. (Φ2)
- net at U1307.: now also U1242., U1243., U1306.
- net at U1225.: no longer U1224.
- net at U1298.: now also U1273.; no longer U1335.
- net at U1266.: no longer U1265.
- net at U1290.: now also U1289.
- net at U831.: now also U832., U833., U839. (Φ1); no longer U830. (Φ1)
- net at U1301.: now also U1281.; no longer U1331.
- net at U813.: now also U933. (Φ2); no longer U934. (Φ2)
- net at U808.: now also U936. (Φ2); no longer U934. (Φ2)
- net at U1237.: now also U1236.
- net at U1221.: no longer U1220.
- net at U1016.: no longer U1013.
- net at U1219.: no longer U1218.
- net at U1241.: no longer U1240.
- net at U1282.: now also U1281.
- net at U1100.: now also U1102.; no longer U1101.
- net at U1286.: now also U1285.
- net at U1300.: now also U1279.; no longer U1330.
- net NET.~{GT106}_Z: now reaches U1199. (Φ1)
- net at U1215.: no longer U1214.
- net at U1227.: no longer U1226.
- net at U1305.: now also U1338., U1339.; no longer U1289.
- net at U1288.: now also U1287.
- net at U1280.: now also U1279.
- net at U1303.: now also U1285.; no longer U1333.
- net at U1299.: now also U1277.; no longer U1329.
- net at U1270.: now also U1269.
- net at U821.: now also U822. (Φ1); no longer U823. (Φ1)
- net at U804.: now also TP?.1, U689., U795., U797., U798., U839. (Φ1); no longer U803. (~{DOUT})
- net at U1071.: now also U1066., U1067.; no longer U1088.
- net at U843.: now also U900.; no longer U842. (Φ1)
- net at U1235.: no longer U1234.
- net at U1231.: no longer U1230.
- net at U807.: now also U806.; no longer U838. (Φ1)
- net at U1276.: now also U1275.
- net at U1223.: no longer U1222.
- net at U1189.: now also U1188.
- net at U1239.: now also U1238.
- net at U836.: now also U831.; no longer U661. (Φ1)
- net at U810.: now also U936. (Φ2); no longer U819. (Φ1)
- net at U1297.: now also U1327.; no longer U1275.
- net at U1229.: no longer U1228.
- net at U1268.: no longer U1267.
- net at U1263.: now also U1259.
- net at U1233.: now also U1232.
- net NET.GT109: now reaches U1205.
- net at U1274.: now also U1273.
- net at U806.: now also U661. (Φ1); no longer U807.
- net at U1278.: now also U1277.
- net at U833.: now also U834. (Φ1); no longer U835. (Φ1)
- removed net NET.GT058: U1050. (Φ1), U1086., U1087., U1088., U1122., U1123., U1124., U1135., U1140., U1141., U1145., U1169., U1170., U1171., U1172., U1175., U1256.
- removed net NET.GT075: U1085., U1168., U1175.
- removed net NET.GT082: U1098., U1104., U1140., U1255., U1309., U1326.
- removed net NET.PLA.CNTR.D_{3}_Z: U1012., U1018., U1021., U1125., U992.
- removed net NET.PLA.~{GMODE67}: U1174., U1200., U1206.
- removed net NET.PLA1.CYCDEC_K: U1128., U1177.
- new net: U1283., U1284.
- new net: U1283., U1302.
- new net: U1304., U1337., U1339.
- new net: U1095., U1142., U1143., U1144., U1145., U1146., U1147., U1148., U1149., U1150., U1151., U1152., U1153., U1154., U1155., U1156., U1157., U1158., U1159., U1160., U1161., U1162., U1163., U1164., U1178., U1179., U1180.
- new net: U1114., U1115., U1121.
- new net: U1114., U1119., U1120., U1261., U1264.
- new net: U1114., U1123.
- new net: U1114., U1116.
- new net: U1271., U1272.
- new net: U1271., U1296.
- new net: U1111., U1112.
- new net: U1111., U1112., U1113. (Φ1)
- new net: U876., U966.
- new net: U965., U966.
- new net: U1310., U1311. (Φ1)
- new net: U865., U937.
- new net: U1309., U1312. (Φ1)
- new net: U1216., U1217.
- new net: U818., U820., U925. (Φ1)
- new net: U1208. (Φ1), U1209.
- new net: U1207., U1208. (Φ1)
- new net: U1033., U886.
- new net: U1093., U905.
- new net: U943., U944.
- new net: U868., U944.
- new net: U1260., U1264.
- new net: U1004., U877.
- new net: U1042., U1043.
- new net: U1042., U1043., U1044. (Φ1)
- new net: U981., U982.
- new net: U1056., U892.
- new net: U959., U960.
- new net: U1052., U889.
- new net: U953., U954.
- new net: U1079. (Φ2), U1086., U1087.
- new net: U1083., U1087.
- new net: U1070., U1087., U1088.
- new net: U1104., U1105.
- new net: U873., U958.
- new net: U957., U958.
- new net: U1294., U1295., U1324. (Φ1)
- new net: U808., U809., U810., U813., U824. (Φ1), U825. (Φ1)
- new net: U809., U933. (Φ2)
- new net: U809., U926. (Φ2)
- new net: U1005., U1006.
- new net: U1054., U890.
- new net: U878., U970.
- new net: U1224., U1225.
- new net: U1298., U1335.
- new net: U1265., U1266.
- new net: U1246., U1247.
- new net: U1246., U1247., U1310.
- new net: U1167., U1168., U1169., U1170., U1171., U1176.
- new net: U973., U974.
- new net: U1092., U904.
- new net: U1039., U1040.
- new net: U1039., U1040., U1041. (Φ1)
- new net: U1060., U1061., U1069.
- new net: U1060., U1061.
- new net: U830. (Φ1), U831.
- new net: U807., U829. (Φ1), U830. (Φ1)
- new net: U1074., U896.
- new net: U1045., U1046.
- new net: U1045., U1046., U1047. (Φ1)
- new net: U947., U948.
- new net: U1048., U1049., U1050. (Φ1)
- new net: U1301., U1331.
- new net: U1255., U1257.
- new net: U821., U828., U926. (Φ2)
- new net: U828., U829. (Φ1)
- new net: U813., U934. (Φ2)
- new net: U808., U934. (Φ2)
- new net: U963., U964.
- new net: U1244., U1245.
- new net: U1315., U1316. (Φ1)
- new net: U1316. (Φ1), U1322.
- new net: U871., U948.
- new net: U823. (Φ1), U826., U834. (Φ1), U929.
- new net: U929., U931.
- new net: U843., U929., U931.
- new net: U1115., U1122.
- new net: U1115., U1117.
- new net: U1291., U1292.
- new net: U1291., U1292., U1293. (Φ1)
- new net: U1220., U1221.
- new net: U1013., U1016.
- new net: U1013., U1015.
- new net: U1062., U1063., U1069.
- new net: U1068., U1069., U1070., U1071.
- new net: U1218., U1219.
- new net: U1240., U1241.
- new net: U1197. (Φ1), U1201.
- new net: U1196. (Φ1), U1201.
- new net: U815., U816.
- new net: U815., U816., U817. (Φ1)
- new net: U1057., U893.
- new net: U1006., U880.
- new net: U1101., U912.
- new net: U1100., U1101.
- new net: U955., U956.
- new net: U863., U921.
- new net: U1248., U1249., U1313., U1315.
- new net: U1248., U1249.
- new net: U1300., U1330.
- new net: U870., U998.
- new net: U861., U919.
- new net: U971., U972.
- new net: U879., U982.
- new net: U1012., U1014.
- new net: U1012., U1016.
- new net: U867., U941.
- new net: U1214., U1215.
- new net: U1226., U1227.
- new net: U1289., U1305.
- new net: U927., U930., U935. (Φ1)
- new net: U1182., U1185.
- new net: U1118., U1119.
- new net: U1256., U1258.
- new net: U1200., U1206., U1207.
- new net: U995., U996.
- new net: U983., U984.
- new net: U1325. (Φ1), U1326.
- new net: U1303., U1333.
- new net: U969., U970.
- new net: TP?.1, U661. (Φ1), U799. (~{DOUT})
- new net: U993., U994.
- new net: U1098., U1702. (~{Q})
- new net: U1299., U1329.
- new net: U979., U980.
- new net: U1059., U895.
- new net: U862., U920.
- new net: TP?.1, U661. (Φ1), U687., U689., U792., U793.
- new net: U791. (~{DOUT}), U793.
- new net: U1165., U1184.
- new net: U882., U994.
- new net: U1078., U1079. (Φ2), U1085.
- new net: U818., U820.
- new net: U821., U823. (Φ1)
- new net: U661. (Φ1), U799. (~{DOUT}), U800. (~{DOUT}), U801. (~{DOUT}), U802. (~{DOUT}), U803. (~{DOUT})
- new net: U803. (~{DOUT}), U804.
- new net: U802. (~{DOUT}), U803. (~{DOUT})
- new net: U1031., U884.
- new net: U1071., U1088.
- new net: U807., U824. (Φ1), U826.
- new net: U1073., U1077.
- new net: U812., U915.
- new net: U857., U915.
- new net: U1099., U1702. (~{Q})
- new net: U1019., U1021.
- new net: U1254., U1257.
- new net: U1076., U1078., U1080. (Φ2)
- new net: U842. (Φ1), U843.
- new net: U949., U950.
- new net: U869., U946.
- new net: U945., U946.
- new net: U1242., U1243.
- new net: U687., U689., U796., U797., U798., U804., U840. (Φ1)
- new net: U827. (Φ1), U831., U832., U840. (Φ1)
- new net: U1234., U1235.
- new net: U1082., U901.
- new net: U874., U962.
- new net: U1110., U908.
- new net: U1230., U1231.
- new net: U1166., U1182.
- new net: U807., U838. (Φ1)
- new net: U1002., U875.
- new net: U797., U801. (~{DOUT})
- new net: U801. (~{DOUT}), U802. (~{DOUT})
- new net: U800. (~{DOUT}), U801. (~{DOUT})
- new net: U661. (Φ1), U686. (~{DOUT}), U690. (~{DOUT}), U790. (~{DOUT}), U791. (~{DOUT})
- new net: U686. (~{DOUT}), U690. (~{DOUT})
- new net: U690. (~{DOUT}), U790. (~{DOUT})
- new net: U860., U918.
- new net: U1071., U1080. (Φ2)
- new net: U661. (Φ1), U795., U796., U797., U798., U804.
- new net: U1222., U1223.
- new net: U1099., U1103. (Φ1)
- new net: U961., U962.
- new net: U1317., U1321. (Φ1)
- new net: U1109., U907.
- new net: U938., U939., U940. (Φ1)
- new net: U661. (Φ1), U836.
- new net: U1062., U1063.
- new net: U866., U942.
- new net: U807., U819. (Φ1)
- new net: U810., U819. (Φ1)
- new net: U1313., U1314. (Φ1)
- new net: U864., U922.
- new net: U1066., U1067.
- new net: U1275., U1297.
- new net: U1318., U1319. (Φ1)
- new net: U997., U998.
- new net: U1091., U903.
- new net: U1206., U1210.
- new net: U831., U832., U841. (Φ1)
- new net: U977., U978.
- new net: U1090., U902.
- new net: U1081., U1082.
- new net: U858., U916.
- new net: U989., U991.
- new net: U927., U930.
- new net: U1294., U1295.
- new net: U1261., U1262.
- new net: U1228., U1229.
- new net: U1267., U1268.
- new net: U1202. (Φ1), U1211.
- new net: U661. (Φ1), U832.
- new net: U975., U976.
- new net: U1252., U1253.
- new net: U1252., U1253., U1320. (Φ1)
- new net: U883., U996.
- new net: U985., U986.
- new net: U1058., U894.
- new net: U914., U923.
- new net: U856., U914.
- new net: U1072., U897.
- new net: U1034., U887.
- new net: U1064., U1065., U1070.
- new net: U1064., U1065.
- new net: U967., U968.
- new net: U1003., U1004.
- new net: U938., U939.
- new net: U1001., U1002.
- new net: U1204. (Φ1), U1205.
- new net: U1032., U885.
- new net: U990., U992.
- new net: U1055., U891.
- new net: U1198., U1203. (Φ1)
- new net: U859., U917.
- new net: U799. (~{DOUT}), U800. (~{DOUT})
- new net: U1200., U1202. (Φ1)
- new net: U1250., U1251., U1318.
- new net: U1051., U888.
- new net: U833., U835. (Φ1)
- new net: U835. (Φ1), U932.
- new net: U790. (~{DOUT}), U792.
- new net: U790. (~{DOUT}), U791. (~{DOUT})
- new net: U837., U913.
- new net: U853., U913.
- new net: U951., U952.
- new net: U987., U988.
- new net: U1073., U898.
- new net: U1317., U1322.
- new net: U1306., U1308. (Φ1)
- new net: U1000., U999.
- new net: U1000., U872.
- new net: U1094., U906.
- new net: U928., U942.
- new net: U1250., U1251.
- new net: U881., U984.
- now unconnected: U1016., U1113. (Φ1)
Other:
- note added: "COMMON PLA COUNTER"
- moved on the sheet: TP008, TP009, TP?
