File: resources/V9958_kicad/REG0.kicad_sch (KiCad schematic)
At the start: 281 parts, among them U100 GA042, U101 GA043, U102 DLPEN, U103 DLPEN, U104 GA044, U105 GA045, U106 GA047, U107 GA046, U108 INV, U109 GA048, U110 GA049, U111 INV, U112 GA051, U113 GA050, U114 GA052, U115 GA053, U116 GA054, U117 GA055, U118 GA056, U119 DLPRPEN, U119 GA057, U120 DLPRPEN, U120 GA058, U121 DLPRPEN, U121 GA059, U122 DLPRPEN, U122 INV, U123 DLPRPEN, U123 INV, U124 GA061, U125 GA060, U126 INV, U127 GA062, U128 GA063, U129 GA064, U130 GA065, U131 GA066, U132 GA067, U133 DLPRPEN, U133 GA068, U134 DLPRPEN, U134 GA069, U135 GA098, U136 INV, U137 INV, U138 INV, U139 GA070, U14 GA001, U140 GA073, U141 GA074, U142 GA071, U143 GA072, U144 INV, U145 VY_CONSTCNTR1, U146 VY_CONSTCNTR1, U148 VY_CONSTCNTR1, U149 VY_CONSTCNTR1, U15 DSR, U150 VY_CONSTCNTR1, U155 GA075, U156 GA076, U157 GA078, U158 GA077, U159 GA079, U160 GA080, U161 GA081, U162 NAND2OD, U162 VY_CONSTCNTR1, U163 NAND2OD, U164 GA082, U165 GA083, U166 DLPEN, U166 NAND2OD, U167 INV, U167 NAND2OD, U168 DLPEN, U168 NAND2OD, U169 GA085, U169 NAND2OD, U170 DLPEN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

Commit message: update 20240825
Parts:
- removed TP001: ~, symbol Connector:TestPoint
- removed U100: GA042, symbol Raki_ASIC_cells:NOR3
- removed U101: GA043, symbol Raki_ASIC_cells:VY_DSR_small
- removed U102, U103, U166, U168, U170, U171, U174, U175, U176, U177: DLPEN, symbol Raki_ASIC_cells:DLPEN
- removed U104: GA044, symbol Raki_ASIC_cells:AOI211
- removed U105: GA045, symbol Raki_ASIC_cells:AOI21
- removed U106: GA047, symbol Raki_ASIC_cells:NOR2
- removed U107: GA046, symbol Raki_ASIC_cells:NOR6
- removed U108, U111, U122, U123, U138, U167, U183, U265, U266, U268, U270, U272, U274, U276, U278, U75, U87, U88: INV, symbol Raki_ASIC_cells:INV
- removed U109: GA048, symbol Raki_ASIC_cells:AOI211
- removed U110: GA049, symbol Raki_ASIC_cells:AOI21
- removed U112: GA051, symbol Raki_ASIC_cells:NOR2
- removed U113: GA050, symbol Raki_ASIC_cells:NOR4
- removed U114: GA052, symbol Raki_ASIC_cells:NOR4
- removed U115: GA053, symbol Raki_ASIC_cells:NOR4
- removed U116: GA054, symbol Raki_ASIC_cells:NOR3
- removed U117: GA055, symbol Raki_ASIC_cells:NOR3
- removed U118: GA056, symbol Raki_ASIC_cells:NOR4
- removed U119: GA057, symbol Raki_ASIC_cells:NOR4
- removed U119, U120, U121, U122, U123, U133, U134, U329: DLPRPEN, symbol Raki_ASIC_cells:DLPRPEN
- removed U120: GA058, symbol Raki_ASIC_cells:NOR2
- removed U121: GA059, symbol Raki_ASIC_cells:NOR3
- removed U139: GA070, symbol Raki_ASIC_cells:NOR2
- removed U14: GA001, symbol Raki_ASIC_cells:AOI21
- removed U140: GA073, symbol Raki_ASIC_cells:VY_DSR_small
- removed U141: GA074, symbol Raki_ASIC_cells:VY_DSR_small
- removed U142: GA071, symbol Raki_ASIC_cells:NOR3
- removed U143: GA072, symbol Raki_ASIC_cells:NOR2
- removed U15, U84: DSR, symbol Raki_ASIC_cells:VY_DSR_small
- removed U162, U163, U166, U167, U168, U169, U264, U267, U269, U271, U273, U275, U277, U279: NAND2OD, symbol Raki_ASIC_cells:NAND2OD
- removed U169: GA085, symbol Raki_ASIC_cells:NOR3
- removed U182: GA084, symbol Raki_ASIC_cells:NOR2
- removed U184: GA086, symbol Raki_ASIC_cells:NOR4
- removed U185: GA087, symbol Raki_ASIC_cells:NOR4
- removed U186: GA088, symbol Raki_ASIC_cells:NOR3
- removed U187: GA097, symbol Raki_ASIC_cells:NOR2
- removed U190: GA095, symbol Raki_ASIC_cells:NOR2P
- removed U190: GA100, symbol Raki_ASIC_cells:NOR2P
- removed U218, U219, U220, U221, U223, U224, U226, U227, U228, U229, U230, U231, U234, U235, U236, U237, U238, U239, U240, U241, U242, U243, U244, U245: NMOS, symbol Raki_ASIC_cells:NMOS
- removed U222, U225, U232, U233, U246, U247, U248, U249: COMPBUF, symbol Raki_ASIC_cells:COMPBUF
- removed U251: GA096, symbol Raki_ASIC_cells:BUF
- removed U254: GA092, symbol Raki_ASIC_cells:INVP
- removed U52: NOR2, symbol Raki_ASIC_cells:NOR2
- removed U53: GA002, symbol Raki_ASIC_cells:VY_DSR_small
- removed U54: GA003, symbol Raki_ASIC_cells:VY_DDL_small
- removed U55: GA004, symbol Raki_ASIC_cells:INVP
- removed U56: GA005, symbol Raki_ASIC_cells:VY_DDL_small
- removed U57, U70: GA006, symbol Raki_ASIC_cells:VY_DSR_small
- removed U58: GA007, symbol Raki_ASIC_cells:INVP
- removed U59: GA008, symbol Raki_ASIC_cells:AOI21
- removed U60: GA010, symbol Raki_ASIC_cells:AOI21
- removed U61: GA009, symbol Raki_ASIC_cells:AOI21
- removed U62: GA012, symbol Raki_ASIC_cells:NOR3
- removed U63: GA011, symbol Raki_ASIC_cells:NOR3
- removed U64: GA013, symbol Raki_ASIC_cells:INV
- removed U65: GA014, symbol Raki_ASIC_cells:INV
- removed U66: GA015, symbol Raki_ASIC_cells:NAND2P
- removed U67: GA016, symbol Raki_ASIC_cells:INV
- removed U68: GA017, symbol Raki_ASIC_cells:NAND2
- removed U69: GA018, symbol Raki_ASIC_cells:INV
- removed U71: GA020, symbol Raki_ASIC_cells:NOR3
- removed U72: GA021, symbol Raki_ASIC_cells:NOR2
- removed U73: GA022, symbol Raki_ASIC_cells:NOR3
- removed U74: GA023, symbol Raki_ASIC_cells:NOR3
- removed U76: GA024, symbol Raki_ASIC_cells:INV
- removed U77: GA025, symbol Raki_ASIC_cells:NOR2
- removed U78: GA026, symbol Raki_ASIC_cells:INVP
- removed U79: GA027, symbol Raki_ASIC_cells:VY_DDL_small
- removed U80: GA029, symbol Raki_ASIC_cells:NOR3
- removed U81: GA028, symbol Raki_ASIC_cells:NOR2
- removed U82: GA030, symbol Raki_ASIC_cells:NOR3
- removed U83: GA031, symbol Raki_ASIC_cells:NOR5
- removed U85: GA032, symbol Raki_ASIC_cells:VY_DSR_small
- removed U86: GA094, symbol Raki_ASIC_cells:VY_DSR_small
- removed U86: GA033, symbol Raki_ASIC_cells:VY_DSR_small
- removed U86: GA093, symbol Raki_ASIC_cells:VY_DSR_small
- removed U89: GA035, symbol Raki_ASIC_cells:VY_DSR_small
- removed U90: GA034, symbol Raki_ASIC_cells:INVP
- removed U91: GA036, symbol Raki_ASIC_cells:NOR3
- removed U92: GA037, symbol Raki_ASIC_cells:AOI21
- removed U93: GA038, symbol Raki_ASIC_cells:VY_DDL_small
- removed U94: GA039, symbol Raki_ASIC_cells:NOR3
- removed U95: GA106, symbol Raki_ASIC_cells:VY_DSR_small
- removed U95: GA107, symbol Raki_ASIC_cells:VY_DSR_small
- removed U95 (x2): GB001, symbol Raki_ASIC_cells:VY_DSR_small
- removed U96: GA040, symbol Raki_ASIC_cells:NOR4
- removed U97: GB003, symbol Raki_ASIC_cells:NAND2
- removed U98: GB002, symbol Raki_ASIC_cells:DFFNR
- removed U99: GA099, symbol Raki_ASIC_cells:INV
- removed U99: GA041, symbol Raki_ASIC_cells:INV
- removed U99: GA108, symbol Raki_ASIC_cells:INV
- added U204, U337: NOR7, symbol Raki_ASIC_cells:NOR7
- added U338: AND2, symbol Raki_ASIC_cells:AND2
- added U339, U340, U342, U343, U344, U345: DLPEN, symbol Raki_ASIC_cells:DLPEN
Connections:
- net BUS.FIRST_DATA.D_{1}: now also U345. (~{Q})
- net BUS.FIRST_DATA.D_{2}: now also U344. (~{Q})
- net BUS.FIRST_DATA.D_{3}: now also U343. (~{Q})
- net BUS.FIRST_DATA.D_{4}: now also U342. (~{Q})
- net BUS.FIRST_DATA.D_{5}: now also U340. (~{Q})
- net BUS.FIRST_DATA.D_{6}: now also U339. (~{Q})
- net CLK.phiL: now also U338.
- net NET.REGNUM.D_{0}: now also U204., U337.
- net NET.REGNUM.D_{1}: now also U204., U337.
- net NET.REGNUM.D_{2}: now also U204., U337.
- net NET.REGNUM.D_{3}: now also U204., U337.
- net NET.REGNUM.D_{4}: now also U337.
- net NET.REGNUM.D_{5}: now also U204., U337.
- net NET.REGNUM.~{D_{4}}: now also U204.
- net NET.REG_DEC_~{EN}: now also U204., U337.
- net NET.REG_d16_EN: now also U204.
- net at U156.: now also U158. (~{Q}); no longer U161. (Φ1)
- net at U126.: now also U124., U125.; no longer U127.
- net at U133.: now also U134.
- new net: U190., U191., U194., U195., U197., U198., U206., U207., U209., U210., U212., U213.
- new net: U145. (~{DOUT}), U148. (~{DOUT}) (x4)
- new net: U146. (~{DOUT}), U148. (~{DOUT}) (x9)
- new net: U145. (~{DOUT}), U146. (~{DOUT}) (x7)
- new net: U156., U161. (Φ1)
- new net: U160. (Φ2), U161. (Φ1)
- new net: U187., U190., U190., U190., U190., U190., U190., U284.
- new net: U190., U190., U99.
- new net: U127., U128. (Φ1)
- new net: U126., U127.
- new net: U211., U213.
- new net: U133., U134., U136.
- new net: U133., U135. (Φ2)
- new net: U338., U339. (~{Q}), U340. (~{Q}), U342. (~{Q}), U343. (~{Q}), U344. (~{Q}), U345. (~{Q})
- new net: U132., U187., U334.
- new net: U187., U99. (x2)
- new net: U157., U159. (Φ2), U187.
- new net: U145. (~{DOUT}), U203.
- new net: U208., U210.
- new net: U196., U198.
- new net: U148. (~{DOUT}), U201.
- new net: U128. (Φ1), U129. (Φ2), U131.
- new net: U155., U164., U214.
- new net: U159. (Φ2), U160. (Φ2)
- new net: U148. (~{DOUT}), U149. (~{DOUT}) (x2)
- new net: U188. (Φ1), U189.
- new net: U187., U188. (Φ1)
- new net: U124., U125.
- new net: U164., U165.
- new net: U155., U156.
- new net: U130. (Φ2), U132.
- new net: U129. (Φ2), U130. (Φ2)
- new net: U193., U195.
- new net: U150. (~{DOUT}), U199.
- new net: U205., U207.
- new net: U146. (~{DOUT}), U202.
- new net: U149. (~{DOUT}), U200.
- new net: U162. (~{DOUT}), U341.
- new net: U191., U192.
- new net: U150. (~{DOUT}), U162. (~{DOUT})
- new net: U149. (~{DOUT}), U150. (~{DOUT})
- new net NET.REG_d0.D_{1}: U345. (~{Q})
- new net NET.REG_d0.D_{2}: U344. (~{Q})
- new net NET.REG_d0.D_{3}: U343. (~{Q})
- new net NET.REG_d0.D_{4}: U342. (~{Q})
- new net NET.REG_d0.D_{5}: U340. (~{Q})
- new net NET.REG_d0.D_{6}: U339. (~{Q})
- new net NET.REG_d0_EN: U337., U338.
- no-connect marks 81 -> 44
Other:
- note removed: "CPU R/W REQUEST SYNCHRONIZER"
- note removed: "FIRST BYTE INLATCH(PORT123)"
- note removed: "INLATCH(TEMPORARY REGISTER) ENABLE GENERATOR"
- note removed: "Indirect writing data in a register"
- note removed: "NEDET"
- note removed: "PORT1 ACCESS TYPE DECODER"
- note removed: "REGISTER WRITE"
- note removed: "SECOND BYTE INLATCH(PORT12)"
- note removed: "SEL0"
- note removed: "SEL1"
- note removed: "VRAM ADDR CNTR ACCESS"
- note removed: "VRAM ADDR CNTR READ"
- note removed: "VRAM address and register set-up"
- note removed: "VRAM01X IOLATCH(CPU<->VRAM)"
- note removed: "Writing Data in the palette register"
- note removed: "Writing Data into the VRAM"
- note removed: "from CPU"
- note removed: "from VRAM INBUF"
- note removed: "to CPU"
- note removed: "to VRAM OUTBUF"
- note removed: "~{LD}"

Commit message: update 20240913
Connections:
- net at U156.: now also U158. (~{Q}); no longer U161. (Φ1)
- net at U126.: now also U124., U125.; no longer U127.
- net at U133.: now also U134.
- new net: U190., U191., U194., U195., U197., U198., U206., U207., U209., U210., U212., U213.
- new net: U145. (~{DOUT}), U148. (~{DOUT}) (x4)
- new net: U146. (~{DOUT}), U148. (~{DOUT}) (x9)
- new net: U145. (~{DOUT}), U146. (~{DOUT}) (x7)
- new net: U156., U161. (Φ1)
- new net: U160. (Φ2), U161. (Φ1)
- new net: U187., U190., U190., U190., U190., U190., U190., U284.
- new net: U190., U190., U99.
- new net: U127., U128. (Φ1)
- new net: U126., U127.
- new net: U211., U213.
- new net: U133., U134., U136.
- new net: U133., U135. (Φ2)
- new net: U338., U339. (~{Q}), U340. (~{Q}), U342. (~{Q}), U343. (~{Q}), U344. (~{Q}), U345. (~{Q})
- new net: U132., U187., U334.
- new net: U187., U99. (x2)
- new net: U157., U159. (Φ2), U187.
- new net: U145. (~{DOUT}), U203.
- new net: U208., U210.
- new net: U196., U198.
- new net: U148. (~{DOUT}), U201.
- new net: U128. (Φ1), U129. (Φ2), U131.
- new net: U155., U164., U214.
- new net: U159. (Φ2), U160. (Φ2)
- new net: U148. (~{DOUT}), U149. (~{DOUT}) (x2)
- new net: U188. (Φ1), U189.
- new net: U187., U188. (Φ1)
- new net: U124., U125.
- new net: U164., U165.
- new net: U155., U156.
- new net: U130. (Φ2), U132.
- new net: U129. (Φ2), U130. (Φ2)
- new net: U193., U195.
- new net: U150. (~{DOUT}), U199.
- new net: U205., U207.
- new net: U146. (~{DOUT}), U202.
- new net: U149. (~{DOUT}), U200.
- new net: U162. (~{DOUT}), U341.
- new net: U191., U192.
- new net: U150. (~{DOUT}), U162. (~{DOUT})
- new net: U149. (~{DOUT}), U150. (~{DOUT})

Commit message: update 20240921
Connections:
- net at U156.: now also U158. (~{Q}); no longer U161. (Φ1)
- net at U126.: now also U124., U125.; no longer U127.
- net at U133.: now also U134.
- new net: U190., U191., U194., U195., U197., U198., U206., U207., U209., U210., U212., U213.
- new net: U145. (~{DOUT}), U148. (~{DOUT}) (x4)
- new net: U146. (~{DOUT}), U148. (~{DOUT}) (x9)
- new net: U145. (~{DOUT}), U146. (~{DOUT}) (x7)
- new net: U156., U161. (Φ1)
- new net: U160. (Φ2), U161. (Φ1)
- new net: U187., U190., U190., U190., U190., U190., U190., U284.
- new net: U190., U190., U99.
- new net: U127., U128. (Φ1)
- new net: U126., U127.
- new net: U211., U213.
- new net: U133., U134., U136.
- new net: U133., U135. (Φ2)
- new net: U338., U339. (~{Q}), U340. (~{Q}), U342. (~{Q}), U343. (~{Q}), U344. (~{Q}), U345. (~{Q})
- new net: U132., U187., U334.
- new net: U187., U99. (x2)
- new net: U157., U159. (Φ2), U187.
- new net: U145. (~{DOUT}), U203.
- new net: U208., U210.
- new net: U196., U198.
- new net: U148. (~{DOUT}), U201.
- new net: U128. (Φ1), U129. (Φ2), U131.
- new net: U155., U164., U214.
- new net: U159. (Φ2), U160. (Φ2)
- new net: U148. (~{DOUT}), U149. (~{DOUT}) (x2)
- new net: U188. (Φ1), U189.
- new net: U187., U188. (Φ1)
- new net: U124., U125.
- new net: U164., U165.
- new net: U155., U156.
- new net: U130. (Φ2), U132.
- new net: U129. (Φ2), U130. (Φ2)
- new net: U193., U195.
- new net: U150. (~{DOUT}), U199.
- new net: U205., U207.
- new net: U146. (~{DOUT}), U202.
- new net: U149. (~{DOUT}), U200.
- new net: U162. (~{DOUT}), U341.
- new net: U191., U192.
- new net: U150. (~{DOUT}), U162. (~{DOUT})
- new net: U149. (~{DOUT}), U150. (~{DOUT})

Commit message: update 20241020
Connections:
- net at U156.: now also U158. (~{Q}); no longer U161. (Φ1)
- net at U126.: now also U124., U125.; no longer U127.
- net at U133.: now also U134.
- new net: U190., U191., U194., U195., U197., U198., U206., U207., U209., U210., U212., U213.
- new net: U145. (~{DOUT}), U148. (~{DOUT}) (x4)
- new net: U146. (~{DOUT}), U148. (~{DOUT}) (x9)
- new net: U145. (~{DOUT}), U146. (~{DOUT}) (x7)
- new net: U156., U161. (Φ1)
- new net: U160. (Φ2), U161. (Φ1)
- new net: U187., U190., U190., U190., U190., U190., U190., U284.
- new net: U190., U190., U99.
- new net: U127., U128. (Φ1)
- new net: U126., U127.
- new net: U211., U213.
- new net: U133., U134., U136.
- new net: U133., U135. (Φ2)
- new net: U338., U339. (~{Q}), U340. (~{Q}), U342. (~{Q}), U343. (~{Q}), U344. (~{Q}), U345. (~{Q})
- new net: U132., U187., U334.
- new net: U187., U99. (x2)
- new net: U157., U159. (Φ2), U187.
- new net: U145. (~{DOUT}), U203.
- new net: U208., U210.
- new net: U196., U198.
- new net: U148. (~{DOUT}), U201.
- new net: U128. (Φ1), U129. (Φ2), U131.
- new net: U155., U164., U214.
- new net: U159. (Φ2), U160. (Φ2)
- new net: U148. (~{DOUT}), U149. (~{DOUT}) (x2)
- new net: U188. (Φ1), U189.
- new net: U187., U188. (Φ1)
- new net: U124., U125.
- new net: U164., U165.
- new net: U155., U156.
- new net: U130. (Φ2), U132.
- new net: U129. (Φ2), U130. (Φ2)
- new net: U193., U195.
- new net: U150. (~{DOUT}), U199.
- new net: U205., U207.
- new net: U146. (~{DOUT}), U202.
- new net: U149. (~{DOUT}), U200.
- new net: U162. (~{DOUT}), U341.
- new net: U191., U192.
- new net: U150. (~{DOUT}), U162. (~{DOUT})
- new net: U149. (~{DOUT}), U150. (~{DOUT})

Commit message: update 20250809
HVCNTR
Parts:
- renumbered U157 to U130, U187 to U131, U124 to U132, U135 to U137, U125 to U138, U159 to U139, U188 to U140, U126 to U141, U189 to U142, U160 to U143, U145 to U154, U127 to U155, U158 to U156, U161 to U157, U128 to U158, U156 to U159, U165 to U160, U129 to U161, U131 to U164, U155 to U165, U133 to U170, U134 to U171, U146 to U172, U136 to U173, U137 to U174, U144 to U175, U148 to U176, U149 to U177, U150 to U180, U162 to U183, U164 to U187, U130 to U188, U132 to U189, U192 to U190, U193 to U191, U196 to U192, U205 to U193, U208 to U194, U211 to U195, U190 to U196, U191 to U197, U194 to U198, U195 to U205, U197 to U206, U198 to U207, U206 to U208, U207 to U209, U209 to U210, U210 to U211, U99 to U282, U187 to U283, U145 to U285, U146 to U286, U148 to U287, U145 to U288, U146 to U289, U148 to U290, U145 to U291, U146 to U292, U148 to U293, U146 to U294, U148 to U295, U145 to U296, U146 to U297, U148 to U298, U145 to U299, U146 to U300, U148 to U301, U190 to U302, U190 to U303, U99 to U304, U190 to U305, U190 to U306, U190 to U310, U190 to U311, U145 to U330, U146 to U331, U148 to U332, U149 to U333, U187 to U335, U99 to U336
Connections:
- net at U159.: now also U156. (~{Q}); no longer U157. (Φ1)
- net at U141.: now also U132., U138.; no longer U155.
- net at U170.: now also U171.
- new net: U196., U197., U198., U205., U206., U207., U208., U209., U210., U211., U212., U213.
- new net: U295. (~{DOUT}), U296. (~{DOUT})
- new net: U294. (~{DOUT}), U295. (~{DOUT})
- new net: U296. (~{DOUT}), U297. (~{DOUT})
- new net: U300. (~{DOUT}), U301. (~{DOUT})
- new net: U288. (~{DOUT}), U301. (~{DOUT})
- new net: U298. (~{DOUT}), U299. (~{DOUT})
- new net: U299. (~{DOUT}), U300. (~{DOUT})
- new net: U297. (~{DOUT}), U298. (~{DOUT})
- new net: U157. (Φ1), U159.
- new net: U143. (Φ2), U157. (Φ1)
- new net: U283., U284., U302., U303., U305., U306., U310., U311.
- new net: U302., U303., U304.
- new net: U155., U158. (Φ1)
- new net: U141., U155.
- new net: U195., U213.
- new net: U285. (~{DOUT}), U286. (~{DOUT})
- new net: U170., U171., U173.
- new net: U137. (Φ2), U170.
- new net: U338., U339. (~{Q}), U340. (~{Q}), U342. (~{Q}), U343. (~{Q}), U344. (~{Q}), U345. (~{Q})
- new net: U292. (~{DOUT}), U293. (~{DOUT})
- new net: U293. (~{DOUT}), U294. (~{DOUT})
- new net: U330. (~{DOUT}), U331. (~{DOUT})
- new net: U331. (~{DOUT}), U332. (~{DOUT})
- new net: U287. (~{DOUT}), U289. (~{DOUT})
- new net: U288. (~{DOUT}), U289. (~{DOUT})
- new net: U189., U334., U335.
- new net: U335., U336.
- new net: U130., U131., U139. (Φ2)
- new net: U154. (~{DOUT}), U203.
- new net: U154. (~{DOUT}), U172. (~{DOUT})
- new net: U194., U211.
- new net: U192., U207.
- new net: U176. (~{DOUT}), U201.
- new net: U158. (Φ1), U161. (Φ2), U164.
- new net: U165., U187., U214.
- new net: U139. (Φ2), U143. (Φ2)
- new net: U332. (~{DOUT}), U333. (~{DOUT})
- new net: U140. (Φ1), U142.
- new net: U131., U140. (Φ1)
- new net: U172. (~{DOUT}), U176. (~{DOUT})
- new net: U176. (~{DOUT}), U177. (~{DOUT})
- new net: U282., U283.
- new net: U132., U138.
- new net: U160., U187.
- new net: U159., U165.
- new net: U188. (Φ2), U189.
- new net: U161. (Φ2), U188. (Φ2)
- new net: U191., U205.
- new net: U180. (~{DOUT}), U199.
- new net: U193., U209.
- new net: U172. (~{DOUT}), U202.
- new net: U291. (~{DOUT}), U292. (~{DOUT})
- new net: U177. (~{DOUT}), U200.
- new net: U290. (~{DOUT}), U291. (~{DOUT})
- new net: U286. (~{DOUT}), U290. (~{DOUT})
- new net: U183. (~{DOUT}), U341.
- new net: U190., U197.
- new net: U180. (~{DOUT}), U183. (~{DOUT})
- new net: U177. (~{DOUT}), U180. (~{DOUT})

Commit message: update 20251106
Parts:
- removed U339, U340, U342, U343, U344, U345: DLPEN, symbol Raki_ASIC_cells:DLPEN
- added U1691, U1692, U1693: NOR7, symbol Raki_ASIC_cells:NOR7
- added U1694: AND2, symbol Raki_ASIC_cells:AND2
- added U1695, U1696, U1697, U1698, U1699, U1700, U339, U340, U342, U343, U344, U345, U586: DLPE, symbol Raki_ASIC_cells:DLPE
Connections:
- net BUS.FIRST_DATA.D_{0}: now also U1700. (~{Q})
- net BUS.FIRST_DATA.D_{1}: now also U1699. (~{Q}), U344. (~{Q})
- net BUS.FIRST_DATA.D_{2}: now also U1698. (~{Q}), U343. (~{Q})
- net BUS.FIRST_DATA.D_{3}: now also U1697. (~{Q}), U342. (~{Q})
- net BUS.FIRST_DATA.D_{4}: now also U1696. (~{Q}), U340. (~{Q})
- net BUS.FIRST_DATA.D_{5}: now also U1695. (~{Q}), U339. (~{Q})
- net BUS.FIRST_DATA.D_{6}: now also U345. (~{Q}), U586. (~{Q})
- net CLK.phiL: now also U1694.
- net NET.REGNUM.D_{0}: now also U1692.
- net NET.REGNUM.D_{1}: now also U1691., U1692.
- net NET.REGNUM.D_{2}: now also U1691., U1692.
- net NET.REGNUM.D_{3}: now also U1691.
- net NET.REGNUM.D_{4}: now also U1691., U1692., U1693.
- net NET.REGNUM.D_{5}: now also U1691., U1692., U1693.
- net NET.REGNUM.~{D_{0}}: now also U1691., U1693.
- net NET.REGNUM.~{D_{1}}: now also U1693.
- net NET.REGNUM.~{D_{2}}: now also U1693.
- net NET.REGNUM.~{D_{3}}: now also U1692., U1693.
- net NET.REG_DEC_~{EN}: now also U1691., U1692., U1693.
- net NET.REG_d0.D_{1}: now also U344. (~{Q})
- net NET.REG_d0.D_{2}: now also U343. (~{Q})
- net NET.REG_d0.D_{3}: now also U342. (~{Q})
- net NET.REG_d0.D_{4}: now also U340. (~{Q})
- net NET.REG_d0.D_{5}: now also U339. (~{Q})
- net NET.REG_d0.D_{6}: now also U586. (~{Q})
- net at U159.: now also U156. (~{Q}); no longer U157. (Φ1)
- net at U141.: now also U132., U138.; no longer U155.
- net GBL.phiL_RST: now reaches U170.
- net GBL.phiL_RST: now also U132., U142., U196., U197., U198., U205., U206., U207., U208., U209., U210., U211., U212., U213.
- new net: U295. (~{DOUT}), U296. (~{DOUT})
- new net: U294. (~{DOUT}), U295. (~{DOUT})
- new net: U296. (~{DOUT}), U297. (~{DOUT})
- new net: U300. (~{DOUT}), U301. (~{DOUT})
- new net: U288. (~{DOUT}), U301. (~{DOUT})
- new net: U298. (~{DOUT}), U299. (~{DOUT})
- new net: U299. (~{DOUT}), U300. (~{DOUT})
- new net: U297. (~{DOUT}), U298. (~{DOUT})
- new net: U157. (Φ1), U159.
- new net: U143. (Φ2), U157. (Φ1)
- new net: U1694., U1695. (~{Q}), U1696. (~{Q}), U1697. (~{Q}), U1698. (~{Q}), U1699. (~{Q}), U1700. (~{Q}), U345. (~{Q})
- new net: U283., U284., U302., U303., U305., U306., U310., U311.
- new net: U302., U303., U304.
- new net: U155., U158. (Φ1)
- new net: U141., U155.
- new net: U195., U213.
- new net: U285. (~{DOUT}), U286. (~{DOUT})
- new net: U338., U339. (~{Q}), U340. (~{Q}), U342. (~{Q}), U343. (~{Q}), U344. (~{Q}), U586. (~{Q})
- new net: U170., U171., U173.
- new net: U137. (Φ2), U170.
- new net: U170., U171.
- new net: U292. (~{DOUT}), U293. (~{DOUT})
- new net: U293. (~{DOUT}), U294. (~{DOUT})
- new net: U330. (~{DOUT}), U331. (~{DOUT})
- new net: U331. (~{DOUT}), U332. (~{DOUT})
- new net: U287. (~{DOUT}), U289. (~{DOUT})
- new net: U288. (~{DOUT}), U289. (~{DOUT})
- new net: U189., U334., U335.
- new net: U335., U336.
- new net: U130., U131., U139. (Φ2)
- new net: U154. (~{DOUT}), U203.
- new net: U154. (~{DOUT}), U172. (~{DOUT})
- new net: U194., U211.
- new net: U192., U207.
- new net: U176. (~{DOUT}), U201.
- new net: U158. (Φ1), U161. (Φ2), U164.
- new net: U165., U187., U214.
- new net: U139. (Φ2), U143. (Φ2)
- new net: U332. (~{DOUT}), U333. (~{DOUT})
- new net: U140. (Φ1), U142.
- new net: U131., U140. (Φ1)
- new net: U172. (~{DOUT}), U176. (~{DOUT})
- new net: U176. (~{DOUT}), U177. (~{DOUT})
- new net: U282., U283.
- new net: U132., U138.
- new net: U160., U187.
- new net: U159., U165.
- new net: U188. (Φ2), U189.
- new net: U161. (Φ2), U188. (Φ2)
- new net: U191., U205.
- new net: U180. (~{DOUT}), U199.
- new net: U193., U209.
- new net: U172. (~{DOUT}), U202.
- new net: U291. (~{DOUT}), U292. (~{DOUT})
- new net: U177. (~{DOUT}), U200.
- new net: U290. (~{DOUT}), U291. (~{DOUT})
- new net: U286. (~{DOUT}), U290. (~{DOUT})
- new net: U183. (~{DOUT}), U341.
- new net: U190., U197.
- new net: U180. (~{DOUT}), U183. (~{DOUT})
- new net: U177. (~{DOUT}), U180. (~{DOUT})
- new net NET.REG_d1.D_{0}: U1700. (~{Q})
- new net NET.REG_d1.D_{1}: U1699. (~{Q})
- new net NET.REG_d1.D_{2}: U1698. (~{Q})
- new net NET.REG_d1.D_{3}: U1697. (~{Q})
- new net NET.REG_d1.D_{4}: U1696. (~{Q})
- new net NET.REG_d1.D_{5}: U1695. (~{Q})
- new net NET.REG_d1.D_{6}: U345. (~{Q})
- new net NET.REG_d15_EN: U1693.
- new net NET.REG_d1_EN: U1691., U1694.
- new net NET.REG_d8_EN: U1692.
- no-connect marks 44 -> 51
Other:
- note added: "COLOR DI BUS"
- note added: "CONFIG REG DECODER"
- note added: "CPU DI BUS"
- note added: "CPU DO BUS"
- note added: "VRAM A BUS"
- note added: "VRAM DI BUS"
- note added: "VRAM DO BUS"
- note removed: "RST?"
