File: resources/V9958_kicad/ST.kicad_sch (KiCad schematic)
At the start: 394 parts, among them U10 DSR, U11 INVP, U1191 GC001, U1192 GC002, U1193 GC003, U1194 GC004, U1195 GC005, U12 AND2, U13 DSR, U1344 GC006, U1345 GC007, U1346 GC008, U1347 GC009, U1348 GC016, U1349 GC017, U1350 GC014, U1351 GC015, U1352 GC018, U1353 GC013, U1354 GC012, U1355 GC011, U1356 INV, U1357 NORWIDE, U1358 NMOS, U1359 NORWIDE, U1360 NMOS, U1361 NORWIDE, U1362 NMOS, U1363 NORWIDE, U1364 NMOS, U1365 NORWIDE, U1366 NMOS, U1367 NORWIDE, U1368 NMOS, U1369 NORWIDE, U1370 NMOS, U1371 NORWIDE, U1372 NMOS, U1373 NORWIDE, U1374 NMOS, U1375 NORWIDE, U1376 NMOS, U1377 NMOS, U1378 NORWIDE, U1379 NORWIDE, U1380 NMOS, U1381 NMOS, U1382 NORWIDE, U1383 NORWIDE, U1384 NMOS, U1385 NMOS, U1386 NORWIDE, U1387 NORWIDE, U1388 NMOS, U1389 NORWIDE, U1390 NMOS, U1391 NORWIDE, U1392 NMOS, U1393 NORWIDE, U1394 NMOS, U1395 NORWIDE, U1396 NMOS, U1397 NORWIDE, U1398 NMOS, U1399 GC019, U1400 GC020, U1401 GC021, U1402 GC022, U1403 GC023, U1404 INV, U1405 GC024, U1406 GC025, U1407 INV, U1408 GC026, U1409 NOR2, U1410 GC010, U1411 DDL, U1412 NMOS, U1413 NMOS, U1414 NMOS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

Commit message: update 20251106
Parts:
- removed U10, U13, U16, U17, U18, U19, U20, U21, U22, U23, U27, U28, U29, U30, U31: DSR, symbol Raki_ASIC_cells:VY_DSR_small
- removed U11: INVP, symbol Raki_ASIC_cells:INVP
- removed U12: AND2, symbol Raki_ASIC_cells:AND2
- removed U1412, U1413, U1414, U1415, U1416, U1417, U1418, U1419, U39, U40: NMOS, symbol Raki_ASIC_cells:NMOS
- removed U24: NOR4, symbol Raki_ASIC_cells:NOR4
- removed U25, U26, U32, U46, U47, U48, U49, U50, U51: NOR2, symbol Raki_ASIC_cells:NOR2
- removed U35, U41, U42, U43, U44, U45: INV, symbol Raki_ASIC_cells:INV
- removed U36: NOR6, symbol Raki_ASIC_cells:NOR6
- removed U37, U38: BUFP, symbol Raki_ASIC_cells:BUFP
- removed U9: BUF, symbol Raki_ASIC_cells:BUF
- U1686: value GC105 -> NOR2
Connections:
- net NET.REG_d9_b3_IL is gone; now on net NET.FIELDNUM: U1540.
- net NET.ST.HCNTR.D_{6} is gone; now on net NET.ST.HCNTR.D_{0}: U1345. (~{DOUT}), U1467. (~{S})
- net NET.ST.HCNTR.~{D_{3}} is gone; now on net NET.ST.HCNTR.D_{0}: U1194. (~{DOUT})
- net NET.ST.VACNTR.D_{0} is gone; now on net NET.ST.VACNTR.RST: U1527. (~{DOUT})
- net NET.ST.VACNTR.D_{1} is gone; now on net NET.ST.VACNTR.RST: U1528. (~{DOUT})
- net NET.ST.VACNTR.D_{2} is gone; now on net NET.ST.VACNTR.RST: U1529. (~{DOUT})
- net NET.ST.VACNTR.D_{3} is gone; now on net NET.ST.VACNTR.RST: U1530. (~{DOUT})
- net NET.ST.VACNTR.D_{4} is gone; now on net NET.ST.VACNTR.RST: U1531. (~{DOUT})
- net NET.ST.VACNTR.D_{5} is gone; now on net NET.ST.VACNTR.RST: U1532. (~{DOUT})
- net NET.ST.VACNTR.D_{6} is gone; now on net NET.ST.VACNTR.RST: U1533. (~{DOUT})
- net NET.ST.VACNTR.D_{7} is gone; now on net NET.ST.VACNTR.RST: U1534. (~{DOUT})
- net NET.ST.VACNTR.D_{8} is gone; now on net NET.ST.VACNTR.RST: U1535. (~{DOUT})
- net NET.ST.VACNTR.~{D_{0}} is gone; now on net NET.ST.VACNTR.RST: U1527. (~{DOUT})
- net NET.ST.VACNTR.~{D_{1}} is gone; now on net NET.ST.VACNTR.RST: U1528. (~{DOUT})
- net NET.ST.VACNTR.~{D_{2}} is gone; now on net NET.ST.VACNTR.RST: U1529. (~{DOUT})
- net NET.ST.VACNTR.~{D_{3}} is gone; now on net NET.ST.VACNTR.RST: U1530. (~{DOUT})
- net NET.ST.VACNTR.~{D_{4}} is gone; now on net NET.ST.VACNTR.RST: U1531. (~{DOUT})
- net NET.ST.VACNTR.~{D_{5}} is gone; now on net NET.ST.VACNTR.RST: U1532. (~{DOUT})
- net NET.ST.VACNTR.~{D_{6}} is gone; now on net NET.ST.VACNTR.RST: U1533. (~{DOUT})
- net NET.ST.VACNTR.~{D_{7}} is gone; now on net NET.ST.VACNTR.RST: U1534. (~{DOUT})
- net NET.ST.VACNTR.~{D_{8}} is gone; now on net NET.ST.VACNTR.RST: U1535. (~{DOUT})
- net NET.ST.VCNTR.~{D_{1}} is gone; now on net NET.ST.VCNTR.RST: U1488. (~{DOUT})
- net NET.ST.VCNTR.~{D_{2}} is gone; now on net NET.ST.VCNTR.RST: U1489. (~{DOUT})
- net NET.ST.VCNTR.~{D_{3}} is gone; now on net NET.ST.VCNTR.RST: U1490. (~{DOUT})
- net NET.ST.VCNTR.~{D_{4}} is gone; now on net NET.ST.VCNTR.RST: U1491. (~{DOUT})
- net NET.ST.VCNTR.~{D_{5}} is gone; now on net NET.ST.VCNTR.RST: U1492. (~{DOUT})
- net CLK.phiL: now also U1657., U1662., U1664., U1666., U1668., U1670., U1672., U1674., U1676., U1678.
- net NET.FIELDNUM: now also TP011.1, TP012.1, U1487. (~{DOUT}), U1488. (~{DOUT}), U1489. (~{DOUT}), U1490. (~{DOUT}), U1491. (~{DOUT}), U1492. (~{DOUT}), U1493. (~{DOUT}), U1494. (~{DOUT}), U1495. (~{DOUT}), U1536., U1539., U1541., U1543., U1545., U1547., U1550., U1551., U1553., U1556., U1557., U1559., U1562., U1563., U1565., U1568., U1569., U1571., U1574., U1575., U1578., U1580., U1581., U1583., U1586., U1587., U1589., U1593., U1594., U1599. (~{S}), U1600. (~{S}), U1601. (~{S}), U1602. (~{S}), U1603. (~{S}), U1604. (~{S}), U1605. (~{S}), U1606. (~{S}), U1607. (~{S}), U1653., U1654., U1655.
- net NET.REG_d9_b7_LN: now also U1527. (~{DOUT}), U1528. (~{DOUT}), U1529. (~{DOUT}), U1530. (~{DOUT}), U1531. (~{DOUT}), U1532. (~{DOUT}), U1533. (~{DOUT}), U1534. (~{DOUT}), U1535. (~{DOUT}), U1658., U1661., U1663., U1665., U1667., U1669., U1671., U1673., U1675., U1677., U1679.
- net NET.ST.HCNTR.D_{0}: now also U1192. (~{DOUT}), U1193. (~{DOUT}), U1195. (~{DOUT}), U1344. (~{DOUT}), U1346. (~{DOUT}), U1347. (~{DOUT}), U1357., U1359., U1361., U1363., U1365., U1367., U1369., U1371., U1373., U1375., U1378., U1379., U1382., U1383., U1386., U1387., U1389., U1391., U1393., U1395., U1397., U1410., U1461. (~{S}), U1463. (~{S}), U1464. (~{S}), U1465. (~{S}), U1466. (~{S}), U1468. (~{S}), U1469. (~{S})
- net at U1513.: now also U1514., U1515. (Φ2); no longer U1522.
- net at U1508.: now also U1498. (Φ2); no longer U1509. (Φ2)
- net at U1447.: now also U1449.; no longer U1448.
- net at U1624.: now also U1634.; no longer U1623.
- net at U1479.: now also U1477. (Φ1); no longer U1470. (Φ1)
- net at U1449.: now also U1450. (Φ1), U1458.; no longer U1447.
- net at U1632.: now also U1631.; no longer U1630.
- net at U1640.: now also U1632., U1638.; no longer U1641.
- net at U1501.: now also U1502.; no longer U1503. (Φ2)
- net at U1354.: now also U1355.; no longer U1353. (Φ2)
- net at U1444.: now also U1442. (Y), U1443.; no longer U1445.
- net at U1611.: now also U1606. (~{S}); no longer U1613.
- net at U1455.: now also U1446. (Φ1); no longer U1454.
- net at U1406.: now also U1408. (Φ1); no longer U1407.
- net at U1610.: now also U1605. (~{S}); no longer U1613.
- net at U1403.: now also U1405. (Φ1); no longer U1404.
- net at U1521.: now also U1511., U1514., U1518., U1520.; no longer U1523. (Φ2)
- net at U1356.: now also U1410.; no longer U1354.
- net at U1612.: now also U1613.; no longer U1607. (~{S})
- net at U1635.: now also U1634.; no longer U1619.
- net at U1619.: now also U1596.; no longer U1618.
- net at U1637., U1638.: now also U1639. (Φ2)
- net at U1485.: no longer U1486.
- net at U1608.: now also U1603. (~{S}); no longer U1613.
- net at U1609.: now also U1604. (~{S}); no longer U1613.
- net at U1441.: now also U1440.; no longer U1442. (Y)
- net at U1627.: now also U1625.; no longer U1626.
- removed net NET.REG_d9_b1_~{NT}: U1539., U1653., U1654., U1655.
- removed net NET.ST.HCNTR.D_{1}: U1191. (~{DOUT}), U1192. (~{DOUT}), U1193. (~{DOUT}), U1194. (~{DOUT}), U1195. (~{DOUT}), U1344. (~{DOUT}), U1345. (~{DOUT}), U1346. (~{DOUT}), U1347. (~{DOUT}), U1357., U1369., U1410., U1461. (~{S}), U1463. (~{S}), U1464. (~{S}), U1465. (~{S}), U1466. (~{S}), U1468. (~{S}), U1469. (~{S})
- removed net NET.ST.VCNTR.D_{0}: U1487. (~{DOUT}), U1599. (~{S})
- removed net NET.ST.VCNTR.D_{1}: U1488. (~{DOUT}), U1600. (~{S})
- removed net NET.ST.VCNTR.D_{2}: U1489. (~{DOUT}), U1601. (~{S})
- removed net NET.ST.VCNTR.D_{3}: U1490. (~{DOUT}), U1602. (~{S})
- removed net NET.ST.VCNTR.D_{4}: U1491. (~{DOUT}), U1603. (~{S})
- removed net NET.ST.VCNTR.D_{5}: U1492. (~{DOUT}), U1604. (~{S})
- removed net NET.ST.VCNTR.D_{6}: U1493. (~{DOUT}), U1605. (~{S})
- removed net NET.ST.VCNTR.D_{7}: U1494. (~{DOUT}), U1606. (~{S})
- removed net NET.ST.VCNTR.D_{8}: U1495. (~{DOUT}), U1607. (~{S})
- removed net NET.ST.VCNTR.~{D_{0}}: TP011.1, U1487. (~{DOUT})
- removed net NET.ST.VCNTR.~{D_{8}}: TP012.1, U1495. (~{DOUT})
- new net: U1579., U1580.
- new net: U1629., U1631.
- new net: U1497., U1498. (Φ2), U1501.
- new net: U1497., U1500., U1501.
- new net: U1497., U1499., U1502.
- new net: U1651., U1654., U1656.
- new net: U1674., U1675.
- new net: U1513., U1522.
- new net: U1581., U1582.
- new net: U1393., U1394.
- new net: U1371., U1372.
- new net: U1348., U1352.
- new net: U1365., U1366.
- new net: U1508., U1509. (Φ2)
- new net: U1508., U1509. (Φ2), U1510.
- new net: U1447., U1448.
- new net: U1623., U1624.
- new net: U1467. (~{S}), U1468. (~{S})
- new net: U1468. (~{S}), U1469. (~{S})
- new net: U1468. (~{S}), U1477. (Φ1)
- new net: U1470. (Φ1), U1479.
- new net: U1474. (Φ1), U1479.
- new net: U1472. (Φ1), U1479.
- new net: U1471. (Φ1), U1479.
- new net: U1475. (Φ1), U1479.
- new net: U1476. (Φ1), U1479.
- new net: U1479., U1480. (Φ2)
- new net: U1473. (Φ1), U1479.
- new net: U1478. (Φ1), U1479.
- new net: U1462. (~{S}), U1470. (Φ1)
- new net: U1510., U1518., U1519. (Φ2)
- new net: U1516., U1518., U1519. (Φ2)
- new net: U1350., U1351., U1353. (Φ2), U1354.
- new net: U1348., U1349., U1351.
- new net: U1350., U1351.
- new net: U1513., U1516., U1517., U1520.
- new net: U1410., U1411. (Φ1)
- new net: U1585., U1586.
- new net: U1543., U1544.
- new net: U1505. (Φ2), U1506.
- new net: U1437., U1440., U1447.
- new net: U1533. (~{DOUT}), U1534. (~{DOUT}), U1535. (~{DOUT}), U1649.
- new net: U1534. (~{DOUT}), U1535. (~{DOUT})
- new net: U1533. (~{DOUT}), U1534. (~{DOUT})
- new net: U1628., U1630.
- new net: U1630., U1632.
- new net: U1567., U1568.
- new net: U1400., U1401., U1406.
- new net: U1400., U1401.
- new net: U1423., U1425., U1427. (Φ1)
- new net: U1423., U1425.
- new net: U1361., U1362.
- new net: U1563., U1564.
- new net: U1640., U1641.
- new net: U1640., U1641., U1642.
- new net: U1547., U1548.
- new net: U1680., U1681., U1682.
- new net: U1680., U1681.
- new net: U1432., U1433., U1434. (Φ1)
- new net: U1432., U1433.
- new net: U1575., U1576.
- new net: U1501., U1503. (Φ2) (x2)
- new net: U1465. (~{S}), U1474. (Φ1)
- new net: U1670., U1671.
- new net: U1466. (~{S}), U1467. (~{S})
- new net: U1466. (~{S}), U1475. (Φ1)
- new net: U1465. (~{S}), U1466. (~{S})
- new net: U1551., U1552.
- new net: U1353. (Φ2), U1354.
- new net: U1569., U1570.
- new net: U1643., U1644., U1645., U1646., U1647., U1648., U1649., U1650. (Φ1)
- new net: U1643., U1644., U1645., U1646., U1648., U1652.
- new net: U1643., U1645., U1648., U1651.
- new net: U1444., U1445.
- new net: U1672., U1673.
- new net: U1611., U1613.
- new net: U1577., U1578.
- new net: U1454., U1455.
- new net: U1622., U1624.
- new net: U1620., U1622.
- new net: U1678., U1679.
- new net: U1487. (~{DOUT}), U1504.
- new net: U1406., U1407.
- new net: U1510., U1514., U1515. (Φ2), U1517.
- new net: U1511., U1512. (Φ2), U1517.
- new net: U1429., U1430.
- new net: U1429., U1430., U1431. (Φ1)
- new net: U1491. (~{DOUT}), U1492. (~{DOUT})
- new net: U1492. (~{DOUT}), U1493. (~{DOUT})
- new net: U1389., U1390.
- new net: U1541., U1542.
- new net: U1463. (~{S}), U1472. (Φ1)
- new net: U1359., U1360.
- new net: U1610., U1613.
- new net: U1461. (~{S}), U1462. (~{S})
- new net: U1461. (~{S}), U1471. (Φ1)
- new net: U1461. (~{S}), U1463. (~{S})
- new net: U1683., U1684. (Φ2)
- new net: U1367., U1368.
- new net: U1592., U1593.
- new net: U1403., U1404.
- new net: U1383., U1384.
- new net: U1549., U1550.
- new net: U1493. (~{DOUT}), U1494. (~{DOUT})
- new net: U1494. (~{DOUT}), U1495. (~{DOUT})
- new net: U1420., U1421., U1422. (Φ1)
- new net: U1444., U1456. (Φ1)
- new net: U1192. (~{DOUT}), U1193. (~{DOUT})
- new net: U1191. (~{DOUT}), U1192. (~{DOUT})
- new net: U1385., U1386.
- new net: U1557., U1558.
- new net: U1523. (Φ2), U1524.
- new net: U1521., U1523. (Φ2)
- new net: U1354., U1356.
- new net: U1607. (~{S}), U1612.
- new net: U1606. (~{S}), U1607. (~{S})
- new net: U1490. (~{DOUT}), U1491. (~{DOUT})
- new net: U1645., U1647., U1653.
- new net: U1685., U1686., U1687.
- new net: U1685., U1686.
- new net: U1499., U1597.
- new net: U1458., U1459. (Φ1)
- new net: U1573., U1574.
- new net: U1387., U1388.
- new net: U1565., U1566.
- new net: U1688., U1689., U1690.
- new net: U1688., U1689.
- new net: U1644., U1646., U1654.
- new net: U1591., U1594.
- new net: U1666., U1667.
- new net: U1619., U1635.
- new net: U1634., U1635., U1636. (Φ2)
- new net: U1601. (~{S}), U1602. (~{S})
- new net: U1601. (~{S}), U1613.
- new net: U1600. (~{S}), U1601. (~{S})
- new net: U1555., U1556.
- new net: U1618., U1619.
- new net: U1617., U1618.
- new net: U1489. (~{DOUT}), U1490. (~{DOUT})
- new net: U1463. (~{S}), U1464. (~{S})
- new net: U1464. (~{S}), U1473. (Φ1)
- new net: U1464. (~{S}), U1465. (~{S})
- new net: U1391., U1392.
- new net: U1402. (Y), U1403.
- new net: U1637., U1638.
- new net: U1571., U1572.
- new net: U1424., U1426., U1428. (Φ1)
- new net: U1424., U1426.
- new net: U1437., U1438., U1439.
- new net: U1437., U1438., U1440.
- new net: U1545., U1546.
- new net: U1482., U1483.
- new net: U1443., U1481. (Φ1), U1482.
- new net: U1451., U1452. (Φ1)
- new net: U1602. (~{S}), U1613.
- new net: U1602. (~{S}), U1603. (~{S})
- new net: U1485., U1486.
- new net: U1524., U1525.
- new net: U1595., U1596.
- new net: U1375., U1376.
- new net: U1668., U1669.
- new net: U1664., U1665.
- new net: U1369., U1370.
- new net: U1608., U1613.
- new net: U1609., U1613.
- new net: U1600. (~{S}), U1613.
- new net: U1599. (~{S}), U1613.
- new net: U1435. (Φ1), U1484., U1485.
- new net: U1193. (~{DOUT}), U1194. (~{DOUT})
- new net: U1194. (~{DOUT}), U1195. (~{DOUT})
- new net: U1536., U1537.
- new net: U1467. (~{S}), U1476. (Φ1)
- new net: U1441., U1442. (Y)
- new net: U1529. (~{DOUT}), U1530. (~{DOUT})
- new net: U1530. (~{DOUT}), U1531. (~{DOUT})
- new net: U1487. (~{DOUT}), U1488. (~{DOUT})
- new net: U1346. (~{DOUT}), U1347. (~{DOUT})
- new net: U1459. (Φ1), U1460.
- new net: U1528. (~{DOUT}), U1529. (~{DOUT})
- new net: U1420., U1421.
- new net: U1527. (~{DOUT}), U1528. (~{DOUT})
- new net: U1526., U1527. (~{DOUT})
- new net: U1561., U1562.
- new net: U1344. (~{DOUT}), U1345. (~{DOUT})
- new net: U1195. (~{DOUT}), U1344. (~{DOUT})
- new net: U1377., U1378.
- new net: U1446. (Φ1), U1457.
- new net: U1345. (~{DOUT}), U1346. (~{DOUT})
- new net: U1488. (~{DOUT}), U1489. (~{DOUT})
- new net: U1583., U1584.
- new net: U1357., U1358.
- new net: U1348., U1349., U1350.
- new net: U1651., U1652., U1655.
- new net: U1603. (~{S}), U1604. (~{S})
- new net: U1604. (~{S}), U1605. (~{S})
- new net: U1614. (Φ2), U1615. (Φ1)
- new net: U1599. (~{S}), U1600. (~{S})
- new net: U1450. (Φ1), U1451.
- new net: U1373., U1374.
- new net: U1469. (~{S}), U1478. (Φ1)
- new net: U1559., U1560.
- new net: U1531. (~{DOUT}), U1532. (~{DOUT})
- new net: U1532. (~{DOUT}), U1533. (~{DOUT})
- new net: U1381., U1382.
- new net: U1395., U1396.
- new net: U1657., U1658.
- new net: U1379., U1380.
- new net: U1553., U1554.
- new net: U1500., U1598.
- new net: U1626., U1627.
- new net: U1676., U1677.
- new net: U1397., U1398.
- new net: U1363., U1364.
- new net: U1662., U1663.
- new net: U1589., U1590.
- new net: U1587., U1588.
- new net: U1621., U1625.
- new net: U1605. (~{S}), U1606. (~{S})
- now unconnected: U1485.
- no-connect marks 195 -> 180
Other:
- note added: "HORIZONTAL COUNTER"
- note removed: "0"
- note removed: "1"
- note removed: "2"
- note removed: "3"
- note removed: "A"
- note removed: "B"
- note removed: "Follows XTAL1/2's toggling"
- note removed: "INTERNAL CLOCK DIVIDER"
- note removed: "Super duper high side bootstrapped NOR2"
- moved on the sheet: TP010, TP011, TP012, TP013
