File: resources/V9958_kicad/V9958.kicad_sch (KiCad schematic)
At the start: 47 parts, among them U1 NMOS, U10 NMOS, U11 NMOS, U12 NMOS, U13 NMOS, U16 AND2, U17 DSR, U18 NOR6, U19 DSR, U2 NOR2, U20 DSR, U21 DSR, U22 DSR, U23 DSR, U24 DSR, U25 DSR, U26 BUF, U27 INVP, U28 NOR2, U29 NOR2, U3 INV, U30 DSR, U31 DSR, U32 DSR, U35 NOR4, U36 DSR, U37 DSR, U38 DSR, U39 NOR2, U4 INV, U40 BUFP, U41 DSR, U42 INV, U43 BUFP, U44 NMOS, U45 NMOS, U46 NOR2, U47 NOR2, U48 INV, U49 INV, U5 INV, U50 NOR2, U51 NOR2, U6 NMOS, U7 NMOS, U8 NMOS, U9 NOR2

Commit message: update 20240825
Connections:
- net at U18.: now also U24. (Φ2); no longer U17. (Φ2)
- net at U43.: now also U44.; no longer U42.
- net at U48.: now also U21. (Φ2), U46.; no longer U47.
- net at U40.: now also U45.; no longer U39.
- net at U27.: now also U16.; no longer U25. (Φ2)
- new net: U18., U19. (Φ2), U20. (Φ2), U29.
- new net: U18., U20. (Φ2), U28.
- new net: U17. (Φ2), U18., U19. (Φ2), U28., U29.
- new net: U17. (Φ2), U18.
- new net: U18., U36. (Φ2)
- new net: U18., U23. (Φ2), U24. (Φ2)
- new net: U1., U2., U8.
- new net: U1., U6., U7.
- new net: U42., U43.
- new net: U47., U48.
- new net: U38. (Φ2), U39.
- new net: U39., U40.
- new net: U31. (Φ2), U32. (Φ2), U35.
- new net: U32. (Φ2), U35.
- new net: U10., U11., U13.
- new net: U37. (Φ2), U49., U50.
- new net: U22. (Φ2), U23. (Φ2)
- new net: U16., U22. (Φ2)
- new net: U11., U12., U9.
- new net: U28., U37. (Φ2), U41. (Φ2)
- new net: U21. (Φ2), U29., U30. (Φ2), U38. (Φ2)
- new net: U25. (Φ2), U27.
- new net: U25. (Φ2), U26.
- new net: U10., U5., U9.
- new net: U2., U3., U6.
- new net: U30. (Φ2), U31. (Φ2)
- new net: U35., U36. (Φ2)
Other:
- sheet DI renamed MI
- added sheet CI (CI.kicad_sch)
- added sheet VT (VT.kicad_sch)
- sheet MI: file DI.kicad_sch -> MI.kicad_sch
Changed lines of the file:
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@@
   (title_block
     (title "V9958")
-    (date "2024-07-16")
+    (date "2024-08-24")
+    (rev "WIP")
     (company "IKA Microelectronics Inc.")
-    (comment 1 "WIP")
   )
   (junction (at 111.76 77.47) (diameter 0) (color 0 0 0 0)
@@
     (stroke (width 0.1524) (type solid))
     (fill (color 0 0 0 0.0000))
-    (property "Sheetname" "DI" (at 78.74 225.3484 0)
+    (property "Sheetname" "MI" (at 78.74 225.3484 0)
       (effects (font (size 1.27 1.27)) (justify left bottom))
     )
-    (property "Sheetfile" "DI.kicad_sch" (at 78.74 258.3946 0)
+    (property "Sheetfile" "MI.kicad_sch" (at 78.74 258.3946 0)
       (effects (font (size 1.27 1.27)) (justify left top))
     )
@@
       )
     )
+  )
+  (sheet (at 78.74 265.43) (size 33.02 31.75) (fields_autoplaced)
+    (stroke (width 0.1524) (type solid))
+    (fill (color 0 0 0 0.0000))
+    (property "Sheetname" "VT" (at 78.74 264.7184 0)
+      (effects (font (size 1.27 1.27)) (justify left bottom))
+    )
+    (property "Sheetfile" "VT.kicad_sch" (at 78.74 297.7646 0)
+      (effects (font (size 1.27 1.27)) (justify left top))
+    )
+    (instances
+      (project "V9958"
+        (path "/b5e1370a-fef4-4131-9314-bdfc21cb5e0f" (page "5"))
+      )
+    )
+  )
+  (sheet (at 41.91 265.43) (size 31.75 31.75) (fields_autoplaced)
+    (stroke (width 0.1524) (type solid))
+    (fill (color 0 0 0 0.0000))
+    (property "Sheetname" "CI" (at 41.91 264.7184 0)
+      (effects (font (size 1.27 1.27)) (justify left bottom))
+    )
+    (property "Sheetfile" "CI.kicad_sch" (at 41.91 297.7646 0)
+      (effects (font (size 1.27 1.27)) (justify left top))
+    )
+    (instances
+      (project "V9958"
+        (path "/b5e1370a-fef4-4131-9314-bdfc21cb5e0f" (page "4"))
+      )
+    )

Commit message: update 20240913
Connections:
- net at U18.: now also U24. (Φ2); no longer U17. (Φ2)
- net at U43.: now also U44.; no longer U42.
- net at U48.: now also U21. (Φ2), U46.; no longer U47.
- net at U40.: now also U45.; no longer U39.
- net at U27.: now also U16.; no longer U25. (Φ2)
- new net: U18., U19. (Φ2), U20. (Φ2), U29.
- new net: U18., U20. (Φ2), U28.
- new net: U17. (Φ2), U18., U19. (Φ2), U28., U29.
- new net: U17. (Φ2), U18.
- new net: U18., U36. (Φ2)
- new net: U18., U23. (Φ2), U24. (Φ2)
- new net: U1., U2., U8.
- new net: U1., U6., U7.
- new net: U42., U43.
- new net: U47., U48.
- new net: U38. (Φ2), U39.
- new net: U39., U40.
- new net: U31. (Φ2), U32. (Φ2), U35.
- new net: U32. (Φ2), U35.
- new net: U10., U11., U13.
- new net: U37. (Φ2), U49., U50.
- new net: U22. (Φ2), U23. (Φ2)
- new net: U16., U22. (Φ2)
- new net: U11., U12., U9.
- new net: U28., U37. (Φ2), U41. (Φ2)
- new net: U21. (Φ2), U29., U30. (Φ2), U38. (Φ2)
- new net: U25. (Φ2), U27.
- new net: U25. (Φ2), U26.
- new net: U10., U5., U9.
- new net: U2., U3., U6.
- new net: U30. (Φ2), U31. (Φ2)
- new net: U35., U36. (Φ2)

Commit message: update 20240921
Connections:
- net at U18.: now also U24. (Φ2); no longer U17. (Φ2)
- net at U43.: now also U44.; no longer U42.
- net at U48.: now also U21. (Φ2), U46.; no longer U47.
- net at U40.: now also U45.; no longer U39.
- net at U27.: now also U16.; no longer U25. (Φ2)
- new net: U18., U19. (Φ2), U20. (Φ2), U29.
- new net: U18., U20. (Φ2), U28.
- new net: U17. (Φ2), U18., U19. (Φ2), U28., U29.
- new net: U17. (Φ2), U18.
- new net: U18., U36. (Φ2)
- new net: U18., U23. (Φ2), U24. (Φ2)
- new net: U1., U2., U8.
- new net: U1., U6., U7.
- new net: U42., U43.
- new net: U47., U48.
- new net: U38. (Φ2), U39.
- new net: U39., U40.
- new net: U31. (Φ2), U32. (Φ2), U35.
- new net: U32. (Φ2), U35.
- new net: U10., U11., U13.
- new net: U37. (Φ2), U49., U50.
- new net: U22. (Φ2), U23. (Φ2)
- new net: U16., U22. (Φ2)
- new net: U11., U12., U9.
- new net: U28., U37. (Φ2), U41. (Φ2)
- new net: U21. (Φ2), U29., U30. (Φ2), U38. (Φ2)
- new net: U25. (Φ2), U27.
- new net: U25. (Φ2), U26.
- new net: U10., U5., U9.
- new net: U2., U3., U6.
- new net: U30. (Φ2), U31. (Φ2)
- new net: U35., U36. (Φ2)
Changed lines of the file:
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@@
   (title_block
     (title "V9958")
-    (date "2024-08-24")
+    (date "2024-09-13")
     (rev "WIP")
     (company "IKA Microelectronics Inc.")

Commit message: update 20241020
Connections:
- net at U18.: now also U24. (Φ2); no longer U17. (Φ2)
- net at U43.: now also U44.; no longer U42.
- net at U48.: now also U21. (Φ2), U46.; no longer U47.
- net at U40.: now also U45.; no longer U39.
- net at U27.: now also U16.; no longer U25. (Φ2)
- new net: U18., U19. (Φ2), U20. (Φ2), U29.
- new net: U18., U20. (Φ2), U28.
- new net: U17. (Φ2), U18., U19. (Φ2), U28., U29.
- new net: U17. (Φ2), U18.
- new net: U18., U36. (Φ2)
- new net: U18., U23. (Φ2), U24. (Φ2)
- new net: U1., U2., U8.
- new net: U1., U6., U7.
- new net: U42., U43.
- new net: U47., U48.
- new net: U38. (Φ2), U39.
- new net: U39., U40.
- new net: U31. (Φ2), U32. (Φ2), U35.
- new net: U32. (Φ2), U35.
- new net: U10., U11., U13.
- new net: U37. (Φ2), U49., U50.
- new net: U22. (Φ2), U23. (Φ2)
- new net: U16., U22. (Φ2)
- new net: U11., U12., U9.
- new net: U28., U37. (Φ2), U41. (Φ2)
- new net: U21. (Φ2), U29., U30. (Φ2), U38. (Φ2)
- new net: U25. (Φ2), U27.
- new net: U25. (Φ2), U26.
- new net: U10., U5., U9.
- new net: U2., U3., U6.
- new net: U30. (Φ2), U31. (Φ2)
- new net: U35., U36. (Φ2)
Other:
- sheet VT renamed PLA0
- sheet PLA0: file VT.kicad_sch -> PLA0.kicad_sch
Changed lines of the file:
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@@
     (stroke (width 0.1524) (type solid))
     (fill (color 0 0 0 0.0000))
-    (property "Sheetname" "VT" (at 78.74 264.7184 0)
+    (property "Sheetname" "PLA0" (at 78.74 264.7184 0)
       (effects (font (size 1.27 1.27)) (justify left bottom))
     )
-    (property "Sheetfile" "VT.kicad_sch" (at 78.74 297.7646 0)
+    (property "Sheetfile" "PLA0.kicad_sch" (at 78.74 297.7646 0)
       (effects (font (size 1.27 1.27)) (justify left top))
     )

Commit message: update 20250809
HVCNTR
Connections:
- net at U18.: now also U24. (Φ2); no longer U17. (Φ2)
- net at U43.: now also U44.; no longer U42.
- net at U48.: now also U21. (Φ2), U46.; no longer U47.
- net at U40.: now also U45.; no longer U39.
- net at U27.: now also U16.; no longer U25. (Φ2)
- new net: U18., U19. (Φ2), U20. (Φ2), U29.
- new net: U18., U20. (Φ2), U28.
- new net: U17. (Φ2), U18., U19. (Φ2), U28., U29.
- new net: U17. (Φ2), U18.
- new net: U18., U36. (Φ2)
- new net: U18., U23. (Φ2), U24. (Φ2)
- new net: U1., U2., U8.
- new net: U1., U6., U7.
- new net: U42., U43.
- new net: U47., U48.
- new net: U38. (Φ2), U39.
- new net: U39., U40.
- new net: U31. (Φ2), U32. (Φ2), U35.
- new net: U32. (Φ2), U35.
- new net: U10., U11., U13.
- new net: U37. (Φ2), U49., U50.
- new net: U22. (Φ2), U23. (Φ2)
- new net: U16., U22. (Φ2)
- new net: U11., U12., U9.
- new net: U28., U37. (Φ2), U41. (Φ2)
- new net: U21. (Φ2), U29., U30. (Φ2), U38. (Φ2)
- new net: U25. (Φ2), U27.
- new net: U25. (Φ2), U26.
- new net: U10., U5., U9.
- new net: U2., U3., U6.
- new net: U30. (Φ2), U31. (Φ2)
- new net: U35., U36. (Φ2)
Other:
- added sheet HVCNTR (HVCNTR.kicad_sch)
- added sheet PLA1 (PLA1.kicad_sch)

Commit message: update 20251028
Parts:
- removed U1, U10, U11, U12, U13, U44, U45, U6, U7, U8: NMOS, symbol Raki_ASIC_cells:NMOS
- removed U16: AND2, symbol Raki_ASIC_cells:AND2
- removed U17, U19, U20, U21, U22, U23, U24, U25, U30, U31, U32, U36, U37, U38, U41: DSR, symbol Raki_ASIC_cells:VY_DSR_small
- removed U18: NOR6, symbol Raki_ASIC_cells:NOR6
- removed U2, U28, U29, U39, U46, U47, U50, U51, U9: NOR2, symbol Raki_ASIC_cells:NOR2
- removed U26: BUF, symbol Raki_ASIC_cells:BUF
- removed U27: INVP, symbol Raki_ASIC_cells:INVP
- removed U3, U4, U42, U48, U49, U5: INV, symbol Raki_ASIC_cells:INV
- removed U35: NOR4, symbol Raki_ASIC_cells:NOR4
- removed U40, U43: BUFP, symbol Raki_ASIC_cells:BUFP
Connections:
- no-connect marks 15 -> 0
Other:
- sheet HVCNTR renamed ST
- sheet ST: file HVCNTR.kicad_sch -> ST.kicad_sch
- note removed: "0"
- note removed: "1"
- note removed: "2"
- note removed: "3"
- note removed: "A"
- note removed: "B"
- note removed: "INTERNAL CLOCK DIVIDER"
- note removed: "Super duper high side bootstrapped NOR2"

Commit message: update 20251106
Other:
- added sheet RCC (RCC.kicad_sch)
Changed lines of the file:
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@@
 	(title_block
 		(title "V9958")
-		(date "2024-09-13")
+		(date "2025-11-06")
 		(rev "WIP")
 		(company "IKA Microelectronics Inc.")
@@
 			(project "V9958"
 				(path "/b5e1370a-fef4-4131-9314-bdfc21cb5e0f"
-					(page "3")
+					(page "4")
 				)
 			)
@@
 			(project "V9958"
 				(path "/b5e1370a-fef4-4131-9314-bdfc21cb5e0f"
-					(page "6")
+					(page "7")
 				)
 			)
@@
 			(project "V9958"
 				(path "/b5e1370a-fef4-4131-9314-bdfc21cb5e0f"
-					(page "2")
+					(page "5")
 				)
 			)
@@
 			(project "V9958"
 				(path "/b5e1370a-fef4-4131-9314-bdfc21cb5e0f"
-					(page "7")
+					(page "2")
+				)
+			)
+		)
+	)
+	(sheet
+		(at 31.75 304.8)
+		(size 26.67 12.7)
+		(fields_autoplaced yes)
+		(stroke
+			(width 0.1524)
+			(type solid)
+		)
+		(fill
+			(color 0 0 0 0.0000)
+		)
+		(property "Sheetname" "RCC"
+			(at 31.75 304.0884 0)
+			(effects
+				(font
+					(size 1.27 1.27)
+				)
+				(justify left bottom)
+			)
+		)
+		(property "Sheetfile" "RCC.kicad_sch"
+			(at 31.75 318.0846 0)
+			(effects
+				(font
+					(size 1.27 1.27)
+				)
+				(justify left top)
+			)
+		)
+		(instances
+			(project "V9958"
+				(path "/b5e1370a-fef4-4131-9314-bdfc21cb5e0f"
+					(page "1")
 				)
 			)
@@
 			(project "V9958"
 				(path "/b5e1370a-fef4-4131-9314-bdfc21cb5e0f"
-					(page "5")
+					(page "6")
 				)
 			)
@@
 			(project "V9958"
 				(path "/b5e1370a-fef4-4131-9314-bdfc21cb5e0f"
-					(page "4")
-				)
-			)
+					(page "3")
+				)
+			)
